File: AppleII/FujiApple-DevKit-Combo-Rev1/FujiApple-DevKit-Combo.kicad_sch (KiCad schematic)
At the start: 31 parts, among them J1 DB19_Plug, J2 Conn_02x10_Odd_Even, P1 ST-TF-003A, SW1 ButtonA, SW2 Reset, U1 LSF0204DPWR, U2 LSF0204DPWR, U3 LSF0204DPWR, U4 ESP32-DevKitC-VE, U5 SFH690AT

Commit message: Update Apple II docs
Parts:
- C2: value 47uF 10v -> 220uF 10v
- R2: value 1.2K -> 1K
Changed lines of the file:
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@@
       (effects (font (size 1.27 1.27)))
     )
-    (property "Value" "1.2K" (at 52.07 38.1 90)
+    (property "Value" "1K" (at 52.07 38.1 90)
       (effects (font (size 1.27 1.27)))
     )
@@
       (effects (font (size 1.27 1.27)) (justify left))
     )
-    (property "Value" "47uF 10v" (at 153.67 153.67 0)
+    (property "Value" "220uF 10v" (at 153.67 153.67 0)
       (effects (font (size 1.27 1.27)) (justify left))
     )

Commit message: Fix BOM for Apple II DevKit flavors, should be LSF0204PWR (no D)
Parts:
- U1, U2, U3: value LSF0204DPWR -> LSF0204PWR
Changed lines of the file:
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@@
       (effects (font (size 1.524 1.524)))
     )
-    (property "Value" "LSF0204DPWR" (at 99.06 157.48 0)
+    (property "Value" "LSF0204PWR" (at 99.06 157.48 0)
       (effects (font (size 1.524 1.524)))
     )
@@
       (effects (font (size 1.27 1.27) italic) hide)
     )
-    (property "Datasheet" "LSF0204DPWR" (at 99.06 170.18 0)
+    (property "Datasheet" "LSF0204PWR" (at 99.06 170.18 0)
       (effects (font (size 1.27 1.27) italic) hide)
     )
@@
       (effects (font (size 1.524 1.524)))
     )
-    (property "Value" "LSF0204DPWR" (at 99.06 90.17 0)
+    (property "Value" "LSF0204PWR" (at 99.06 90.17 0)
       (effects (font (size 1.524 1.524)))
     )
@@
       (effects (font (size 1.27 1.27) italic) hide)
     )
-    (property "Datasheet" "LSF0204DPWR" (at 99.06 102.87 0)
+    (property "Datasheet" "LSF0204PWR" (at 99.06 102.87 0)
       (effects (font (size 1.27 1.27) italic) hide)
     )
@@
       (effects (font (size 1.524 1.524)))
     )
-    (property "Value" "LSF0204DPWR" (at 99.06 124.46 0)
+    (property "Value" "LSF0204PWR" (at 99.06 124.46 0)
       (effects (font (size 1.524 1.524)))
     )
@@
       (effects (font (size 1.27 1.27) italic) hide)
     )
-    (property "Datasheet" "LSF0204DPWR" (at 99.06 137.16 0)
+    (property "Datasheet" "LSF0204PWR" (at 99.06 137.16 0)
       (effects (font (size 1.27 1.27) italic) hide)
     )
