File: AppleII/FujiApple-DevKit-IDC-20-Rev1/FujiApple-DevKit-IDC-20.kicad_pcb (KiCad board)
At the start: 2 copper layers, 41 x 56.9 mm, 32 parts, among them J1 Conn_02x10_Odd_Even, P1 ST-TF-003A, SW1 ButtonA, SW2 Reset, U1 LSF0204DPWR, U2 LSF0204DPWR, U3 LSF0204DPWR, U4 ESP32-DevKitC-VE, U5 SFH690AT

Commit message: Update Apple II docs
Parts:
- C2: value 47uF 10v -> 220uF 10v
- R2: value 1.2K -> 1K

Commit message: Fix BOM for Apple II DevKit flavors, should be LSF0204PWR (no D)
Parts:
- U1, U2, U3: value LSF0204DPWR -> LSF0204PWR
Changed lines of the file:
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@@
         (effects (font (size 1 1) (thickness 0.15)))
     )
-    (fp_text value "LSF0204DPWR" (at 0 3.45 -90) (layer "F.Fab")
+    (fp_text value "LSF0204PWR" (at 0 3.45 -90) (layer "F.Fab")
         (effects (font (size 1 1) (thickness 0.15)))
     )
@@
         (effects (font (size 1 1) (thickness 0.15)))
     )
-    (fp_text value "LSF0204DPWR" (at 0 3.45 -90) (layer "F.Fab")
+    (fp_text value "LSF0204PWR" (at 0 3.45 -90) (layer "F.Fab")
         (effects (font (size 1 1) (thickness 0.15)))
     )
@@
         (effects (font (size 1 1) (thickness 0.15)))
     )
-    (fp_text value "LSF0204DPWR" (at 0 3.45 -90) (layer "F.Fab")
-        (effects (font (size 1 1) (thickness 0.15)))
-    )
+    (fp_text value "LSF0204PWR" (at 0 3.45 -90) (layer "F.Fab")
+        (effects (font (size 1 1) (thickness 0.15)))
+    )
