File: NES/FujiNet-NES-Rev0/esp32s3-sd.kicad_sch (KiCad schematic)
At the start: 14 parts, among them J2 microSD, SW3 S3_RST, SW4 S3_BOOT, U9 ESP32-S3-WROOM-1-N16R8

Commit message: NES Rev0: audit the schematic with kicad-happy and redo it
Datasheet-backed review of the first Rev0 schematic (kicad-happy analyzer,
ngspice, 28 deep-review findings all evidence-gated, 453 netlist checks
against fujinet-firmware nes-bringup) and the fixes it called for:

- edge footprint was mirrored (pin 1 west); nesdev and two measured
  NES-EWROM-01 references put pin 1 east on the label side. Fingers are now
  2.0 x 12 mm (ends 3.0 at +/-44.25), 2.50 pitch, copper 1.0-13.0 mm in,
  Nintendo's front/back mask depths
- RP2350 pads are 5 V-tolerant only while IOVDD is powered: the IOVDD group
  moves to an AP2112K (20 us) rail +3V3_RP; VREG_VIN stays on the buck
- 74HCT595 /OE = NAND(PWR_OK, POR) with 100k pull-downs on every bit, so
  the register cannot enable the SRAMs before the RP loads it or while
  the console is off
- PRG /WE = NAND4(M2, ROMSEL, !R/W, PRG_WE_EN) on a CD74HCT20, one gate
  after M2 (was three after the console's /ROMSEL decoder vs ~30 ns hold)
- CIRAM /CE through the 74HCT253's second half, tri-stated by PWR_OK_N
- console 5 V through an AO3401A P-FET (gate = VBUS) instead of a Schottky
- console-sense divider 22k/100k (TI 74HCT14 VT+ reaches 0.70 x VCC)
- WS2812B-2020 on +5V (datasheet VDD 3.7-5.3 V, VIH 2.7 V)
- VBUS decoupling at the USB-C; CIClone (ATtiny13A, DNP) on the CIC pins

tools: design.py is the source of truth as before; check_nets.py verifies
the new decode gate by gate and asserts the edge orientation from the
footprint file; make_fp_extra.py adds SOT-23-5 / SOIC-8; export.py flags
DNP; .kicad-happy.json documents the analyzer suppressions;
docs/design-review-rev0.md is the review; tools/audit/ holds the
computations the review cites.

Co-Authored-By: Claude Fable 5.1 <noreply@anthropic.com>
Parts:
- removed C29: 22uF, FujiNet-NES:C_0805_2012Metric, symbol Device:C
- removed C30: 100nF, FujiNet-NES:C_0603_1608Metric, symbol Device:C
- removed C31: 1uF, FujiNet-NES:C_0603_1608Metric, symbol Device:C
- removed R13: 10k, FujiNet-NES:R_0603_1608Metric, symbol Device:R
- removed RN1: 4x10k, FujiNet-NES:R_Array_Convex_4x0603, symbol Device:R_Pack04
- removed U9: ESP32-S3-WROOM-1-N16R8, FujiNet-NES:ESP32-S3-WROOM-1, symbol RF_Module:ESP32-S3-WROOM-1
- added C34: 1uF, FujiNet-NES:C_0603_1608Metric, symbol Device:C
- added C35: 10uF, FujiNet-NES:C_0603_1608Metric, symbol Device:C
- added C36: 100nF, FujiNet-NES:C_0603_1608Metric, symbol Device:C
- added R16: 330R, FujiNet-NES:R_0603_1608Metric, symbol Device:R
- added RN3: 4x10k, FujiNet-NES:R_Array_Convex_4x0603, symbol Device:R_Pack04
- added U11: ESP32-S3-WROOM-1-N16R8, FujiNet-NES:ESP32-S3-WROOM-1, symbol RF_Module:ESP32-S3-WROOM-1
- C32: value 10uF -> 22uF; footprint FujiNet-NES:C_0603_1608Metric -> FujiNet-NES:C_0805_2012Metric; LCSC C19702 -> C45783; MPN CL10A106KP8NNNC -> CL21A226MAQNNNE
- R15: value 330R -> 10k; LCSC C23138 -> C25804; MPN 0603WAF3300T5E -> 0603WAF1002T5E
Connections:
- net +3V3: now also R15.1, C35.1, RN3.5 (R4.2), RN3.6 (R3.2), RN3.7 (R2.2), RN3.8 (R1.2), U11.2 (3V3); no longer D3.4 (VDD)
- net BOOTSEL_CTL: now also U11.5 (IO5)
- net GND: now also C34.2, C35.2, C36.2, U11.1 (GND), U11.40 (GND), U11.41 (GND)
- net LED_STRIP: now also R16.1, U11.25 (IO48); no longer R15.1
- net RUN_CTL: now also U11.4 (IO4)
- net S3_EN: now also R14.2, C34.1, U11.3 (EN)
- net S3_IO0: now also U11.27 (IO0)
- net S3_RXD: now also U11.36 (RXD0)
- net S3_TXD: now also U11.37 (TXD0)
- net SD_CD: now also R15.2, U11.35 (IO42); no longer R14.2
- net SD_CS: now also RN3.1 (R1.1), U11.34 (IO41)
- net SD_DAT1: now also RN3.3 (R3.1)
- net SD_DAT2: now also RN3.4 (R4.1)
- net SD_MISO: now also RN3.2 (R2.1), U11.33 (IO40)
- net SD_MOSI: now also U11.31 (IO38)
- net SD_SCK: now also U11.32 (IO39)
- net USB_DM: now also U11.13 (USB_D-)
- net USB_DP: now also U11.14 (USB_D+)
- net WS_DIN: now also R16.2; no longer R15.2
- new net +5V: C36.1, D3.4 (VDD)
Other:
- moved on the sheet: C32, C33, D3, R14, R15
Changed lines of the file:
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@@
 	(title_block
 		(title "FujiNet NES Rev0 - ESP32-S3 FujiNet core, microSD, status LED")
-		(date "2026-09-30")
+		(date "2026-10-01")
 		(rev "0")
 		(company "FujiNet")
 		(comment 1 "Generated by tools/gen_sch.py from tools/design.py - edit design.py, not this file")
 		(comment 2 "CERN-OHL-W-2.0 (derived from FujiNet-Astrocade-Rev0 / FujiNet-INTV-Rev0 / PiNTY CARD)")
+		(comment 3 "Rev0 audit 2026-10-01: kicad-happy + datasheets; see docs/design-review-rev0.md")
 	)
 	(symbol
@@
 		(on_board yes)
 		(dnp no)
-		(property "Reference" "U9"
+		(property "Reference" "U11"
 			(at 45.72 32.37 0)
 			(effects
@@
 			(project "FujiNet-NES-Rev0"
 				(path "/5810f54f-2240-53c0-bbad-5b0b7a2c3f6b/81529a91-63f4-52a2-8914-d0d150a26d30"
-					(reference "U9")
+					(reference "U11")
 					(unit 1)
 				)
@@
 		(on_board yes)
 		(dnp no)
-		(property "Reference" "C29"
+		(property "Reference" "C32"
 			(at 125.222 41.91 0)
 			(effects
@@
 			(project "FujiNet-NES-Rev0"
 				(path "/5810f54f-2240-53c0-bbad-5b0b7a2c3f6b/81529a91-63f4-52a2-8914-d0d150a26d30"
-					(reference "C29")
+					(reference "C32")
 					(unit 1)
 				)
@@
 		(on_board yes)
 		(dnp no)
-		(property "Reference" "C30"
+		(property "Reference" "C33"
 			(at 143.002 41.91 0)
 			(effects
@@
 			(project "FujiNet-NES-Rev0"
 				(path "/5810f54f-2240-53c0-bbad-5b0b7a2c3f6b/81529a91-63f4-52a2-8914-d0d150a26d30"
-					(reference "C30")
+					(reference "C33")
 					(unit 1)
 				)
@@
 		(on_board yes)
 		(dnp no)
-		(property "Reference" "R13"
+		(property "Reference" "R14"
 			(at 159.766 41.91 0)
 			(effects
@@
 			(project "FujiNet-NES-Rev0"
 				(path "/5810f54f-2240-53c0-bbad-5b0b7a2c3f6b/81529a91-63f4-52a2-8914-d0d150a26d30"
-					(reference "R13")
+					(reference "R14")
 					(unit 1)
 				)
@@
 		(on_board yes)
 		(dnp no)
-		(property "Reference" "C31"
+		(property "Reference" "C34"
 			(at 176.022 41.91 0)
 			(effects
@@
 			(project "FujiNet-NES-Rev0"
 				(path "/5810f54f-2240-53c0-bbad-5b0b7a2c3f6b/81529a91-63f4-52a2-8914-d0d150a26d30"
-					(reference "C31")
+					(reference "C34")
 					(unit 1)
 				)
@@
 		(on_board yes)
 		(dnp no)
-		(property "Reference" "RN1"
+		(property "Reference" "RN3"
 			(at 259.08 32.37 0)
 			(effects
@@
 			(project "FujiNet-NES-Rev0"
 				(path "/5810f54f-2240-53c0-bbad-5b0b7a2c3f6b/81529a91-63f4-52a2-8914-d0d150a26d30"
-					(reference "RN1")
+					(reference "RN3")
 					(unit 1)
 				)
@@
 		(on_board yes)
 		(dnp no)
-		(property "Reference" "R14"
+		(property "Reference" "R15"
 			(at 274.066 41.91 0)
 			(effects
@@
 			(project "FujiNet-NES-Rev0"
 				(path "/5810f54f-2240-53c0-bbad-5b0b7a2c3f6b/81529a91-63f4-52a2-8914-d0d150a26d30"
-					(reference "R14")
+					(reference "R15")
 					(unit 1)
 				)
@@
 		(on_board yes)
 		(dnp no)
-		(property "Reference" "C32"
+		(property "Reference" "C35"
 			(at 290.322 41.91 0)
 			(effects
@@
 			(project "FujiNet-NES-Rev0"
 				(path "/5810f54f-2240-53c0-bbad-5b0b7a2c3f6b/81529a91-63f4-52a2-8914-d0d150a26d30"
-					(reference "C32")
+					(reference "C35")
 					(unit 1)
 				)
@@
 		(on_board yes)
 		(dnp no)
-		(property "Reference" "R15"
+		(property "Reference" "R16"
 			(at 304.546 46.99 0)
 			(effects
@@
 			(project "FujiNet-NES-Rev0"
 				(path "/5810f54f-2240-53c0-bbad-5b0b7a2c3f6b/81529a91-63f4-52a2-8914-d0d150a26d30"
-					(reference "R15")
+					(reference "R16")
 					(unit 1)
 				)
@@
 	(symbol
 		(lib_id "LED:WS2812B-2020")
-		(at 335.28 50.8 0)
+		(at 335.28 48.26 0)
 		(unit 1)
 		(exclude_from_sim no)
@@
 		(dnp no)
 		(property "Reference" "D3"
-			(at 335.28 32.37 0)
+			(at 335.28 30.83 0)
 			(effects
 				(font
@@
 		)
 		(property "Value" "WS2812B-2020-V6"
-			(at 335.28 34.91 0)
+			(at 335.28 33.37 0)
 			(effects
 				(font
@@
 		)
 		(property "Footprint" "FujiNet-NES:LED_WS2812B-2020_PLCC4_2.0x2.0mm"
-			(at 335.28 50.8 0)
+			(at 335.28 48.26 0)
 			(effects
 				(font
@@
 		)
 		(property "Datasheet" "https://cdn-shop.adafruit.com/product-files/4684/4684_WS2812B-2020_V1.3_EN.pdf"
-			(at 335.28 50.8 0)
-			(effects
-				(font
-					(size 1.27 1.27)
-				)
-				(hide yes)
-			)
-		)
-		(property "Description" "status LED (3.3V-rated V6 part: no data-level shifting needed)"
-			(at 335.28 50.8 0)
+			(at 335.28 48.26 0)
+			(effects
+				(font
+					(size 1.27 1.27)
+				)
+				(hide yes)
+			)
+		)
+		(property "Description" "status LED on +5V (datasheet VDD 3.7-5.3 V; VIH 2.7 V takes the S3 3.3 V data directly)"
+			(at 335.28 48.26 0)
 			(effects
 				(font
@@
 		)
 		(property "MPN" "WS2812B-2020-V6"
-			(at 335.28 50.8 0)
+			(at 335.28 48.26 0)
 			(effects
 				(font
@@
 		)
 		(property "LCSC" "C52917434"
-			(at 335.28 50.8 0)
+			(at 335.28 48.26 0)
 			(effects
 				(font
@@
 	)
 	(no_connect
-		(at 342.9 50.8)
+		(at 342.9 48.26)
 	)
 	(global_label "GND"
 		(shape passive)
-		(at 335.28 58.42 90)
+		(at 335.28 55.88 90)
 		(fields_autoplaced yes)
 		(effects
@@
 	(global_label "WS_DIN"
 		(shape passive)
-		(at 327.66 50.8 0)
-		(fields_autoplaced yes)
-		(effects
-			(font
-				(size 1.27 1.27)
-			)
-			(justify right)
-		)
-	)
-	(global_label "+3V3"
-		(shape passive)
-		(at 335.28 43.18 270)
+		(at 327.66 48.26 0)
+		(fields_autoplaced yes)
+		(effects
+			(font
+				(size 1.27 1.27)
+			)
+			(justify right)
+		)
+	)
+	(global_label "+5V"
+		(shape passive)
+		(at 335.28 40.64 270)
 		(fields_autoplaced yes)
 		(effects
@@
 	(symbol
 		(lib_id "Device:C")
-		(at 353.06 43.18 0)
+		(at 353.06 40.64 0)
 		(unit 1)
 		(exclude_from_sim no)
@@
 		(on_board yes)
 		(dnp no)
-		(property "Reference" "C33"
+		(property "Reference" "C36"
+			(at 356.362 39.37 0)
+			(effects
+				(font
+					(size 1.27 1.27)
+				)
+				(justify left)
+			)
+		)
+		(property "Value" "100nF"
 			(at 356.362 41.91 0)
 			(effects
@@
 			)
 		)
-		(property "Value" "100nF"
-			(at 356.362 44.45 0)
-			(effects
-				(font
-					(size 1.27 1.27)
-				)
-				(justify left)
-			)
-		)
 		(property "Footprint" "FujiNet-NES:C_0603_1608Metric"
-			(at 353.06 43.18 0)
+			(at 353.06 40.64 0)
 			(effects
 				(font
@@
 		)
 		(property "Datasheet" ""
-			(at 353.06 43.18 0)
+			(at 353.06 40.64 0)
 			(effects
 				(font
@@
 		)
 		(property "Description" "WS2812 decoupling"
-			(at 353.06 43.18 0)
+			(at 353.06 40.64 0)
 			(effects
 				(font
@@
 		)
 		(property "MPN" "CC0603KRX7R9BB104"
-			(at 353.06 43.18 0)
+			(at 353.06 40.64 0)
 			(effects
 				(font
@@
 		)
 		(property "LCSC" "C14663"
-			(at 353.06 43.18 0)
+			(at 353.06 40.64 0)
 			(effects
 				(font
@@
 			(project "FujiNet-NES-Rev0"
 				(path "/5810f54f-2240-53c0-bbad-5b0b7a2c3f6b/81529a91-63f4-52a2-8914-d0d150a26d30"
-					(reference "C33")
+					(reference "C36")
 					(unit 1)
 				)
@@
 		)
 	)
-	(global_label "+3V3"
-		(shape passive)
-		(at 353.06 39.37 270)
+	(global_label "+5V"
+		(shape passive)
+		(at 353.06 36.83 270)
 		(fields_autoplaced yes)
 		(effects
@@
 	(global_label "GND"
 		(shape passive)
-		(at 353.06 46.99 90)
-		(fields_autoplaced yes)
-		(effects
+		(at 353.06 44.45 90)
+		(fields_autoplaced yes)
+		(effects
