File: NES/FujiNet-NES-Rev0/esp32s3-sd.kicad_sch (KiCad schematic)
At the start: 14 parts, among them J2 microSD, SW3 S3_RST, SW4 S3_BOOT, U11 ESP32-S3-WROOM-1-N16R8

Commit message: [nes] redo schematic1
Other:
- title: FujiNet NES Rev0 - ESP32-S3 FujiNet core, microSD, status LED -> FujiNet NES Rev0 - ESP32-S3, microSD, status LED
- moved on the sheet: C32, C33, C34, C35, C36, D3, J2, R14, R15, R16, RN3, SW3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
