File: NES/FujiNet-NES-Rev0/cart-rp2354b.kicad_sch (KiCad schematic)
At the start: 61 parts, among them J1 NES_Cart_Edge_72, SW1 RESET, SW2 BOOTSEL, U1 RP2354B, U2 AS6C4008-55TIN, U3 AS6C4008-55TIN, U4 74HCT595, U5 74HCT253, U6 74HCT14, U7 74HCT00, U8 74HCT32, Y1 12MHz

Commit message: NES Rev0: audit the schematic with kicad-happy and redo it
Datasheet-backed review of the first Rev0 schematic (kicad-happy analyzer,
ngspice, 28 deep-review findings all evidence-gated, 453 netlist checks
against fujinet-firmware nes-bringup) and the fixes it called for:

- edge footprint was mirrored (pin 1 west); nesdev and two measured
  NES-EWROM-01 references put pin 1 east on the label side. Fingers are now
  2.0 x 12 mm (ends 3.0 at +/-44.25), 2.50 pitch, copper 1.0-13.0 mm in,
  Nintendo's front/back mask depths
- RP2350 pads are 5 V-tolerant only while IOVDD is powered: the IOVDD group
  moves to an AP2112K (20 us) rail +3V3_RP; VREG_VIN stays on the buck
- 74HCT595 /OE = NAND(PWR_OK, POR) with 100k pull-downs on every bit, so
  the register cannot enable the SRAMs before the RP loads it or while
  the console is off
- PRG /WE = NAND4(M2, ROMSEL, !R/W, PRG_WE_EN) on a CD74HCT20, one gate
  after M2 (was three after the console's /ROMSEL decoder vs ~30 ns hold)
- CIRAM /CE through the 74HCT253's second half, tri-stated by PWR_OK_N
- console 5 V through an AO3401A P-FET (gate = VBUS) instead of a Schottky
- console-sense divider 22k/100k (TI 74HCT14 VT+ reaches 0.70 x VCC)
- WS2812B-2020 on +5V (datasheet VDD 3.7-5.3 V, VIH 2.7 V)
- VBUS decoupling at the USB-C; CIClone (ATtiny13A, DNP) on the CIC pins

tools: design.py is the source of truth as before; check_nets.py verifies
the new decode gate by gate and asserts the edge orientation from the
footprint file; make_fp_extra.py adds SOT-23-5 / SOIC-8; export.py flags
DNP; .kicad-happy.json documents the analyzer suppressions;
docs/design-review-rev0.md is the review; tools/audit/ holds the
computations the review cites.

Co-Authored-By: Claude Fable 5.1 <noreply@anthropic.com>
Parts:
- removed unit 4 of U7
- removed unit 5 of U7
- added C29, C30, C31: 100nF, FujiNet-NES:C_0603_1608Metric, symbol Device:C
- added R13: 1k, FujiNet-NES:R_0603_1608Metric, symbol Device:R
- added RN1, RN2: 4x100k, FujiNet-NES:R_Array_Convex_4x0603, symbol Device:R_Pack04
- added TP7: CIC_RST, FujiNet-NES:TestPoint_Pad_D1.5mm, symbol Connector:TestPoint
- added U10: ATtiny13A-SSU, FujiNet-NES:SOIC-8_3.9x4.9mm_P1.27mm, symbol MCU_Microchip_ATtiny:ATtiny13A-SS
- added U9: 74HCT32, FujiNet-NES:SOIC-14_3.9x8.7mm_P1.27mm, symbol 74xx:74LS32
- C12: value 4.7uF -> 10uF; LCSC C19666 -> C19702; MPN CL10A475KO8NNNC -> CL10A106KP8NNNC
- C13: value 10uF -> 4.7uF; LCSC C19702 -> C19666; MPN CL10A106KP8NNNC -> CL10A475KO8NNNC
- C21: value 100nF -> 1uF; LCSC C14663 -> C15849; MPN CC0603KRX7R9BB104 -> CL10A105KB8NNNC
- C23: value 10uF -> 100nF; LCSC C19702 -> C14663; MPN CL10A106KP8NNNC -> CC0603KRX7R9BB104
- C24: value 100nF -> 10uF; LCSC C14663 -> C19702; MPN CC0603KRX7R9BB104 -> CL10A106KP8NNNC
- R10: value 100k -> 22k; LCSC C25803 -> C31850; MPN 0603WAF1003T5E -> 0603WAF2202T5E
- R11: value 150k -> 100k; LCSC C22807 -> C25803; MPN 0603WAF1503T5E -> 0603WAF1003T5E
- R12: value 1k -> 100k; LCSC C21190 -> C25803; MPN 0603WAF1001T5E -> 0603WAF1003T5E
- U7: value 74HCT00 -> 74HCT20; symbol 74xx:74HCT00 -> 74xx:74LS20; LCSC C6764 -> C2878717; MPN SN74HCT00DR -> CD74HCT20M96
- U8: value 74HCT32 -> 74HCT00; symbol 74xx:74LS32 -> 74xx:74HCT00; LCSC C5985 -> C6764; MPN 74HCT32D,653 -> SN74HCT00DR
Connections:
- net FOURSCREEN_OK_N is gone; now on net RW: U6.11
- net +3V3: no longer C1.1, C10.1, C11.1, C12.1, C2.1, C3.1, C4.1, C5.1, C6.1, C7.1, C8.1, C9.1, R3.1, R4.1, U1.15 (IOVDD), U1.24 (IOVDD), U1.29 (IOVDD), U1.41 (IOVDD), U1.5 (IOVDD), U1.50 (IOVDD), U1.59 (ADC_AVDD), U1.60 (IOVDD), U1.68 (USB_OTP_VDD), U1.69 (QSPI_IOVDD), U1.76 (IOVDD)
- net +5V: now also C21.2, U7.12, U7.13, U7.14 (VCC), C29.1, C30.1, U9.14 (VCC); no longer C21.1, U5.15 (OEb)
- net CHR_OE_N: now also U9.3; no longer U8.3
- net CHR_WE_EN: now also RN1.3 (R3.1)
- net CHR_WE_EN_N: now also U9.5; no longer U8.5
- net CHR_WE_N: now also U9.6; no longer U8.6
- net CIRAM_CE_N: now also U5.9 (Zb); no longer U8.11
- net CONS_5V: now also C31.1, U10.8 (VCC)
- net FOURSCREEN: now also RN1.4 (R4.1), U9.13
- net GND: now also R12.2, U7.7 (GND), U8.10, U8.12, U8.13, U8.9, C29.2, C30.2, C31.2, RN1.5 (R4.2), RN1.6 (R3.2), RN1.7 (R2.2), RN1.8 (R1.2), RN2.5 (R4.2), RN2.6 (R3.2), RN2.7 (R2.2), RN2.8 (R1.2), U10.4 (GND), U9.10, U9.7 (GND), U9.9; no longer C21.2, U4.13 (~{OE}), U5.10 (I0b), U5.11 (I1b), U5.12 (I2b), U5.13 (I3b), U6.13
- net M2: now also U7.1
- net MIR0: now also RN2.1 (R1.1)
- net MIR1: now also RN2.2 (R2.1)
- net PA13_N: now also U9.12; no longer U8.12
- net PPU_RD_N: now also U9.1; no longer U8.1
- net PPU_WR_N: now also U9.4; no longer U8.4
- net PRG_CE_N: now also U7.8; no longer U7.3
- net PRG_OE_N: now also U8.3; no longer U7.6
- net PRG_WE_EN: now also U7.5, RN1.2 (R2.1); no longer U7.10
- net PRG_WE_N: now also U7.6; no longer U8.8
- net PWR_OK: now also U8.2, U8.4; no longer U7.5
- net PWR_OK_N: now also U5.15 (OEb), U9.2; no longer U8.2
- net ROMSEL: now also U7.2, U7.9; no longer U7.1, U7.9
- net RW: now also U8.1; no longer U7.4, U8.10
- net SRAM_EN: now also U7.10, RN1.1 (R1.1); no longer U7.2
- net SR_LED: now also R13.1, RN2.3 (R3.1); no longer R12.1
- net SR_LED_A: now also R13.2; no longer R12.2
- net SR_SPARE: now also RN2.4 (R4.1)
- net POR: now reaches U6.12
- net POR: now also U8.5
- net CIC_TOPAK: now reaches J1.34 (CIC toPak)
- net CIC_TOPAK: now also U10.6 (PB1)
- net CIC_TOMB: now reaches J1.35 (CIC toMB)
- net CIC_TOMB: now also U10.5 (PB0)
- net CIC_RST: now reaches J1.70 (CIC +RST)
- net CIC_RST: now also U10.7 (PB2)
- net CIC_CLK: now reaches J1.71 (CIC CLK)
- net CIC_CLK: now also U10.2 (PB3)
- net FOURSCREEN_OK renamed RW_N
- net RW_N: now also U7.4; no longer U8.13
- removed net PRG_WGATE_N: U7.8, U8.9
- new net +3V3_RP: C1.1, C10.1, C11.1, C12.1, C2.1, C3.1, C4.1, C5.1, C6.1, C7.1, C8.1, C9.1, R3.1, R4.1, U1.15 (IOVDD), U1.24 (IOVDD), U1.29 (IOVDD), U1.41 (IOVDD), U1.5 (IOVDD), U1.50 (IOVDD), U1.59 (ADC_AVDD), U1.60 (IOVDD), U1.68 (USB_OTP_VDD), U1.69 (QSPI_IOVDD), U1.76 (IOVDD)
- new net CIC_RESET_N: TP7.1, U10.1 (~{RESET}/PB5)
- new net CIRAM_CE_PRE: U5.10 (I0b), U5.11 (I1b), U5.12 (I2b), U5.13 (I3b), U9.11
- new net POR_RC: C21.1, R12.1, U6.13
- new net SR_OE_N: U4.13 (~{OE}), U8.6
- no-connect marks 23 -> 21
Other:
- title: FujiNet NES Rev0 - RP2354B bus controller, PRG/CHR SRAM, 5V glue, 72-pin edge -> FujiNet NES Rev0 - RP2354B bus controller, PRG/CHR SRAM, 5V glue, CIClone, 72-pin edge
- moved on the sheet: C1, C10, C11, C12, C13, C14, C15, C16, C17, C18, C19, C2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

Commit message: NES Rev0: route the 6-layer board and audit it with kicad-happy
Layout for the audited Rev0 schematic, generated by the tools/ pipeline
(gen_pcb + placement -> locked pre-routes -> Freerouting -> A* finisher
-> tidy -> GND stitching -> models -> export).

- 100 x 110 mm NES-EWROM-01 outline, 1.2 mm, 6 layers, all parts on the
  label side. KiCad DRC with schematic parity: 0 errors, 0 unconnected,
  0 parity issues. ERC clean; check_nets 453/453 against the firmware.
- RP2354B: VREG_VIN/VREG_AVDD join the IOVDD group on the fast LDO rail
  (+3V3_RP), as the datasheet pairs them. Decoupling ring at 10 mm, east
  IOVDD caps moved to the corner, plane vias of pins 24/29 pushed out
  (fanout.FAR_VIA) so pins 25-28 can escape; DVDD island covers the DVDD
  pin vias and has a 1.6 mm bridge to the regulator lobe.
- CHR-side glue ('32, '253) moved to a west column out of the PPU bus band;
  crystal block planar (R2 on the XOUT lane); SWD test pads ordered to
  match the pins; R8/R9 (USB D+/D-) placed so the pair does not cross.
- Finisher: island fills no longer block vias, cost-aware rip-up, no vias
  in or against own pads, escape lanes kept clear of tracks in the final
  0.15/0.12 mm neck-down pass (signal clearance floor 0.12 mm, above
  JLCPCB's 0.09). New tools: drc_fix.py, stitch_gnd.py (DRC-filtered GND
  grid, never in a pad), audit/run_pcb_audit.sh.
- Three fiducials, 3x3 thermal vias under the CP2102N exposed pad.
- docs/design-review-rev0.md Part 2: PCB, cross-domain, EMC, thermal and
  gerber analyzer results triaged; README status, rules and pipeline.
- exports/jlcpcb: gerbers, BOM, CPL (CIClone DNP); renders in docs/.
- case/: OpenSCAD shell and generated board anchors; 3d/: bundled models.

Co-Authored-By: Claude Opus 5.5 <noreply@anthropic.com>
Connections:
- net +3V3 is gone; now on net +3V3_RP: C13.1, R1.1, U1.64 (VREG_VIN)
Other:
- moved on the sheet: C13, R1
Changed lines of the file:
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@@
 		)
 	)
-	(global_label "+3V3"
+	(global_label "+3V3_RP"
 		(shape passive)
 		(at 58.42 48.26 270)
@@
 	(symbol
 		(lib_id "Device:C")
-		(at 243.84 231.14 0)
+		(at 243.84 236.22 0)
 		(unit 1)
 		(exclude_from_sim no)
@@
 		(dnp no)
 		(property "Reference" "C13"
-			(at 247.142 229.87 0)
+			(at 247.142 234.95 0)
 			(effects
 				(font
@@
 		)
 		(property "Value" "4.7uF"
-			(at 247.142 232.41 0)
+			(at 247.142 237.49 0)
 			(effects
 				(font
@@
 		)
 		(property "Footprint" "FujiNet-NES:C_0603_1608Metric"
-			(at 243.84 231.14 0)
+			(at 243.84 236.22 0)
 			(effects
 				(font
@@
 		)
 		(property "Datasheet" ""
-			(at 243.84 231.14 0)
+			(at 243.84 236.22 0)
 			(effects
 				(font
@@
 			)
 		)
-		(property "Description" "VREG_VIN bulk"
-			(at 243.84 231.14 0)
+		(property "Description" "VREG_VIN bulk (LDO rail)"
+			(at 243.84 236.22 0)
 			(effects
 				(font
@@
 		)
 		(property "MPN" "CL10A475KO8NNNC"
-			(at 243.84 231.14 0)
+			(at 243.84 236.22 0)
 			(effects
 				(font
@@
 		)
 		(property "LCSC" "C19666"
-			(at 243.84 231.14 0)
+			(at 243.84 236.22 0)
 			(effects
 				(font
@@
 		)
 	)
-	(global_label "+3V3"
+	(global_label "+3V3_RP"
 		(shape passive)
-		(at 243.84 227.33 270)
+		(at 243.84 232.41 270)
 		(fields_autoplaced yes)
 		(effects
@@
 	(global_label "GND"
 		(shape passive)
-		(at 243.84 234.95 90)
+		(at 243.84 240.03 90)
 		(fields_autoplaced yes)
 		(effects
@@
 	(symbol
 		(lib_id "Device:R")
-		(at 335.28 231.14 0)
+		(at 335.28 236.22 0)
 		(unit 1)
 		(exclude_from_sim no)
@@
 		(dnp no)
 		(property "Reference" "R1"
-			(at 337.566 229.87 0)
+			(at 337.566 234.95 0)
 			(effects
 				(font
@@
 		)
 		(property "Value" "33R"
-			(at 337.566 232.41 0)
+			(at 337.566 237.49 0)
 			(effects
 				(font
@@
 		)
 		(property "Footprint" "FujiNet-NES:R_0603_1608Metric"
-			(at 335.28 231.14 0)
+			(at 335.28 236.22 0)
 			(effects
 				(font
@@
 		)
 		(property "Datasheet" ""
-			(at 335.28 231.14 0)
+			(at 335.28 236.22 0)
 			(effects
 				(font
@@
 		)
 		(property "Description" "VREG_AVDD filter"
-			(at 335.28 231.14 0)
+			(at 335.28 236.22 0)
 			(effects
 				(font
@@
 		)
 		(property "MPN" "0603WAF330JT5E"
-			(at 335.28 231.14 0)
+			(at 335.28 236.22 0)
 			(effects
 				(font
@@
 		)
 		(property "LCSC" "C23140"
-			(at 335.28 231.14 0)
+			(at 335.28 236.22 0)
 			(effects
 				(font
@@
 		)
 	)
-	(global_label "+3V3"
+	(global_label "+3V3_RP"
 		(shape passive)
-		(at 335.28 227.33 270)
+		(at 335.28 232.41 270)
 		(fields_autoplaced yes)
 		(effects
@@
 	(global_label "VREG_AVDD"
 		(shape passive)
-		(at 335.28 234.95 90)
+		(at 335.28 240.03 90)
 		(fields_autoplaced yes)
 		(effects
