File: NES/FujiNet-NES-Rev0/FujiNet-NES-Rev0.kicad_sch (KiCad schematic)
At the start: 0 parts

Commit message: [nes] redo schematic1
Other:
- removed sheet cart-rp2354b
- added sheet edge-cic (edge-cic.kicad_sch)
- added sheet glue (glue.kicad_sch)
- added sheet rp2354b (rp2354b.kicad_sch)
- added sheet sram (sram.kicad_sch)
- note added: "5V glue logic, '595 control bits"
- note added: "72-pin cart edge, CIClone"
- note added: "ESP32-S3, microSD, status LED"
- note added: "PRG and CHR SRAM"
- note added: "Power: 5V OR, 3.3V buck, RP LDO"
- note added: "RP2354B bus controller"
- note added: "USB-C, CP2102N bridge"
- note removed: "ESP32-S3 FujiNet core, microSD, status LED"
- note removed: "Power: console 5V P-FET / USB VBUS OR, 3.3V buck, RP I/O LDO"
- note removed: "RP2354B bus controller, PRG/CHR SRAM, 5V glue, CIClone, 72-pin edge"
- note removed: "USB-C, CP2102N programming bridge"
Changed lines of the file:
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@@
 	(title_block
 		(title "FujiNet NES Rev0")
-		(date "2026-10-01")
+		(date "2026-10-04")
 		(rev "0")
 		(company "FujiNet")
@@
 	)
 	(sheet
-		(at 30 40)
-		(size 63.5 25.4)
-		(fields_autoplaced yes)
-		(stroke
-			(width 0.12)
-			(type solid)
-		)
-		(fill
-			(color 0 0 0 0)
-		)
-		(property "Sheetname" "cart-rp2354b"
-			(at 30 39 0)
-			(effects
-				(font
-					(size 1.27 1.27)
-				)
-				(justify left bottom)
-			)
-		)
-		(property "Sheetfile" "cart-rp2354b.kicad_sch"
-			(at 30 66.4 0)
+		(at 20.32 35.56)
+		(size 81.28 25.4)
+		(fields_autoplaced yes)
+		(stroke
+			(width 0.12)
+			(type solid)
+		)
+		(fill
+			(color 0 0 0 0)
+		)
+		(property "Sheetname" "edge-cic"
+			(at 20.32 34.56 0)
+			(effects
+				(font
+					(size 1.27 1.27)
+				)
+				(justify left bottom)
+			)
+		)
+		(property "Sheetfile" "edge-cic.kicad_sch"
+			(at 20.32 61.96 0)
 			(effects
 				(font
@@
 		)
 	)
-	(text "RP2354B bus controller, PRG/CHR SRAM, 5V glue, CIClone, 72-pin edge"
-		(exclude_from_sim no)
-		(at 30 52.7 0)
-		(effects
-			(font
-				(size 1.27 1.27)
-			)
-			(justify left)
-		)
-	)
-	(sheet
-		(at 120 40)
-		(size 63.5 25.4)
+	(text "72-pin cart edge, CIClone"
+		(exclude_from_sim no)
+		(at 22.86 40.64 0)
+		(effects
+			(font
+				(size 1.27 1.27)
+			)
+			(justify left top)
+		)
+	)
+	(sheet
+		(at 116.84 35.56)
+		(size 81.28 25.4)
+		(fields_autoplaced yes)
+		(stroke
+			(width 0.12)
+			(type solid)
+		)
+		(fill
+			(color 0 0 0 0)
+		)
+		(property "Sheetname" "rp2354b"
+			(at 116.84 34.56 0)
+			(effects
+				(font
+					(size 1.27 1.27)
+				)
+				(justify left bottom)
+			)
+		)
+		(property "Sheetfile" "rp2354b.kicad_sch"
+			(at 116.84 61.96 0)
+			(effects
+				(font
+					(size 1.27 1.27)
+				)
+				(justify left top)
+			)
+		)
+		(instances
+			(project "FujiNet-NES-Rev0"
+				(path "/5810f54f-2240-53c0-bbad-5b0b7a2c3f6b"
+					(page "3")
+				)
+			)
+		)
+	)
+	(text "RP2354B bus controller"
+		(exclude_from_sim no)
+		(at 119.38 40.64 0)
+		(effects
+			(font
+				(size 1.27 1.27)
+			)
+			(justify left top)
+		)
+	)
+	(sheet
+		(at 213.36 35.56)
+		(size 81.28 25.4)
+		(fields_autoplaced yes)
+		(stroke
+			(width 0.12)
+			(type solid)
+		)
+		(fill
+			(color 0 0 0 0)
+		)
+		(property "Sheetname" "sram"
+			(at 213.36 34.56 0)
+			(effects
+				(font
+					(size 1.27 1.27)
+				)
+				(justify left bottom)
+			)
+		)
+		(property "Sheetfile" "sram.kicad_sch"
+			(at 213.36 61.96 0)
+			(effects
+				(font
+					(size 1.27 1.27)
+				)
+				(justify left top)
+			)
+		)
+		(instances
+			(project "FujiNet-NES-Rev0"
+				(path "/5810f54f-2240-53c0-bbad-5b0b7a2c3f6b"
+					(page "4")
+				)
+			)
+		)
+	)
+	(text "PRG and CHR SRAM"
+		(exclude_from_sim no)
+		(at 215.9 40.64 0)
+		(effects
+			(font
+				(size 1.27 1.27)
+			)
+			(justify left top)
+		)
+	)
+	(sheet
+		(at 309.88 35.56)
+		(size 81.28 25.4)
+		(fields_autoplaced yes)
+		(stroke
+			(width 0.12)
+			(type solid)
+		)
+		(fill
+			(color 0 0 0 0)
+		)
+		(property "Sheetname" "glue"
+			(at 309.88 34.56 0)
+			(effects
+				(font
+					(size 1.27 1.27)
+				)
+				(justify left bottom)
+			)
+		)
+		(property "Sheetfile" "glue.kicad_sch"
+			(at 309.88 61.96 0)
+			(effects
+				(font
+					(size 1.27 1.27)
+				)
+				(justify left top)
+			)
+		)
+		(instances
+			(project "FujiNet-NES-Rev0"
+				(path "/5810f54f-2240-53c0-bbad-5b0b7a2c3f6b"
+					(page "5")
+				)
+			)
+		)
+	)
+	(text "5V glue logic, '595 control bits"
+		(exclude_from_sim no)
+		(at 312.42 40.64 0)
+		(effects
+			(font
+				(size 1.27 1.27)
+			)
+			(justify left top)
+		)
+	)
+	(sheet
+		(at 20.32 81.28)
+		(size 81.28 25.4)
 		(fields_autoplaced yes)
 		(stroke
@@
 		)
 		(property "Sheetname" "esp32s3-sd"
-			(at 120 39 0)
+			(at 20.32 80.28 0)
 			(effects
 				(font
@@
 		)
 		(property "Sheetfile" "esp32s3-sd.kicad_sch"
-			(at 120 66.4 0)
-			(effects
-				(font
-					(size 1.27 1.27)
-				)
-				(justify left top)
-			)
-		)
-		(instances
-			(project "FujiNet-NES-Rev0"
-				(path "/5810f54f-2240-53c0-bbad-5b0b7a2c3f6b"
-					(page "3")
-				)
-			)
-		)
-	)
-	(text "ESP32-S3 FujiNet core, microSD, status LED"
-		(exclude_from_sim no)
-		(at 120 52.7 0)
-		(effects
-			(font
-				(size 1.27 1.27)
-			)
-			(justify left)
-		)
-	)
-	(sheet
-		(at 210 40)
-		(size 63.5 25.4)
+			(at 20.32 107.68 0)
+			(effects
+				(font
+					(size 1.27 1.27)
+				)
+				(justify left top)
+			)
+		)
+		(instances
+			(project "FujiNet-NES-Rev0"
+				(path "/5810f54f-2240-53c0-bbad-5b0b7a2c3f6b"
+					(page "6")
+				)
+			)
+		)
+	)
+	(text "ESP32-S3, microSD, status LED"
+		(exclude_from_sim no)
+		(at 22.86 86.36 0)
+		(effects
+			(font
+				(size 1.27 1.27)
+			)
+			(justify left top)
+		)
+	)
+	(sheet
+		(at 116.84 81.28)
+		(size 81.28 25.4)
 		(fields_autoplaced yes)
 		(stroke
@@
 		)
 		(property "Sheetname" "usb-uart"
-			(at 210 39 0)
+			(at 116.84 80.28 0)
 			(effects
 				(font
@@
 		)
 		(property "Sheetfile" "usb-uart.kicad_sch"
-			(at 210 66.4 0)
-			(effects
-				(font
-					(size 1.27 1.27)
-				)
-				(justify left top)
-			)
-		)
-		(instances
-			(project "FujiNet-NES-Rev0"
-				(path "/5810f54f-2240-53c0-bbad-5b0b7a2c3f6b"
-					(page "4")
-				)
-			)
-		)
-	)
-	(text "USB-C, CP2102N programming bridge"
-		(exclude_from_sim no)
-		(at 210 52.7 0)
-		(effects
-			(font
-				(size 1.27 1.27)
-			)
-			(justify left)
-		)
-	)
-	(sheet
-		(at 300 40)
-		(size 63.5 25.4)
+			(at 116.84 107.68 0)
+			(effects
+				(font
+					(size 1.27 1.27)
+				)
+				(justify left top)
+			)
+		)
+		(instances
+			(project "FujiNet-NES-Rev0"
+				(path "/5810f54f-2240-53c0-bbad-5b0b7a2c3f6b"
+					(page "7")
+				)
+			)
+		)
+	)
+	(text "USB-C, CP2102N bridge"
+		(exclude_from_sim no)
+		(at 119.38 86.36 0)
+		(effects
+			(font
+				(size 1.27 1.27)
+			)
+			(justify left top)
+		)
+	)
+	(sheet
+		(at 213.36 81.28)
+		(size 81.28 25.4)
 		(fields_autoplaced yes)
 		(stroke
@@
 		)
 		(property "Sheetname" "power"
-			(at 300 39 0)
+			(at 213.36 80.28 0)
 			(effects
 				(font
@@
 		)
 		(property "Sheetfile" "power.kicad_sch"
-			(at 300 66.4 0)
-			(effects
-				(font
-					(size 1.27 1.27)
-				)
-				(justify left top)
-			)
-		)
-		(instances
-			(project "FujiNet-NES-Rev0"
-				(path "/5810f54f-2240-53c0-bbad-5b0b7a2c3f6b"
-					(page "5")
-				)
-			)
-		)
-	)
-	(text "Power: console 5V P-FET / USB VBUS OR, 3.3V buck, RP I/O LDO"
-		(exclude_from_sim no)
-		(at 300 52.7 0)
-		(effects
-			(font
-				(size 1.27 1.27)
-			)
-			(justify left)
+			(at 213.36 107.68 0)
+			(effects
+				(font
+					(size 1.27 1.27)
+				)
+				(justify left top)
+			)
+		)
+		(instances
+			(project "FujiNet-NES-Rev0"
+				(path "/5810f54f-2240-53c0-bbad-5b0b7a2c3f6b"
+					(page "8")
+				)
+			)
+		)
+	)
+	(text "Power: 5V OR, 3.3V buck, RP LDO"
+		(exclude_from_sim no)
+		(at 215.9 86.36 0)
+		(effects
+			(font
+				(size 1.27 1.27)
+			)
+			(justify left top)
 		)
 	)
 	(text "FujiNet for the Nintendo Entertainment System - Rev0 (RP2354B)\n\nRP2354B (48 GPIO) sits on the 5V cart bus directly through its 5V-tolerant pads: CPU A0-A14, D0-D7, M2, R/W,\n/ROMSEL, PPU A10-A12 in; /IRQ out; it serves $5000-$7FFF and the reset vectors itself and drives the two\nAS6C4008 SRAMs' bank lines (PRG A13-A18 = GP33-38, CHR A10-A18 = GP39-47) from PIO lookup tables.\nIts IOVDD group runs from a fast LDO (+3V3_RP) so the pads are powered before the console bus is; the core\nregulator input stays on the buck (+3V3).  The SRAMs and the 74HCT glue run on +5V: console 5V through a\nP-FET (on without USB) ORed with USB VBUS through a Schottky, so their outputs drive the 5V bus at full level.\n74HCT595 holds the slow control bits (SRAM_EN PRG_WE_EN CHR_WE_EN MIR0 MIR1 FOURSCREEN LED spare); its /OE\nis held off for ~140 ms after power-on and whenever the console is off, with 100k pull-downs on every bit.\n74HCT253 muxes CIRAM A10 for mirroring and gates CIRAM /CE; PWR_OK (console +5V sense) tri-states both and\ndisables every SRAM output toward the console.  PRG /WE = NAND4(M2, ROMSEL, !R/W, PRG_WE_EN) on a 74HCT20: one gate after M2.\nESP32-S3-WROOM-1-N16R8 runs FujiNet (fujiversal-nes) and is the USB host of the RP (CDC, VID 0xCafe);\nS3 IO4/IO5 force RP RUN/QSPI_SS so the S3 can re-flash the RP over PICOBOOT.\nUSB-C: power + CP2102N UART bridge for flashing the S3.  microSD on S3 SPI.  CIClone (ATtiny13A) on the\nCIC fingers, DNP until its firmware exists.\nEdge: 72 pins, 2.50 mm pitch, 1-36 on the label side, pin 1 at the RIGHT seen from the label side with the\nfingers down (nesdev Cartridge connector; NES-EWROM-01 geometry).  EXP and SYSTEM CLK unconnected."
 		(exclude_from_sim no)
-		(at 30 90 0)
-		(effects
-			(font
+		(at 20 125 0)
+		(effects
+			(font
