File: NES/FujiNet-NES-Rev0/power.kicad_sch (KiCad schematic)
At the start: 15 parts, among them Q1 AO3401A, U14 AP63203WU, U15 AP2112K-3.3

Commit message: [nes] redo schematic1
Other:
- title: FujiNet NES Rev0 - Power: console 5V P-FET / USB VBUS OR, 3.3V buck, RP I/O LDO -> FujiNet NES Rev0 - Power: 5V OR, 3.3V buck, RP LDO
- moved on the sheet: C41, C42, C43, C44, C45, C46, C47, C48, C49, C50, D7, L2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
