File: NES/FujiNet-NES-Rev0/power.kicad_sch (KiCad schematic)
At the start: 15 parts, among them Q1 AO3401A, U14 AP63203WU, U15 AP2112K-3.3

Commit message: NES Rev0: add the VBUS pull-down (R22 4.7k) against SS34 reverse leakage
Q1's gate is VBUS, which only the 69k CP2102N sense divider pulled down.
With the console powering the cart the SS34 is reverse-biased and leaks
into VBUS (0.5 mA max at 25 C); at >= 100 uA the AO3401A turns off and the
console feeds +5V through the body diode, ~0.7 V down, under the 74HCT /
SRAM 4.5 V minimum.  R22 4.7k VBUS-GND (0603WAF4701T5E, C23162) holds VGS
beyond -2.8 V up to 500 uA; same fix as 2600 Rev1 R_VBPD and SMS Rev0.

- design.py: R22 declared after every other resistor (no ref changes).
- power sheet redrawn with R22 on the VBUS rail; ERC 0, check_nets 453/453.
- Board: R22 inserted into the routed layout at (141.45, 59.6) beside the
  F.Cu VBUS run, VBUS stub + GND via; placement.py carries it for LAYOUT=1.
  KiCad DRC (all severities, schematic parity): 0 / 0 / 0.
- Exports regenerated (BOM/CPL 105 rows, gerbers, PDF, SVGs, renders);
  README power section and design review (post-layout change) updated.

Co-Authored-By: Claude Opus 5.5 <noreply@anthropic.com>
Parts:
- added R22: 4.7k, FujiNet-NES:R_0603_1608Metric, symbol Device:R
Connections:
- net GND: now also R22.2
- net VBUS: now also R22.1
Changed lines of the file:
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@@
+	)
+	(symbol
+		(lib_id "Device:R")
+		(at 121.92 135.89 0)
+		(unit 1)
+		(exclude_from_sim no)
+		(in_bom yes)
+		(on_board yes)
+		(dnp no)
+		(property "Reference" "R22"
+			(at 124.206 134.62 0)
+			(effects
+				(font
+					(size 1.27 1.27)
+				)
+				(justify left)
+			)
+		)
+		(property "Value" "4.7k"
+			(at 124.206 137.16 0)
+			(effects
+				(font
+					(size 1.27 1.27)
+				)
+				(justify left)
+			)
+		)
+		(property "Footprint" "FujiNet-NES:R_0603_1608Metric"
+			(at 121.92 135.89 0)
+			(effects
+				(font
+					(size 1.27 1.27)
+				)
+				(hide yes)
+			)
+		)
+		(property "Datasheet" ""
+			(at 121.92 135.89 0)
+			(effects
+				(font
+					(size 1.27 1.27)
+				)
+				(hide yes)
+			)
+		)
+		(property "Description" "P-FET gate pull-down against the SS34 reverse leakage"
+			(at 121.92 135.89 0)
+			(effects
+				(font
+					(size 1.27 1.27)
+				)
+				(hide yes)
+			)
+		)
+		(property "MPN" "0603WAF4701T5E"
+			(at 121.92 135.89 0)
+			(effects
+				(font
+					(size 1.27 1.27)
+				)
+				(hide yes)
+			)
+		)
+		(property "LCSC" "C23162"
+			(at 121.92 135.89 0)
+			(effects
+				(font
+					(size 1.27 1.27)
+				)
+				(hide yes)
+			)
+		)
+		(pin "1"
+		)
+		(pin "2"
+		)
+		(instances
+			(project "FujiNet-NES-Rev0"
+				(path "/5810f54f-2240-53c0-bbad-5b0b7a2c3f6b/d44cc47e-bd9a-52ed-901d-413852c5812b"
+					(reference "R22")
+					(unit 1)
+				)
+			)
+		)
 	)
 	(symbol
@@
 	)
 	(symbol
+		(lib_id "power:GND")
+		(at 121.92 139.7 0)
+		(unit 1)
+		(exclude_from_sim no)
+		(in_bom no)
+		(on_board no)
+		(dnp no)
+		(property "Reference" "#PWR121"
+			(at 121.92 146.05 0)
+			(effects
+				(font
+					(size 1.27 1.27)
+				)
+				(hide yes)
+			)
+		)
+		(property "Value" "GND"
+			(at 121.92 143.51 0)
+			(effects
+				(font
+					(size 1.27 1.27)
+				)
+			)
+		)
+		(property "Footprint" ""
+			(at 121.92 139.7 0)
+			(effects
+				(font
+					(size 1.27 1.27)
+				)
+				(hide yes)
+			)
+		)
+		(property "Datasheet" ""
+			(at 121.92 139.7 0)
+			(effects
+				(font
+					(size 1.27 1.27)
+				)
+				(hide yes)
+			)
+		)
+		(property "Description" ""
+			(at 121.92 139.7 0)
+			(effects
+				(font
+					(size 1.27 1.27)
+				)
+				(hide yes)
+			)
+		)
+		(pin "1"
+		)
+		(instances
+			(project "FujiNet-NES-Rev0"
+				(path "/5810f54f-2240-53c0-bbad-5b0b7a2c3f6b/d44cc47e-bd9a-52ed-901d-413852c5812b"
+					(reference "#PWR121")
+					(unit 1)
+				)
+			)
+		)
+	)
+	(symbol
 		(lib_id "power:+5V")
 		(at 172.72 104.14 0)
@@
 		(on_board no)
 		(dnp no)
-		(property "Reference" "#PWR121"
+		(property "Reference" "#PWR122"
 			(at 172.72 97.79 0)
 			(effects
@@
 			(project "FujiNet-NES-Rev0"
 				(path "/5810f54f-2240-53c0-bbad-5b0b7a2c3f6b/d44cc47e-bd9a-52ed-901d-413852c5812b"
-					(reference "#PWR121")
+					(reference "#PWR122")
 					(unit 1)
 				)
@@
 		(on_board no)
 		(dnp no)
-		(property "Reference" "#PWR122"
+		(property "Reference" "#PWR123"
 			(at 182.88 118.11 0)
 			(effects
@@
 			(project "FujiNet-NES-Rev0"
 				(path "/5810f54f-2240-53c0-bbad-5b0b7a2c3f6b/d44cc47e-bd9a-52ed-901d-413852c5812b"
-					(reference "#PWR122")
+					(reference "#PWR123")
 					(unit 1)
 				)
@@
 		(on_board no)
 		(dnp no)
-		(property "Reference" "#PWR123"
+		(property "Reference" "#PWR124"
 			(at 193.04 118.11 0)
 			(effects
@@
 			(project "FujiNet-NES-Rev0"
 				(path "/5810f54f-2240-53c0-bbad-5b0b7a2c3f6b/d44cc47e-bd9a-52ed-901d-413852c5812b"
-					(reference "#PWR123")
+					(reference "#PWR124")
 					(unit 1)
 				)
@@
 		(on_board no)
 		(dnp no)
-		(property "Reference" "#PWR124"
+		(property "Reference" "#PWR125"
 			(at 203.2 118.11 0)
 			(effects
@@
 			(project "FujiNet-NES-Rev0"
 				(path "/5810f54f-2240-53c0-bbad-5b0b7a2c3f6b/d44cc47e-bd9a-52ed-901d-413852c5812b"
-					(reference "#PWR124")
+					(reference "#PWR125")
 					(unit 1)
 				)
@@
 		(on_board no)
 		(dnp no)
-		(property "Reference" "#PWR125"
+		(property "Reference" "#PWR126"
 			(at 213.36 118.11 0)
 			(effects
@@
 			(project "FujiNet-NES-Rev0"
 				(path "/5810f54f-2240-53c0-bbad-5b0b7a2c3f6b/d44cc47e-bd9a-52ed-901d-413852c5812b"
-					(reference "#PWR125")
+					(reference "#PWR126")
 					(unit 1)
 				)
@@
 		(on_board no)
 		(dnp no)
-		(property "Reference" "#PWR126"
+		(property "Reference" "#PWR127"
 			(at 246.38 120.65 0)
 			(effects
@@
 			(project "FujiNet-NES-Rev0"
 				(path "/5810f54f-2240-53c0-bbad-5b0b7a2c3f6b/d44cc47e-bd9a-52ed-901d-413852c5812b"
-					(reference "#PWR126")
+					(reference "#PWR127")
 					(unit 1)
 				)
@@
 		(on_board no)
 		(dnp no)
-		(property "Reference" "#PWR127"
+		(property "Reference" "#PWR128"
 			(at 288.29 97.79 0)
 			(effects
@@
 			(project "FujiNet-NES-Rev0"
 				(path "/5810f54f-2240-53c0-bbad-5b0b7a2c3f6b/d44cc47e-bd9a-52ed-901d-413852c5812b"
-					(reference "#PWR127")
+					(reference "#PWR128")
 					(unit 1)
 				)
@@
 		(on_board no)
 		(dnp no)
-		(property "Reference" "#PWR128"
+		(property "Reference" "#PWR129"
 			(at 293.37 118.11 0)
 			(effects
@@
 			(project "FujiNet-NES-Rev0"
 				(path "/5810f54f-2240-53c0-bbad-5b0b7a2c3f6b/d44cc47e-bd9a-52ed-901d-413852c5812b"
-					(reference "#PWR128")
+					(reference "#PWR129")
 					(unit 1)
 				)
@@
 		(on_board no)
 		(dnp no)
-		(property "Reference" "#PWR129"
+		(property "Reference" "#PWR130"
 			(at 303.53 118.11 0)
 			(effects
@@
 			(project "FujiNet-NES-Rev0"
 				(path "/5810f54f-2240-53c0-bbad-5b0b7a2c3f6b/d44cc47e-bd9a-52ed-901d-413852c5812b"
-					(reference "#PWR129")
+					(reference "#PWR130")
 					(unit 1)
 				)
@@
 		(on_board no)
 		(dnp no)
-		(property "Reference" "#PWR130"
+		(property "Reference" "#PWR131"
 			(at 223.52 168.91 0)
 			(effects
@@
 			(project "FujiNet-NES-Rev0"
 				(path "/5810f54f-2240-53c0-bbad-5b0b7a2c3f6b/d44cc47e-bd9a-52ed-901d-413852c5812b"
-					(reference "#PWR130")
+					(reference "#PWR131")
 					(unit 1)
 				)
@@
 		(on_board no)
 		(dnp no)
-		(property "Reference" "#PWR131"
+		(property "Reference" "#PWR132"
 			(at 238.76 171.45 0)
 			(effects
@@
 			(project "FujiNet-NES-Rev0"
 				(path "/5810f54f-2240-53c0-bbad-5b0b7a2c3f6b/d44cc47e-bd9a-52ed-901d-413852c5812b"
-					(reference "#PWR131")
+					(reference "#PWR132")
 					(unit 1)
 				)
@@
 		(on_board no)
 		(dnp no)
-		(property "Reference" "#PWR132"
+		(property "Reference" "#PWR133"
 			(at 254 168.91 0)
 			(effects
@@
 			(project "FujiNet-NES-Rev0"
 				(path "/5810f54f-2240-53c0-bbad-5b0b7a2c3f6b/d44cc47e-bd9a-52ed-901d-413852c5812b"
-					(reference "#PWR132")
+					(reference "#PWR133")
 					(unit 1)
 				)
@@
 		(on_board no)
 		(dnp no)
-		(property "Reference" "#PWR133"
+		(property "Reference" "#PWR134"
 			(at 259.08 148.59 0)
 			(effects
@@
 			(project "FujiNet-NES-Rev0"
 				(path "/5810f54f-2240-53c0-bbad-5b0b7a2c3f6b/d44cc47e-bd9a-52ed-901d-413852c5812b"
-					(reference "#PWR133")
+					(reference "#PWR134")
 					(unit 1)
 				)
@@
 		(pts
 			(xy 111.76 132.08)
+			(xy 121.92 132.08)
+		)
+		(stroke
+			(width 0)
+			(type default)
+		)
+	)
+	(wire
+		(pts
+			(xy 121.92 132.08)
 			(xy 132.08 132.08)
 		)
@@
 	)
 	(junction
+		(at 121.92 132.08)
+		(diameter 0)
+		(color 0 0 0 0)
+	)
+	(junction
