File: NES/FujiNet-NES-Rev0/usb-uart.kicad_sch (KiCad schematic)
At the start: 15 parts, among them J3 USB-C, U12 CP2102N-A02-GQFN28, U13 UMH3N

Commit message: [nes] redo schematic1
Other:
- title: FujiNet NES Rev0 - USB-C, CP2102N programming bridge -> FujiNet NES Rev0 - USB-C, CP2102N bridge
- moved on the sheet: C37, C38, C39, C40, D4, D5, D6, J3, R17, R18, R19, R20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
