File: NES/FujiNet-NES-Rev0/FujiNet-NES-Rev0.kicad_pcb (KiCad board)
At the start: 6 copper layers, 100 x 110 mm, 117 parts, among them J1 NES_Cart_Edge_72, J2 microSD, J3 USB-C, Q1 AO3401A, SW1 RESET, SW2 BOOTSEL, SW3 S3_RST, SW4 S3_BOOT, U1 RP2354B, U10 ATtiny13A-SSU, U11 ESP32-S3-WROOM-1-N16R8, U12 CP2102N-A02-GQFN28, U13 UMH3N, U14 AP63203WU, U15 AP2112K-3.3, U2 AS6C4008-55TIN, U3 AS6C4008-55TIN, U4 74HCT595, U5 74HCT253, U6 74HCT14, U7 74HCT20, U8 74HCT00, U9 74HCT32, Y1 12MHz

Commit message: fix rp2354 footprint. DRC.
Routing:
- net unconnected-(J1-SYSTEM_CLK-Pad37): track 2.70 -> 0.00 mm
- net unconnected-(J1-EXP9-Pad51): track 2.70 -> 0.00 mm
- net unconnected-(J1-EXP8-Pad52): track 2.70 -> 0.00 mm
- net unconnected-(J1-EXP7-Pad53): track 2.70 -> 0.00 mm
- net unconnected-(J1-EXP6-Pad54): track 2.70 -> 0.00 mm
- net unconnected-(J1-EXP5-Pad55): track 2.70 -> 0.00 mm
- net unconnected-(J1-EXP4-Pad20): track 2.70 -> 0.00 mm
- net unconnected-(J1-EXP3-Pad19): track 2.70 -> 0.00 mm
- net unconnected-(J1-EXP2-Pad18): track 2.70 -> 0.00 mm
- net unconnected-(J1-EXP1-Pad17): track 2.70 -> 0.00 mm
- net unconnected-(J1-EXP0-Pad16): track 2.70 -> 0.00 mm
Changed lines of the file:
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@@
 		(tags "capacitor")
 		(property "Reference" "C18"
-			(at 0 -1.43 0)
+			(at -0.8 1.5836 0)
 			(layer "F.SilkS")
 			(effects
@@
 			)
 		)
-		(property "Datasheet" "http://www.ti.com/lit/gpn/sn74LS253"
+		(property "Datasheet" "https://www.ti.com/lit/gpn/sn74hct253"
 			(at 0 0 0)
 			(layer "F.Fab")
@@
 		(tags "resistor")
 		(property "Reference" "R1"
-			(at 0 -1.43 0)
+			(at 0 1.5836 0)
 			(layer "F.SilkS")
 			(effects
@@
 			(at 0 -1.43 180)
 			(layer "F.SilkS")
+			(hide yes)
 			(effects
 				(font
@@
 		(tags "capacitor")
 		(property "Reference" "C15"
-			(at 0 -1.43 180)
+			(at 0 1.5836 0)
 			(layer "F.SilkS")
 			(effects
@@
 		(tags "LED")
 		(property "Reference" "D2"
-			(at 0 -1.43 0)
+			(at 0.38 1.6236 0)
 			(layer "F.SilkS")
 			(effects
@@
 		(tags "resistor array")
 		(property "Reference" "RN1"
-			(at 0 -2.8 90)
+			(at 2.4036 0 0)
 			(layer "F.SilkS")
 			(effects
@@
 		(tags "capacitor")
 		(property "Reference" "C7"
-			(at 0 -1.43 90)
+			(at -2.3336 -0.4 0)
 			(layer "F.SilkS")
 			(effects
@@
 		(tags "capacitor")
 		(property "Reference" "C10"
-			(at 0 -1.43 180)
+			(at -2.3336 0 90)
 			(layer "F.SilkS")
 			(effects
@@
 		(tags "capacitor")
 		(property "Reference" "C14"
-			(at 0 -1.43 180)
+			(at 0 1.5836 0)
 			(layer "F.SilkS")
 			(effects
@@
 		(tags "resistor")
 		(property "Reference" "R20"
-			(at 0 -1.43 0)
+			(at 0 1.5836 0)
 			(layer "F.SilkS")
 			(effects
@@
 			(at 0 -1.43 0)
 			(layer "F.SilkS")
+			(hide yes)
 			(effects
 				(font
@@
 		(tags "capacitor")
 		(property "Reference" "C24"
-			(at 0 -1.43 0)
+			(at -2.3336 0 90)
 			(layer "F.SilkS")
 			(effects
@@
 		(tags "capacitor")
 		(property "Reference" "C31"
-			(at 0 -1.43 90)
+			(at 0 1.5836 90)
 			(layer "F.SilkS")
 			(effects
@@
 			(at 0 -1.43 0)
 			(layer "F.SilkS")
+			(hide yes)
 			(effects
 				(font
@@
 		(tags "capacitor")
 		(property "Reference" "C26"
-			(at 0 -1.43 90)
+			(at 0 1.5836 90)
 			(layer "F.SilkS")
 			(effects
@@
 		(tags "resistor array")
 		(property "Reference" "RN2"
-			(at 0 -2.8 90)
+			(at -2.4036 0 0)
 			(layer "F.SilkS")
 			(effects
@@
 		(tags "resistor")
 		(property "Reference" "R4"
-			(at 0 -1.43 180)
+			(at -2.535952 -0.4 0)
 			(layer "F.SilkS")
 			(effects
@@
 			(at 0 -1.43 180)
 			(layer "F.SilkS")
+			(hide yes)
 			(effects
 				(font
@@
 		(tags "capacitor")
 		(property "Reference" "C11"
-			(at 0 -1.43 90)
+			(at -2.3336 0 0)
 			(layer "F.SilkS")
 			(effects
@@
 		)
 		(embedded_fonts no)
-		(model "${KIPRJMOD}/3d/QFN-80-1EP_10x10mm_P0.4mm_EP3.4x3.4mm.step"
+		(model "${KIPRJMOD}/3d/RP2354B_QFN-80_10x10.step"
 			(offset
 				(xyz 0 0 0)
@@
 			(layers "F.Cu" "F.Mask")
 			(solder_mask_margin 0.5)
+			(clearance 0.5)
 		)
 		(embedded_fonts no)
@@
 		(tags "capacitor")
 		(property "Reference" "C9"
-			(at 0 -1.43 180)
+			(at -2.535952 -0.4 0)
 			(layer "F.SilkS")
 			(effects
@@
 		(tags "resistor")
 		(property "Reference" "R5"
-			(at 0 -1.43 180)
+			(at 2.535952 0 0)
 			(layer "F.SilkS")
 			(effects
@@
 			(at 0 -1.43 180)
 			(layer "F.SilkS")
+			(hide yes)
 			(effects
 				(font
@@
 		(tags "capacitor")
 		(property "Reference" "C38"
-			(at 0 -1.43 90)
+			(at 0 1.5836 90)
 			(layer "F.SilkS")
 			(effects
@@
 		(tags "SOT-23-5")
 		(property "Reference" "U15"
-			(at 0 -2.65 0)
+			(at 0 2.5536 0)
 			(layer "F.SilkS")
 			(effects
@@
 			(at 0 -1.43 0)
 			(layer "F.SilkS")
+			(hide yes)
 			(effects
 				(font
@@
 		(sheetname "/edge-cic/")
 		(sheetfile "edge-cic.kicad_sch")
-		(attr smd exclude_from_pos_files exclude_from_bom)
+		(attr smd exclude_from_pos_files exclude_from_bom allow_soldermask_bridges)
 		(duplicate_pad_numbers_are_jumpers no)
 		(fp_rect
@@
 		(tags "capacitor")
 		(property "Reference" "C16"
-			(at 0 -1.43 180)
+			(at 0.4 1.5836 0)
 			(layer "F.SilkS")
 			(effects
@@
 			(at 0 -1.43 180)
 			(layer "F.SilkS")
+			(hide yes)
 			(effects
 				(font
@@
 		(tags "capacitor")
 		(property "Reference" "C44"
-			(at 0 -1.68 90)
+			(at 0 1.8336 90)
 			(layer "F.SilkS")
 			(effects
@@
 		(tags "SPST Tactile Switch")
 		(property "Reference" "SW1"
-			(at 0 -3.75 0)
+			(at 0 4.02325 0)
 			(layer "F.SilkS")
 			(effects
@@
 		(tags "capacitor")
 		(property "Reference" "C30"
-			(at 0 -1.43 90)
+			(at 0 1.5836 90)
 			(layer "F.SilkS")
 			(effects
@@
 		(descr "From Raspberry Pi RP2350A minimal design (MIT): RPI_COMPILED:abracon_aota-b201610s3r3-101-t")
 		(property "Reference" "L1"
-			(at 0 -1.55 0)
+			(at -0.625 1.742375 0)
 			(unlocked yes)
 			(layer "F.SilkS")
@@
 			(layers "F.Cu" "F.Mask")
 			(solder_mask_margin 0.5)
+			(clearance 0.5)
 		)
 		(embedded_fonts no)
@@
 			(layers "F.Cu" "F.Mask")
 			(solder_mask_margin 0.5)
+			(clearance 0.5)
 		)
 		(embedded_fonts no)
@@
 		(tags "capacitor")
 		(property "Reference" "C4"
-			(at 0 -1.43 0)
+			(at 0 1.5836 0)
 			(layer "F.SilkS")
 			(effects
@@
 		(tags "capacitor")
 		(property "Reference" "C13"
-			(at 0 -1.43 180)
+			(at 2.3336 0 90)
 			(layer "F.SilkS")
 			(effects
@@
 		(tags "resistor")
 		(property "Reference" "R3"
-			(at 0 -1.43 0)
+			(at 0.4 1.5836 0)
 			(layer "F.SilkS")
 			(effects
@@
 	)
 	(gr_text "label side: pin 1 ->"
-		(at 106 88 0)
+		(at 106 87.75 0)
 		(layer "F.SilkS")
 		(effects
@@
 	)
 	(segment
-		(start 106.25 127.2)
-		(end 106.25 124.5)
-		(width 0.3)
-		(locked yes)
-		(layer "F.Cu")
-		(net "unconnected-(J1-EXP0-Pad16)")
-	)
-	(segment
-		(start 103.75 127.2)
-		(end 103.75 124.5)
-		(width 0.3)
-		(locked yes)
-		(layer "F.Cu")
-		(net "unconnected-(J1-EXP1-Pad17)")
-	)
-	(segment
-		(start 101.25 127.2)
-		(end 101.25 124.5)
-		(width 0.3)
-		(locked yes)
-		(layer "F.Cu")
-		(net "unconnected-(J1-EXP2-Pad18)")
-	)
-	(segment
-		(start 98.75 127.2)
-		(end 98.75 124.5)
-		(width 0.3)
-		(locked yes)
-		(layer "F.Cu")
-		(net "unconnected-(J1-EXP3-Pad19)")
-	)
-	(segment
-		(start 96.25 127.2)
-		(end 96.25 124.5)
-		(width 0.3)
-		(locked yes)
-		(layer "F.Cu")
-		(net "unconnected-(J1-EXP4-Pad20)")
-	)
-	(segment
 		(start 93.75 127.2)
 		(end 93.75 124.5)
@@
 	)
 	(segment
-		(start 144.25 127.2)
-		(end 144.25 124.5)
-		(width 0.3)
-		(locked yes)
-		(layer "B.Cu")
-		(net "unconnected-(J1-SYSTEM_CLK-Pad37)")
-	)
-	(segment
-		(start 108.75 127.2)
-		(end 108.75 124.5)
-		(width 0.3)
-		(locked yes)
-		(layer "B.Cu")
-		(net "unconnected-(J1-EXP9-Pad51)")
-	)
-	(segment
-		(start 106.25 127.2)
-		(end 106.25 124.5)
-		(width 0.3)
-		(locked yes)
-		(layer "B.Cu")
-		(net "unconnected-(J1-EXP8-Pad52)")
-	)
-	(segment
-		(start 103.75 127.2)
-		(end 103.75 124.5)
-		(width 0.3)
-		(locked yes)
-		(layer "B.Cu")
-		(net "unconnected-(J1-EXP7-Pad53)")
-	)
-	(segment
-		(start 101.25 127.2)
-		(end 101.25 124.5)
-		(width 0.3)
-		(locked yes)
-		(layer "B.Cu")
-		(net "unconnected-(J1-EXP6-Pad54)")
-	)
-	(segment
-		(start 98.75 127.2)
-		(end 98.75 124.5)
-		(width 0.3)
-		(locked yes)
-		(layer "B.Cu")
-		(net "unconnected-(J1-EXP5-Pad55)")
-	)
-	(segment
