File: NES/FujiNet-NES-Rev0/FujiNet-NES-Rev0.kicad_pcb (KiCad board)
At the start: 6 copper layers, 100 x 110 mm, 117 parts, among them J1 NES_Cart_Edge_72, J2 microSD, J3 USB-C, Q1 AO3401A, SW1 RESET, SW2 BOOTSEL, SW3 S3_RST, SW4 S3_BOOT, U1 RP2354B, U10 ATtiny13A-SSU, U11 ESP32-S3-WROOM-1-N16R8, U12 CP2102N-A02-GQFN28, U13 UMH3N, U14 AP63203WU, U15 AP2112K-3.3, U2 AS6C4008-55TIN, U3 AS6C4008-55TIN, U4 74HCT595, U5 74HCT253, U6 74HCT14, U7 74HCT20, U8 74HCT00, U9 74HCT32, Y1 12MHz

Commit message: NES Rev0: add the VBUS pull-down (R22 4.7k) against SS34 reverse leakage
Q1's gate is VBUS, which only the 69k CP2102N sense divider pulled down.
With the console powering the cart the SS34 is reverse-biased and leaks
into VBUS (0.5 mA max at 25 C); at >= 100 uA the AO3401A turns off and the
console feeds +5V through the body diode, ~0.7 V down, under the 74HCT /
SRAM 4.5 V minimum.  R22 4.7k VBUS-GND (0603WAF4701T5E, C23162) holds VGS
beyond -2.8 V up to 500 uA; same fix as 2600 Rev1 R_VBPD and SMS Rev0.

- design.py: R22 declared after every other resistor (no ref changes).
- power sheet redrawn with R22 on the VBUS rail; ERC 0, check_nets 453/453.
- Board: R22 inserted into the routed layout at (141.45, 59.6) beside the
  F.Cu VBUS run, VBUS stub + GND via; placement.py carries it for LAYOUT=1.
  KiCad DRC (all severities, schematic parity): 0 / 0 / 0.
- Exports regenerated (BOM/CPL 105 rows, gerbers, PDF, SVGs, renders);
  README power section and design review (post-layout change) updated.

Co-Authored-By: Claude Opus 5.5 <noreply@anthropic.com>
Parts:
- added R22: 4.7k, FujiNet-NES:R_0603_1608Metric, F.Cu at (141.4, 59.6)
Routing:
- net GND: track 131.1 -> 132.4 mm, vias 346 -> 347
- net VBUS: track 196.1 -> 197.2 mm
Changed lines of the file:
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@@
 		)
 	)
+	(footprint "FujiNet-NES:R_0603_1608Metric"
+		(layer "F.Cu")
+		(at 141.45 59.6)
+		(descr "Resistor SMD 0603 (1608 Metric), square (rectangular) end terminal, IPC-7351 nominal, (Body size source: IPC-SM-782 page 72, https://www.pcb-3d.com/wordpress/wp-content/uploads/ipc-sm-782a_amendment_1_and_2.pdf)")
+		(tags "resistor")
+		(property "Reference" "R22"
+			(at 0 1.5836 0)
+			(layer "F.SilkS")
+			(effects
+				(font
+					(size 0.8 0.8)
+					(thickness 0.12)
+				)
+			)
+		)
+		(property "Value" "4.7k"
+			(at 0 1.43 0)
+			(layer "F.Fab")
+			(effects
+				(font
+					(size 1 1)
+					(thickness 0.15)
+				)
+			)
+		)
+		(property "Datasheet" ""
+			(at 0 0 0)
+			(layer "F.Fab")
+			(hide yes)
+			(effects
+				(font
+					(size 1.27 1.27)
+					(thickness 0.15)
+				)
+			)
+		)
+		(property "Description" "P-FET gate pull-down against the SS34 reverse leakage"
+			(at 0 0 0)
+			(layer "F.Fab")
+			(hide yes)
+			(effects
+				(font
+					(size 1.27 1.27)
+					(thickness 0.15)
+				)
+			)
+		)
+		(property "MPN" "0603WAF4701T5E"
+			(at 0 0 0)
+			(layer "F.Fab")
+			(hide yes)
+			(effects
+				(font
+					(size 1.27 1.27)
+					(thickness 0.15)
+				)
+			)
+		)
+		(property "LCSC" "C23162"
+			(at 0 0 0)
+			(layer "F.Fab")
+			(hide yes)
+			(effects
+				(font
+					(size 1.27 1.27)
+					(thickness 0.15)
+				)
+			)
+		)
+		(sheetname "/power/")
+		(sheetfile "power.kicad_sch")
+		(attr smd)
+		(duplicate_pad_numbers_are_jumpers no)
+		(fp_line
+			(start -0.237258 -0.5225)
+			(end 0.237258 -0.5225)
+			(stroke
+				(width 0.12)
+				(type solid)
+			)
+			(layer "F.SilkS")
+		)
+		(fp_line
+			(start -0.237258 0.5225)
+			(end 0.237258 0.5225)
+			(stroke
+				(width 0.12)
+				(type solid)
+			)
+			(layer "F.SilkS")
+		)
+		(fp_rect
+			(start -1.48 -0.73)
+			(end 1.48 0.73)
+			(stroke
+				(width 0.05)
+				(type solid)
+			)
+			(fill no)
+			(layer "F.CrtYd")
+		)
+		(fp_rect
+			(start -0.8 -0.4125)
+			(end 0.8 0.4125)
+			(stroke
+				(width 0.1)
+				(type solid)
+			)
+			(fill no)
+			(layer "F.Fab")
+		)
+		(fp_text user "${REFERENCE}"
+			(at 0 0 0)
+			(layer "F.Fab")
+			(effects
+				(font
+					(size 0.4 0.4)
+					(thickness 0.06)
+				)
+			)
+		)
+		(pad "1" smd roundrect
+			(at -0.825 0)
+			(size 0.8 0.95)
+			(layers "F.Cu" "F.Mask" "F.Paste")
+			(roundrect_rratio 0.25)
+			(net "VBUS")
+		)
+		(pad "2" smd roundrect
+			(at 0.825 0)
+			(size 0.8 0.95)
+			(layers "F.Cu" "F.Mask" "F.Paste")
+			(roundrect_rratio 0.25)
+			(net "GND")
+		)
+		(embedded_fonts no)
+		(model "${KIPRJMOD}/3d/R_0603_1608Metric.step"
+			(offset
+				(xyz 0 0 0)
+			)
+			(scale
+				(xyz 1 1 1)
+			)
+			(rotate
+				(xyz 0 0 0)
+			)
+		)
+	)
 	(footprint "FujiNet-NES:C_0603_1608Metric"
 		(layer "F.Cu")
@@
 		(tags "capacitor")
 		(property "Reference" "C45"
-			(at 0 -1.43 90)
+			(at 0 1.5836 90)
 			(layer "F.SilkS")
 			(effects
@@
 	)
 	(segment
+		(start 142.275 59.6)
+		(end 142.275 60.85)
+		(width 0.3)
+		(locked yes)
+		(layer "F.Cu")
+		(net "GND")
+	)
+	(segment
 		(start 100.625 102.8)
 		(end 99.725 102.8)
@@
 	)
 	(via
+		(at 142.275 60.85)
+		(size 0.6)
+		(drill 0.3)
+		(layers "F.Cu" "B.Cu")
+		(locked yes)
+		(net "GND")
+	)
+	(via
 		(at 95.2 33.2)
 		(size 0.6)
@@
 		(layer "F.Cu")
 		(net "VBUS")
+	)
+	(segment
+		(start 140.625 59.6)
+		(end 139.5831 59.6)
+		(width 0.3)
+		(locked yes)
+		(layer "F.Cu")
+		(net "VBUS")

Commit message: NES Rev0: fix the microSD / USB-C alignment (J3 to the board edge, 3D models)
A reviewer reported J2 (microSD) and J3 (USB-C) as misaligned. Checked
against the SOFNG TF-015 and HRO TYPE-C-31-M-12 drawings, the STEP
vertices and a zoomed render:

- J3 sat 1.35 mm inside the top edge. HRO's recommended layout puts the
  PCB edge 5.79 mm in front of the pegs (fp y +3.19), so the face
  overhangs it by 0.46 mm; set back, a plug's overmold meets the board
  edge before the plug mates. J3 moves (125, 35) -> (125, 33.2). Its
  VBUS / D- ties between the pad row and the pegs move with it, nine
  1.8 mm F.Cu stubs join the new pad centres to the untouched routing,
  and one edge-row GND stitching via under the new front shield slot is
  removed. The front silk (now past the edge) is dropped; a Dwgs.User
  line marks HRO's edge.
- J3's 3D model was 2.47 mm behind its footprint: KiCad applies the
  offset after the rotation and the LCSC model's origin is the front
  shield legs -> offset (0, -1.045, 0), not (0, +1.42, 0).
- J2's 3D model was 5.5 mm behind and 0.9 mm beside its footprint
  (make_tf015_fp.py dropped easyeda2kicad's offset; the model's origin
  is the card centre on the peg line) -> offset (-0.9, -5.5, 0).

Unchanged after checking: J2's copper (SOFNG land pattern within
0.1 mm), J2's card face 0.5 mm inside the edge (a latched card stands
2.5 mm proud, ~2 mm past the edge), J3's KiCad-stock copper.

Every model feature (pegs, shield legs, tails, feet) now lands within
0.02 mm of its pad or hole. KiCad DRC at every severity with schematic
parity: 0 / 0 / 0. placement.py, set_models.py, make_tf015_fp.py and
both library footprints carry the fix for a LAYOUT=1 rebuild. Exports
regenerated: CPL changes J3's Y only; drill changes are J3's slots and
pegs plus the removed via. Design review: "Post-layout change
(2026-10-11)".

Co-Authored-By: Claude Opus 5.5 <noreply@anthropic.com>
Parts:
- moved J3 1.80 mm to (125.0, 33.2)
Routing:
- net GND: track 132.4 -> 136.0 mm, vias 347 -> 346
- net VBUS: track 197.2 -> 200.8 mm
- net UBRG_DP: track 14.7 -> 18.3 mm
- net CC2: track 12.7 -> 14.5 mm
- net CC1: track 11.3 -> 13.1 mm
- net UBRG_DM: track 13.8 -> 15.6 mm
Changed lines of the file:
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@@
 		(model "${KIPRJMOD}/3d/TF-015.step"
 			(offset
-				(xyz 0 0 0)
+				(xyz -0.9 -5.5 0)
 			)
 			(scale
@@
 	(footprint "FujiNet-NES:USB_C_Receptacle_HRO_TYPE-C-31-M-12"
 		(layer "F.Cu")
-		(at 125 35 180)
-		(descr "USB Type-C receptacle for USB 2.0 and PD, http://www.krhro.com/uploads/soft/180320/1-1P320120243.pdf")
+		(at 125 33.2 180)
+		(descr "USB Type-C receptacle for USB 2.0 and PD, http://www.krhro.com/uploads/soft/180320/1-1P320120243.pdf; PCB edge at y 3.19 (HRO recommended layout: 5.79 mm in front of the pegs), the shell face overhangs it by 0.46 mm")
 		(tags "usb usb-c 2.0 pd")
 		(property "Reference" "J3"
@@
 		(duplicate_pad_numbers_are_jumpers no)
 		(fp_line
-			(start 4.7 2)
-			(end 4.7 3.9)
-			(stroke
-				(width 0.12)
-				(type solid)
-			)
-			(layer "F.SilkS")
-		)
-		(fp_line
 			(start 4.7 -1.9)
 			(end 4.7 0.1)
@@
 		)
 		(fp_line
-			(start -4.7 3.9)
-			(end 4.7 3.9)
-			(stroke
-				(width 0.12)
-				(type solid)
-			)
-			(layer "F.SilkS")
-		)
-		(fp_line
-			(start -4.7 2)
-			(end -4.7 3.9)
+			(start -4.7 -1.9)
+			(end -4.7 0.1)
 			(stroke
 				(width 0.12)
@@
 		)
 		(fp_line
-			(start -4.7 -1.9)
-			(end -4.7 0.1)
+			(start -5.32 3.19)
+			(end 5.32 3.19)
 			(stroke
-				(width 0.12)
-				(type solid)
+				(width 0.1)
+				(type dash)
 			)
-			(layer "F.SilkS")
+			(layer "Dwgs.User")
 		)
 		(fp_line
@@
 		(model "${KIPRJMOD}/3d/USB-C_HRO_TYPE-C-31-M-12.step"
 			(offset
-				(xyz 0 1.42 0)
+				(xyz 0 -1.045 0)
 			)
 			(scale
@@
 	)
 	(segment
+		(start 121.75 37.245)
+		(end 121.75 39.045)
+		(width 0.3)
+		(layer "F.Cu")
+		(net "GND")
+	)
+	(segment
 		(start 99.425 95.2)
 		(end 98.525 95.2)
@@
 	)
 	(segment
+		(start 128.25 37.245)
+		(end 128.25 39.045)
+		(width 0.3)
+		(layer "F.Cu")
+		(net "GND")
+	)
+	(segment
 		(start 74.75 37.74)
 		(end 76.056 36.955)
@@
 	)
 	(via
-		(at 120.27 31.2)
-		(size 0.6)
-		(drill 0.3)
-		(layers "F.Cu" "B.Cu")
-		(locked yes)
-		(net "GND")
-	)
-	(via
 		(at 147.2 65.2)
 		(size 0.6)
@@
 	)
 	(segment
-		(start 123.4073 37.5861)
-		(end 122.55 38.4434)
+		(start 123.4073 35.7861)
+		(end 122.55 36.6434)
+		(width 0.3)
+		(layer "F.Cu")
+		(net "VBUS")
+	)
+	(segment
+		(start 122.55 37.245)
+		(end 122.55 39.045)
 		(width 0.3)
 		(layer "F.Cu")
@@
 	)
 	(segment
-		(start 127.45 39.045)
-		(end 127.45 38.4312)
+		(start 127.45 37.245)
+		(end 127.45 36.6312)
 		(width 0.3)
 		(layer "F.Cu")
@@
 	)
 	(segment
+		(start 127.45 37.245)
+		(end 127.45 39.045)
+		(width 0.3)
+		(layer "F.Cu")
+		(net "VBUS")
+	)
+	(segment
 		(start 140.625 59.6)
 		(end 139.5831 59.6)
@@
 	)
 	(segment
-		(start 126.6049 37.5861)
-		(end 123.4073 37.5861)
+		(start 126.6049 35.7861)
+		(end 123.4073 35.7861)
 		(width 0.3)
 		(layer "F.Cu")
@@
 	)
 	(segment
-		(start 122.55 38.4434)
-		(end 122.55 39.045)
+		(start 122.55 36.6434)
+		(end 122.55 37.245)
 		(width 0.3)
 		(layer "F.Cu")
@@
 	)
 	(segment
-		(start 127.45 38.4312)
-		(end 126.6049 37.5861)
+		(start 127.45 36.6312)
+		(end 126.6049 35.7861)
 		(width 0.3)
 		(layer "F.Cu")
@@
 	)
 	(segment
+		(start 124.25 37.245)
+		(end 124.25 39.045)
+		(width 0.25)
+		(layer "F.Cu")
+		(net "UBRG_DP")
+	)
+	(segment
+		(start 125.25 37.245)
+		(end 125.25 39.045)
+		(width 0.25)
+		(layer "F.Cu")
+		(net "UBRG_DP")
+	)
+	(segment
 		(start 125.25 39.8)
 		(end 125 40.05)
@@
 	)
 	(segment
-		(start 125.501 38.0419)
-		(end 125.75 38.2909)
+		(start 125.501 36.2419)
+		(end 125.75 36.4909)
 		(width 0.25)
 		(layer "F.Cu")
@@
 	)
 	(segment
-		(start 124.75 38.2951)
-		(end 125.0032 38.0419)
+		(start 124.75 36.4951)
+		(end 125.0032 36.2419)
+		(width 0.25)
+		(layer "F.Cu")
+		(net "UBRG_DM")
+	)
+	(segment
+		(start 125.75 37.245)
+		(end 125.75 39.045)
 		(width 0.25)
 		(layer "F.Cu")
@@
 	)
 	(segment
-		(start 125.75 38.2909)
-		(end 125.75 39.045)
+		(start 125.75 36.4909)
+		(end 125.75 37.245)
 		(width 0.25)
 		(layer "F.Cu")
@@
 	)
 	(segment
-		(start 125.0032 38.0419)
-		(end 125.501 38.0419)
+		(start 125.0032 36.2419)
+		(end 125.501 36.2419)
 		(width 0.25)
 		(layer "F.Cu")
@@
 	)
 	(segment
-		(start 124.75 39.045)
-		(end 124.75 38.2951)
+		(start 124.75 37.245)
+		(end 124.75 36.4951)
 		(width 0.25)
 		(layer "F.Cu")
@@
 	)
 	(segment
+		(start 123.25 37.245)
+		(end 123.25 39.045)
+		(width 0.2)
+		(layer "F.Cu")
+		(net "CC2")
+	)
+	(segment
 		(start 132.1456 38.4706)
 		(end 132 38.325)
@@
 		(width 0.2)
 		(layer "F.Cu")
+		(net "CC1")
+	)
+	(segment
+		(start 126.25 37.245)
+		(end 126.25 39.045)
+		(width 0.2)
+		(layer "F.Cu")
