File: NES/FujiNet-NES-Rev0/FujiNet-NES-Rev0.kicad_pcb (KiCad board)
At the start: 6 copper layers, 100 x 110 mm, 117 parts, among them J1 NES_Cart_Edge_72, J2 microSD, J3 USB-C, Q1 AO3401A, SW1 RESET, SW2 BOOTSEL, SW3 S3_RST, SW4 S3_BOOT, U1 RP2354B, U10 ATtiny13A-SSU, U11 ESP32-S3-WROOM-1-N16R8, U12 CP2102N-A02-GQFN28, U13 UMH3N, U14 AP63203WU, U15 AP2112K-3.3, U2 AS6C4008-55TIN, U3 AS6C4008-55TIN, U4 74HCT595, U5 74HCT253, U6 74HCT14, U7 74HCT20, U8 74HCT00, U9 74HCT32, Y1 12MHz

Commit message: Fix the microSD / USB-C alignment on every cart (USB-C to HRO's board edge, 3D models) (#61)
* NES Rev0: add the VBUS pull-down (R22 4.7k) against SS34 reverse leakage

Q1's gate is VBUS, which only the 69k CP2102N sense divider pulled down.
With the console powering the cart the SS34 is reverse-biased and leaks
into VBUS (0.5 mA max at 25 C); at >= 100 uA the AO3401A turns off and the
console feeds +5V through the body diode, ~0.7 V down, under the 74HCT /
SRAM 4.5 V minimum.  R22 4.7k VBUS-GND (0603WAF4701T5E, C23162) holds VGS
beyond -2.8 V up to 500 uA; same fix as 2600 Rev1 R_VBPD and SMS Rev0.

- design.py: R22 declared after every other resistor (no ref changes).
- power sheet redrawn with R22 on the VBUS rail; ERC 0, check_nets 453/453.
- Board: R22 inserted into the routed layout at (141.45, 59.6) beside the
  F.Cu VBUS run, VBUS stub + GND via; placement.py carries it for LAYOUT=1.
  KiCad DRC (all severities, schematic parity): 0 / 0 / 0.
- Exports regenerated (BOM/CPL 105 rows, gerbers, PDF, SVGs, renders);
  README power section and design review (post-layout change) updated.

Co-Authored-By: Claude Opus 5.5 <noreply@anthropic.com>

* NES Rev0: fix the microSD / USB-C alignment (J3 to the board edge, 3D models)

A reviewer reported J2 (microSD) and J3 (USB-C) as misaligned. Checked
against the SOFNG TF-015 and HRO TYPE-C-31-M-12 drawings, the STEP
vertices and a zoomed render:

- J3 sat 1.35 mm inside the top edge. HRO's recommended layout puts the
  PCB edge 5.79 mm in front of the pegs (fp y +3.19), so the face
  overhangs it by 0.46 mm; set back, a plug's overmold meets the board
  edge before the plug mates. J3 moves (125, 35) -> (125, 33.2). Its
  VBUS / D- ties between the pad row and the pegs move with it, nine
  1.8 mm F.Cu stubs join the new pad centres to the untouched routing,
  and one edge-row GND stitching via under the new front shield slot is
  removed. The front silk (now past the edge) is dropped; a Dwgs.User
  line marks HRO's edge.
-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
Parts:
- added R22: 4.7k, FujiNet-NES:R_0603_1608Metric, F.Cu at (141.4, 59.6)
- moved J3 1.80 mm to (125.0, 33.2)
Routing:
- net GND: track 131.1 -> 136.0 mm
- net VBUS: track 196.1 -> 200.8 mm
- net UBRG_DP: track 14.7 -> 18.3 mm
- net CC2: track 12.7 -> 14.5 mm
- net CC1: track 11.3 -> 13.1 mm
- net UBRG_DM: track 13.8 -> 15.6 mm
