File: ATARI-7800/FujiNet-7800-Rev0/esp32s3-sd.kicad_sch (KiCad schematic)
At the start: 14 parts, among them J3 microSD, SW3 S3_RST, SW4 S3_BOOT, U7 ESP32-S3-WROOM-1-N16R8

Commit message: ATARI-7800 Rev0: fix the edge, audit the circuit, redraw from the slot, place the board
Edge (board-killer in the schematic-only footprint): the 7800 edge has 18
positions at 2.54 mm with key slots at 3 and 16 for the console's plastic
keys. Pins 1, 2, 15, 16 (and 32, 31, 18, 17) sat one pitch inward, on the
key positions, with no slots and a 42.6 mm tab. tools/edge_geom.py now holds
the geometry (47.0 mm tab, slots centred on +-16.51, 2.4 x 10 mm);
tools/audit/edge_orientation.py checks it against Otaku-flash, tdididit's
boards, the a78-devcart gerbers and this repo's working FujiPlusCart
prototype gerbers (faces and power fingers).

Circuit (console research: Atari C025231 schematic, GCC1702B MARIA spec):
- 4.7k pull-downs on ROM_EN / RAM_EN / A8MASK (RP2350-E9)
- 1k at the /HALT finger (MARIA's HALT is a weak MOS output)
- 10 uF at the console 5V finger; bring-up test pads
- TS-1187A buttons and WS2812C-2020-V1 (the TL3342 and WS2812B-2020
  had 5 in stock at JLC); manufacturer fields for PCBWay
No glue change: R/W is pulled up during MARIA DMA, and the console gates
A15/A14/A12 low while its BIOS is mapped, so CARTSEL never fights it.

Schematic: SMS Rev0's hierarchy (wired root block diagram, hierarchical
labels, netlist parity); sheets in flow order from the slot; the glue
redrawn as a left-to-right gate-depth diagram; references renumbered
from the slot. ERC 0, check_nets 383/383, check_glue 4096/4096.

Board (not yet routed): SMS Rev0's 6-layer pipeline ported. A 72.4 x 115 mm
outline: the stock T-bar width on a 47 x 16.5 mm tab, with the key slots
cut in. Placement variant A (RP over the address fingers, SRAM over the
data fingers): unrouted DRC 0 errors, parity 0, check_vias 0. Shell:
case/FujiNet-7800-Shell.scad. README still describes the old board.

Co-Authored-By: Claude Opus 5.5 <noreply@anthropic.com>
Parts:
- removed R16, R17: 10k, FujiNet-7800:R_0603_1608Metric, symbol Device:R
- removed R18: 330R, FujiNet-7800:R_0603_1608Metric, symbol Device:R
- added R20, R21: 10k, FujiNet-7800:R_0603_1608Metric, symbol Device:R
- added R22: 330R, FujiNet-7800:R_0603_1608Metric, symbol Device:R
- D3: value WS2812B-2020-V6 -> WS2812C-2020-V1; LCSC C52917434 -> C2976072; MPN WS2812B-2020-V6 -> WS2812C-2020-V1
- SW3, SW4: footprint FujiNet-7800:SW_SPST_TL3342 -> FujiNet-7800:SW_SPST_TS-1187A; LCSC C2886898 -> C318884; MPN TL3342F160QG -> TS-1187A-B-A-B
Connections:
- net +3V3: now also R20.1, R21.1
- net LED_STRIP: now also R22.1
- net S3_EN: now also R20.2
- net SD_CD: now also R21.2
- net WS_DIN: now also R22.2
Other:
- title: FujiNet 7800 Rev0 - ESP32-S3, microSD, status LED -> FujiNet 7800 Rev0 - ESP32-S3 FujiNet, microSD, LED
- moved on the sheet: C29, C30, C31, C32, C33, D3, J3, RN3, SW3, SW4, U7
