File: SMS/FujiNet-SMS-Rev0/esp32s3-sd.kicad_sch (KiCad schematic)
At the start: 14 parts, among them J3 microSD, SW3 S3_RST, SW4 S3_BOOT, U9 ESP32-S3-WROOM-1-N16R8

Commit message: SMS Rev0: audit with kicad-happy + datasheets, fix the edge, redraw the schematic
Edge connector: every source (SMS Power slot diagram, little-scale, a 171-5519
scan, raphnet, the barbeque and reidrac footprints) puts the EVEN pins on the
component / label side with pins 1/2 at the right.  The schematic-only
footprint had the faces swapped, which would have put console +5V on /WR.
make_edge_fp.py now writes even pads on F.Cu, odd on B.Cu, 1.75 x 8.75 mm
fingers 0.75-9.5 mm from the edge on a 65.8 mm tab; check_nets.py asserts it
and tools/audit/edge_orientation.py checks it against the sources.

kicad-happy + datasheet audit (docs/design-review-rev0.md Part 1, 27 deep
review findings, gate 27/27): R_VBPD 4.7k VBUS pull-down (SS34 leakage lifts
the P-FET gate), /WAIT gate pull-up 10k -> 4.7k (GPIO34's reset pull-down vs
the 2N7002's 2.5 V threshold), 10 uF bulk on the console 5V.

Schematic: hierarchical sheets wired on a root block diagram (edge -> RP2354B
-> ESP32-S3 -> USB, glue and SRAM under the RP, power below); every sheet
drawn left to right, the glue as a wired logic network by gate depth, the
RP2354B mirrored so its bus faces the console, small sheets on A4.  Parts
are addressed by key (design.py), no more NES reference aliasing.  sch_draw
gains hierarchical labels, sheet blocks, a bus graph and flag / power-pin
lints; gen_sch checks the hierarchy against design.py and names nets by
their last path element (one bus vector per bus: KiCad joins differing
vectors by position).  ERC 0, check_nets 437/437, check_glue 8192/8192.

JLC CPL rotations measured against the EasyEDA footprint of every LCSC part
(tools/audit/jlc); the AS6C4008 has no EasyEDA footprint.

Co-Authored-By: Claude Opus 5.5 <noreply@anthropic.com>
Other:
- moved on the sheet: C29, C30, C31, C32, C33, D3, J3, R14, R15, R16, RN3, SW3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

Commit message: SMS Rev0 v2: port the FujiNet-7800 tooling, swap the near-stock-out parts
- export.py: JLCPCB and PCBWay packages (PCBWay turnkey BOM, centroid,
  assembly drawing); Manufacturer on every BOM part (design.MFR), written
  to symbols and footprints alike
- edge_geom.py: the SMS edge constants in one place (make_edge_fp,
  gen_pcb, check_gerbers); gen_pcb's body height, holes and In4 split now
  come from placement.py
- footprint paths from the schematic netlist (gen_pcb.fp_sheet_unit), so
  a part's units can be drawn on several sheets (prototype 2026-10-08:
  kicad-cli files it under the first sheet, parity accepts it)
- check_vias, check_gerbers, make_happy_config, stitch_gnd second ring,
  set_models main(), route_board.sh 12 passes / hybrid, DRC at all
  severities
- TL3342 -> TS-1187A-B-A-B (C318884), WS2812B-2020-V6 -> WS2812C-2020-V1
  (C2976072): ~5 in stock on 2026-10-07

Co-Authored-By: Claude Opus 5.5 <noreply@anthropic.com>
Parts:
- C29, C31, C32: Manufacturer (none) -> Samsung Electro-Mechanics
- C30, C33: Manufacturer (none) -> YAGEO
- D3: value WS2812B-2020-V6 -> WS2812C-2020-V1; LCSC C52917434 -> C2976072; MPN WS2812B-2020-V6 -> WS2812C-2020-V1; Manufacturer (none) -> Worldsemi
- J3: Manufacturer (none) -> SOFNG
- R14, R15, R16, RN3: Manufacturer (none) -> UNI-ROYAL
- SW3, SW4: footprint FujiNet-SMS:SW_SPST_TL3342 -> FujiNet-SMS:SW_SPST_TS-1187A; LCSC C2886898 -> C318884; MPN TL3342F160QG -> TS-1187A-B-A-B; Manufacturer (none) -> XKB Connection
- U9: Manufacturer (none) -> Espressif
Changed lines of the file:
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@@
+			)
+		)
+		(property "Manufacturer" "Espressif"
+			(at 127 78.74 0)
+			(effects
+				(font
+					(size 1.27 1.27)
+				)
+				(hide yes)
 			)
 		)
@@
 			)
 		)
+		(property "Manufacturer" "YAGEO"
+			(at 137.16 44.45 0)
+			(effects
+				(font
+					(size 1.27 1.27)
+				)
+				(hide yes)
+			)
+		)
 		(property "LCSC" "C14663"
 			(at 137.16 44.45 0)
@@
 			)
 		)
+		(property "Manufacturer" "Samsung Electro-Mechanics"
+			(at 149.86 44.45 0)
+			(effects
+				(font
+					(size 1.27 1.27)
+				)
+				(hide yes)
+			)
+		)
 		(property "LCSC" "C45783"
 			(at 149.86 44.45 0)
@@
 			)
 		)
+		(property "Manufacturer" "UNI-ROYAL"
+			(at 99.06 34.29 0)
+			(effects
+				(font
+					(size 1.27 1.27)
+				)
+				(hide yes)
+			)
+		)
 		(property "LCSC" "C25804"
 			(at 99.06 34.29 0)
@@
 			)
 		)
+		(property "Manufacturer" "Samsung Electro-Mechanics"
+			(at 88.9 41.91 0)
+			(effects
+				(font
+					(size 1.27 1.27)
+				)
+				(hide yes)
+			)
+		)
 		(property "LCSC" "C15849"
 			(at 88.9 41.91 0)
@@
 			)
 		)
-		(property "Footprint" "FujiNet-SMS:SW_SPST_TL3342"
+		(property "Footprint" "FujiNet-SMS:SW_SPST_TS-1187A"
 			(at 78.74 43.18 90)
 			(effects
@@
 			)
 		)
-		(property "MPN" "TL3342F160QG"
+		(property "MPN" "TS-1187A-B-A-B"
 			(at 78.74 43.18 90)
 			(effects
@@
 			)
 		)
-		(property "LCSC" "C2886898"
+		(property "Manufacturer" "XKB Connection"
+			(at 78.74 43.18 90)
+			(effects
+				(font
+					(size 1.27 1.27)
+				)
+				(hide yes)
+			)
+		)
+		(property "LCSC" "C318884"
 			(at 78.74 43.18 90)
 			(effects
@@
 			)
 		)
-		(property "Footprint" "FujiNet-SMS:SW_SPST_TL3342"
+		(property "Footprint" "FujiNet-SMS:SW_SPST_TS-1187A"
 			(at 83.82 66.04 90)
 			(effects
@@
 			)
 		)
-		(property "MPN" "TL3342F160QG"
+		(property "MPN" "TS-1187A-B-A-B"
 			(at 83.82 66.04 90)
 			(effects
@@
 			)
 		)
-		(property "LCSC" "C2886898"
+		(property "Manufacturer" "XKB Connection"
+			(at 83.82 66.04 90)
+			(effects
+				(font
+					(size 1.27 1.27)
+				)
+				(hide yes)
+			)
+		)
+		(property "LCSC" "C318884"
 			(at 83.82 66.04 90)
 			(effects
@@
 		)
 		(property "MPN" "TF-015"
+			(at 203.2 99.06 0)
+			(effects
+				(font
+					(size 1.27 1.27)
+				)
+				(hide yes)
+			)
+		)
+		(property "Manufacturer" "SOFNG"
 			(at 203.2 99.06 0)
 			(effects
@@
 			)
 		)
+		(property "Manufacturer" "UNI-ROYAL"
+			(at 170.18 81.28 90)
+			(effects
+				(font
+					(size 1.27 1.27)
+				)
+				(hide yes)
+			)
+		)
 		(property "LCSC" "C29718"
 			(at 170.18 81.28 90)
@@
 			)
 		)
+		(property "Manufacturer" "UNI-ROYAL"
+			(at 231.14 116.84 0)
+			(effects
+				(font
+					(size 1.27 1.27)
+				)
+				(hide yes)
+			)
+		)
 		(property "LCSC" "C25804"
 			(at 231.14 116.84 0)
@@
 			)
 		)
+		(property "Manufacturer" "Samsung Electro-Mechanics"
+			(at 220.98 116.84 0)
+			(effects
+				(font
+					(size 1.27 1.27)
+				)
+				(hide yes)
+			)
+		)
 		(property "LCSC" "C19702"
 			(at 220.98 116.84 0)
@@
 			)
 		)
+		(property "Manufacturer" "UNI-ROYAL"
+			(at 154.94 139.7 90)
+			(effects
+				(font
+					(size 1.27 1.27)
+				)
+				(hide yes)
+			)
+		)
 		(property "LCSC" "C23138"
 			(at 154.94 139.7 90)
@@
 			)
 		)
-		(property "Value" "WS2812B-2020-V6"
+		(property "Value" "WS2812C-2020-V1"
 			(at 186.69 140.97 0)
 			(effects
@@
 			)
 		)
-		(property "Datasheet" "https://cdn-shop.adafruit.com/product-files/4684/4684_WS2812B-2020_V1.3_EN.pdf"
+		(property "Datasheet" "http://www.world-semi.com/DownLoadFile/1132"
 			(at 180.34 139.7 0)
 			(effects
@@
 			)
 		)
-		(property "MPN" "WS2812B-2020-V6"
+		(property "MPN" "WS2812C-2020-V1"
 			(at 180.34 139.7 0)
 			(effects
@@
 			)
 		)
-		(property "LCSC" "C52917434"
+		(property "Manufacturer" "Worldsemi"
+			(at 180.34 139.7 0)
+			(effects
+				(font
+					(size 1.27 1.27)
+				)
+				(hide yes)
+			)
+		)
+		(property "LCSC" "C2976072"
 			(at 180.34 139.7 0)
 			(effects
@@
 			(at 208.28 139.7 0)
 			(effects
+				(font
+					(size 1.27 1.27)
+				)
+				(hide yes)
+			)
+		)
+		(property "Manufacturer" "YAGEO"
+			(at 208.28 139.7 0)
+			(effects
