File: SMS/FujiNet-SMS-Rev0/cart-bus.kicad_sch (KiCad schematic)
At the start: 38 parts, among them J1 SMS_Cart_Edge_50, J4 DBG UART, Q1 2N7002, U10 AS6C4008-55TIN, U11 74HCT00, U12 74HCT14, U13 74HCT27, U4 RP2354B, U7 AS6C4008-55TIN, U8 74HCT10, U9 74HCT27

Commit message: SMS Rev0 v2: redraw every sheet to mirror the board
Each sheet is now hand-placed in tools/sch_layout.py from where its parts
sit on the board, turned so the edge fingers face left (south -> left,
north -> right, west -> top, east -> bottom), and every connection on a
sheet is a wire:

- rp-core: the RP2354B core unit with its decoupling ring at the pins, the
  regulator corner, the crystal, SWD, RUN / BOOTSEL and the RESET diode
  (planar).
- fujinet: a functional ESP32-S3 symbol, EN / BOOT, the WS2812, and the
  microSD's SPI lines stepping into the socket with the pull-ups between
  them (planar).
- usb: a functional USB-C symbol, the CP2102N mirrored to face the
  receptacle, and the auto-program pair.  This page has one crossing, which
  cannot be avoided: RTS and DTR sit side by side on the bridge and each
  feeds the base of one transistor and the emitter of the other.
- power: the CONS_5V / VBUS OR on one +5V line, the LDO above it, the buck
  below it, and the rail PWR_FLAGs grouped together (planar).
- root: the board outline at 2:1, turned the same way, with each sheet's
  block at its region and the nine signals between sheets wired without a
  crossing; notes cover the stack-up and the firmware contract.

Gates: gen_sch.py checks the mirror (Kendall tau >= 0.85 per axis for the
major parts, multi-unit packages counted at the centre of their units,
parts within 5 mm on the board counted as level; every sheet is at
1.00 / 1.00) and a crossing budget per sheet (cart-bus 75, usb 1,
others 0).  ERC is 0 at all severities, netlist parity holds, the net
names equal tools/nets.lock, check_nets passes 442/442, check_glue
8192/8192, and edge_orientation passes.

Co-Authored-By: Claude Opus 5.5 <noreply@anthropic.com>
Other:
- note added: "How to read this page: it is the board turned so the cartridge fingers face left (board south -> page left, north -> right, west -> top, east -> bottom), and every part sits where it is on the board. A plain wire is a connection the copper makes on one layer: the edge straight into SRAM0, which stands in the classic ROM spot over the fingers (the SMS edge is the JEDEC 32-pin memory pinout unrolle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"
- note added: "fujinet-firmware pico/sms sms_cart.h: sms_glue_oe(), sms_glue_we(). RD, WR, CE = the console's /RD, /WR, /CE asserted; GAME, MBOX, RAM_WE, LOAD = RP GPIO38, 35, 39, 40; PWR_OK = console +5V. CEP_N = !(CE & PWR_OK); WIN8 = A15 & !A14 & !A13 (the $8000-$9FFF load window) MBA_N = !(MBOX & A13 & A12); SLOT2_NM = A15 & !A14 & !(MBOX & A13 & A12) OE_ADDR = !A15 | SLOT2_NM; WE_LOAD = RD & CEP & LOAD & W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"
- title: FujiNet SMS Rev0 - Cartridge bus: edge, RP2354B GPIO, 1 MB SRAM, 74HCT glue -> FujiNet SMS Rev0 - Cartridge bus: edge, SRAM, RP GPIO, glue
- moved on the sheet: C34, C39, C40, C41, C42, C44, C45, C46, D7, J1, J4, Q1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
