File: SMS/FujiNet-SMS-Rev0/rp-core.kicad_sch (KiCad schematic)
At the start: 40 parts, among them SW2 RESET, SW4 BOOTSEL, U4 RP2354B, Y1 12MHz

Commit message: SMS Rev0 v2: redraw every sheet to mirror the board
Each sheet is now hand-placed in tools/sch_layout.py from where its parts
sit on the board, turned so the edge fingers face left (south -> left,
north -> right, west -> top, east -> bottom), and every connection on a
sheet is a wire:

- rp-core: the RP2354B core unit with its decoupling ring at the pins, the
  regulator corner, the crystal, SWD, RUN / BOOTSEL and the RESET diode
  (planar).
- fujinet: a functional ESP32-S3 symbol, EN / BOOT, the WS2812, and the
  microSD's SPI lines stepping into the socket with the pull-ups between
  them (planar).
- usb: a functional USB-C symbol, the CP2102N mirrored to face the
  receptacle, and the auto-program pair.  This page has one crossing, which
  cannot be avoided: RTS and DTR sit side by side on the bridge and each
  feeds the base of one transistor and the emitter of the other.
- power: the CONS_5V / VBUS OR on one +5V line, the LDO above it, the buck
  below it, and the rail PWR_FLAGs grouped together (planar).
- root: the board outline at 2:1, turned the same way, with each sheet's
  block at its region and the nine signals between sheets wired without a
  crossing; notes cover the stack-up and the firmware contract.

Gates: gen_sch.py checks the mirror (Kendall tau >= 0.85 per axis for the
major parts, multi-unit packages counted at the centre of their units,
parts within 5 mm on the board counted as level; every sheet is at
1.00 / 1.00) and a crossing budget per sheet (cart-bus 75, usb 1,
others 0).  ERC is 0 at all severities, netlist parity holds, the net
names equal tools/nets.lock, check_nets passes 442/442, check_glue
8192/8192, and edge_orientation passes.

Co-Authored-By: Claude Opus 5.5 <noreply@anthropic.com>
Other:
- note added: "Supplies (RP2350 datasheet 6.3.7): IOVDD, QSPI_IOVDD, USB_OTP_VDD, ADC_AVDD and VREG_VIN on +3V3_RP, the LDO that rises with the console 5V; the core regulator switches VREG_LX through 3.3 uH onto DVDD (VREG_FB senses it), its analog supply VREG_AVDD through 33R / 4.7 uF. One 100 nF at every supply pin, drawn at the pin it serves. RESET resets the RP2354B and the ESP32-S3 together (D5 steers RST_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"
- title: FujiNet SMS Rev0 - RP2354B core: supplies, core regulator, crystal, USB, RUN / BOOTSEL -> FujiNet SMS Rev0 - RP2354B core: supplies, crystal, USB, RUN
- moved on the sheet: C10, C11, C12, C18, C19, C20, C21, C22, C23, C27, C28, C29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
