File: SMS/FujiNet-SMS-Rev0/FujiNet-SMS-Rev0.kicad_pcb (KiCad board)
At the start: 6 copper layers, 100 x 93 mm, 119 parts, among them J1 SMS_Cart_Edge_50, J2 DBG UART, J3 microSD, J4 USB-C, Q1 2N7002, Q2 AO3401A, SW1 RESET, SW2 BOOTSEL, SW3 S3_RST, SW4 S3_BOOT, U1 RP2354B, U10 CP2102N-A02-GQFN28, U11 UMH3N, U12 AP63203WU, U13 AP2112K-3.3, U2 AS6C4008-55TIN, U3 AS6C4008-55TIN, U4 74HCT14, U5 74HCT27, U6 74HCT27, U7 74HCT10, U8 74HCT00, U9 ESP32-S3-WROOM-1-N16R8, Y1 12MHz

Commit message: SMS Rev0 v2: co-designed floorplan, region sheets, E9 pull-downs, frozen refs and nets
Floorplan study (docs/floorplan-study.md): the SMS edge is the JEDEC
32-pin memory pinout unrolled, so SRAM0 standing upright in the ROM spot
takes A0-A12 / D0-D7 / GND with no crossing.  gen_pcb.sram0_fanin draws
that fan-in locked (funnel, two corner wraps, B-finger jog vias, escape
vias for CE# and OE#).  Four candidates scored and trial-routed in
parallel; P3 (RP2354B straight north of SRAM0, SRAM1 west, glue east over
the strobes) routes best (45 unrouted after 4 passes vs 50 for the first
layout) and reads straight across on the schematic page.

- placement.py: candidates as blocks; the RP2354B + ring as a rigid macro
  (turns as a whole, dvdd_island turns with it); per-variant In4 +5V
  island polygon; label area for the shell
- design.py: sheets are board regions (cart-bus, rp-core, fujinet, usb,
  power); the RP2354B as a two-unit symbol (GPIO on cart-bus, core on
  rp-core); resistor packs one unit per resistor; RP2350-E9 4.7k
  pull-downs on GAME/LOAD/RAM_WE/MBOX/SA19 (check_nets asserts <= 8.2k);
  bring-up pads (CE, OE, WE, PWR_OK, rails, DVDD)
- geographic references (tools/annotate.py -> tools/refs.lock); net names
  frozen in tools/nets.lock (gen_sch fails if a redraw changes one)
- sch_draft.py: an every-pin-labelled draft of the final hierarchy so the
  board is built while the sheets are drawn; sch_draw lint for wired
  sheets (one piece per net, no 4-way junctions, wires clear of text,
  crossing count); sch_place.py mirror check
- check_parts_inside: footprint keep-outs (the S3 antenna bars parts)
- shell: RESET plunger redesigned (captive flange under the guide, stem
  on the TS-1187A actuator, travel asserts, interference part)

ERC 0, parity 126/126, check_nets 442/442, check_glue 8192/8192.
Board placed, not routed yet.

Co-Authored-By: Claude Opus 5.5 <noreply@anthropic.com>
Parts:
- added R23: 330R, FujiNet-SMS:R_0603_1608Metric, F.Cu at (58.0, 85.0)
- added R24: 1k, FujiNet-SMS:R_0603_1608Metric, F.Cu at (66.0, 85.0)
- added R25: 4.7k, FujiNet-SMS:R_0603_1608Metric, F.Cu at (84.2, 104.2)
- added R26: 22k, FujiNet-SMS:R_0603_1608Metric, F.Cu at (121.6, 104.6)
- added R27: 100k, FujiNet-SMS:R_0603_1608Metric, F.Cu at (123.4, 104.6)
- added TP10: WE, FujiNet-SMS:TestPoint_Pad_D1.5mm, F.Cu at (117.2, 94.0)
- added TP11: +5V, FujiNet-SMS:TestPoint_Pad_D1.5mm, F.Cu at (62.0, 96.5)
- added TP12: PWR_OK, FujiNet-SMS:TestPoint_Pad_D1.5mm, F.Cu at (117.2, 97.0)
- added TP13: GND, FujiNet-SMS:TestPoint_Pad_D1.5mm, F.Cu at (117.2, 100.0)
- added TP14: CONS_5V, FujiNet-SMS:TestPoint_Pad_D1.5mm, F.Cu at (148.0, 98.0)
- added TP15: BUSREQ, FujiNet-SMS:TestPoint_Pad_D1.5mm, F.Cu at (77.1, 106.6)
- added TP16: CONT, FujiNet-SMS:TestPoint_Pad_D1.5mm, F.Cu at (89.8, 106.6)
- added TP7: +3V3_RP, FujiNet-SMS:TestPoint_Pad_D1.5mm, F.Cu at (90.5, 80.8)
- added TP8: CE, FujiNet-SMS:TestPoint_Pad_D1.5mm, F.Cu at (117.2, 88.0)
- added TP9: OE, FujiNet-SMS:TestPoint_Pad_D1.5mm, F.Cu at (117.2, 91.0)
- C1, C16, C24, C25, C6: value 100nF -> 22uF; footprint FujiNet-SMS:C_0603_1608Metric -> FujiNet-SMS:C_0805_2012Metric
- C12, C32, C38: value 10uF -> 100nF
- C13, C37: value 4.7uF -> 100nF
- C14, C21, C8: value 100nF -> 4.7uF
- C17: value 4.7uF -> 22uF; footprint FujiNet-SMS:C_0603_1608Metric -> FujiNet-SMS:C_0805_2012Metric
- C19, C20: value 15pF -> 100nF
- C23: value 10uF -> 15pF
- C27, C3: value 100nF -> 10uF
- C29, C40, C42, C45, C46: value 22uF -> 100nF; footprint FujiNet-SMS:C_0805_2012Metric -> FujiNet-SMS:C_0603_1608Metric
- C31, C34, C47: value 1uF -> 100nF
- C33: value 100nF -> 15pF
- C35, C36, C4, C7: value 100nF -> 1uF
- C41: value 22uF -> 10uF; footprint FujiNet-SMS:C_0805_2012Metric -> FujiNet-SMS:C_0603_1608Metric
- C48: value 1uF -> 10uF
- D1: value BAT54C -> SS34; footprint FujiNet-SMS:SOT-23 -> FujiNet-SMS:D_SMA
- D2: value red -> ESD5Z5.0T1G; footprint FujiNet-SMS:LED_0603_1608Metric -> FujiNet-SMS:D_SOD-523
- D3: value WS2812B-2020-V6 -> ESD5Z5.0T1G; footprint FujiNet-SMS:LED_WS2812B-2020_PLCC4_2.0x2.0mm -> FujiNet-SMS:D_SOD-523
- D5: value ESD5Z5.0T1G -> BAT54C; footprint FujiNet-SMS:D_SOD-523 -> FujiNet-SMS:SOT-23
- D6: value ESD5Z5.0T1G -> WS2812C-2020-V1; footprint FujiNet-SMS:D_SOD-523 -> FujiNet-SMS:LED_WS2812B-2020_PLCC4_2.0x2.0mm
- D7: value SS34 -> red; footprint FujiNet-SMS:D_SMA -> FujiNet-SMS:LED_0603_1608Metric
- J2: value DBG UART -> USB-C; footprint FujiNet-SMS:PinHeader_1x03_P2.54mm_Vertical -> FujiNet-SMS:USB_C_Receptacle_HRO_TYPE-C-31-M-12
- J4: value USB-C -> DBG UART; footprint FujiNet-SMS:USB_C_Receptacle_HRO_TYPE-C-31-M-12 -> FujiNet-SMS:PinHeader_1x03_P2.54mm_Vertical
- R1: value 33R -> 5.1k
- R10: value 1k -> 27R
- R11: value 4.7k -> 1k
- R13: value 100k -> 47k
- R14, R15: value 10k -> 1k
- R16: value 330R -> 10k
- R17: value 5.1k -> 27R
- R18: value 5.1k -> 4.7k
- R19: value 22k -> 4.7k
- R2: value 1k -> 5.1k
- R20: value 47k -> 4.7k
- R21, R3: value 10k -> 4.7k
- R5, R7: value 1k -> 10k
- R6: value 1k -> 33R
- R8: value 27R -> 1k
- R9: value 27R -> 10k
- RN1: value 4x100R -> 4x10k
- RN3: value 4x10k -> 4x100R
- SW1: value RESET -> S3_RST; footprint FujiNet-SMS:SW_SPST_TL3342 -> FujiNet-SMS:SW_SPST_TS-1187A
- SW2: value BOOTSEL -> RESET; footprint FujiNet-SMS:SW_SPST_TL3342 -> FujiNet-SMS:SW_SPST_TS-1187A
- SW3: value S3_RST -> S3_BOOT; footprint FujiNet-SMS:SW_SPST_TL3342 -> FujiNet-SMS:SW_SPST_TS-1187A
- SW4: value S3_BOOT -> BOOTSEL; footprint FujiNet-SMS:SW_SPST_TL3342 -> FujiNet-SMS:SW_SPST_TS-1187A
- TP1: value CONT -> DVDD
- TP2: value BUSREQ -> +3V3
- U1: value RP2354B -> ESP32-S3-WROOM-1-N16R8; footprint FujiNet-SMS:QFN-80-1EP_10x10mm_P0.4mm_EP3.4x3.4mm -> FujiNet-SMS:ESP32-S3-WROOM-1
- U10: value CP2102N-A02-GQFN28 -> AS6C4008-55TIN; footprint FujiNet-SMS:QFN-28-1EP_5x5mm_P0.5mm_EP3.35x3.35mm -> FujiNet-SMS:TSOP-I-32_18.4x8mm_P0.5mm
- U11: value UMH3N -> 74HCT00; footprint FujiNet-SMS:SOT-363_SC-70-6 -> FujiNet-SMS:SOIC-14_3.9x8.7mm_P1.27mm
- U12: value AP63203WU -> 74HCT14; footprint FujiNet-SMS:TSOT-23-6 -> FujiNet-SMS:SOIC-14_3.9x8.7mm_P1.27mm
- U13: value AP2112K-3.3 -> 74HCT27; footprint FujiNet-SMS:SOT-23-5 -> FujiNet-SMS:SOIC-14_3.9x8.7mm_P1.27mm
- U2: value AS6C4008-55TIN -> CP2102N-A02-GQFN28; footprint FujiNet-SMS:TSOP-I-32_18.4x8mm_P0.5mm -> FujiNet-SMS:QFN-28-1EP_5x5mm_P0.5mm_EP3.35x3.35mm
- U3: value AS6C4008-55TIN -> UMH3N; footprint FujiNet-SMS:TSOP-I-32_18.4x8mm_P0.5mm -> FujiNet-SMS:SOT-363_SC-70-6
- U4: value 74HCT14 -> RP2354B; footprint FujiNet-SMS:SOIC-14_3.9x8.7mm_P1.27mm -> FujiNet-SMS:QFN-80-1EP_10x10mm_P0.4mm_EP3.4x3.4mm
- U5: value 74HCT27 -> AP63203WU; footprint FujiNet-SMS:SOIC-14_3.9x8.7mm_P1.27mm -> FujiNet-SMS:TSOT-23-6
- U6: value 74HCT27 -> AP2112K-3.3; footprint FujiNet-SMS:SOIC-14_3.9x8.7mm_P1.27mm -> FujiNet-SMS:SOT-23-5
- U7: value 74HCT10 -> AS6C4008-55TIN; footprint FujiNet-SMS:SOIC-14_3.9x8.7mm_P1.27mm -> FujiNet-SMS:TSOP-I-32_18.4x8mm_P0.5mm
- U8: value 74HCT00 -> 74HCT10
- U9: value ESP32-S3-WROOM-1-N16R8 -> 74HCT27; footprint FujiNet-SMS:ESP32-S3-WROOM-1 -> FujiNet-SMS:SOIC-14_3.9x8.7mm_P1.27mm
- moved D1 95.9 mm to (145.5, 39.0), turned to 90 degrees
- moved D7 91.7 mm to (66.0, 88.0), turned to 0 degrees
- moved C43 90.1 mm to (61.5, 88.0)
- moved J4 81.3 mm to (70.0, 96.0), turned to 90 degrees
- moved U9 77.5 mm to (133.0, 84.0)
- moved D6 74.9 mm to (58.0, 88.0), turned to 0 degrees
- moved C41 74.5 mm to (76.5, 80.0)
- moved C16 72.4 mm to (147.5, 49.0), turned to 90 degrees
- moved TP2 70.2 mm to (129.5, 61.0)
- moved C1 69.4 mm to (53.5, 41.0), turned to 90 degrees
- moved C2 69.3 mm to (53.5, 44.5), turned to 90 degrees
- moved C34 68.1 mm to (76.5, 76.5)
- moved C17 67.9 mm to (147.5, 52.5), turned to 90 degrees
- moved J2 66.2 mm to (128.0, 37.0), turned to 180 degrees
- moved C15 63.6 mm to (143.0, 52.5), turned to 0 degrees
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Connections:
- net /WAIT_N renamed /cart-bus/WAIT_N
- C1 pad 1: +3V3_RP -> +3V3
- C13 pad 1: +3V3_RP -> +3V3
- C14 pad 1: DVDD -> +3V3
- C15 pad 1: DVDD -> /power/BUCK_SW
- C15 pad 2: GND -> /power/BUCK_BST
- C16 pad 1: DVDD -> +5V
- C17 pad 1: DVDD -> +5V
- C18 pad 1: /rp2354b/VREG_AVDD -> +3V3_RP
- C19 pad 1: /rp2354b/XIN -> DVDD
- C2 pad 1: +3V3_RP -> +3V3
- C20 pad 1: /rp2354b/XOUT_Y -> DVDD
- C21 pad 1: +5V -> DVDD
- C22 pad 1: +5V -> DVDD
- C23 pad 1: +5V -> /rp-core/XOUT_Y
- C24 pad 1: +5V -> +3V3
- C25 pad 1: +5V -> +3V3
- C27 pad 1: +5V -> +3V3_RP
- C28 pad 1: +5V -> +3V3_RP
- C29 pad 1: +3V3 -> +3V3_RP
- C3 pad 1: +3V3_RP -> +3V3
- C30 pad 1: +3V3 -> +3V3_RP
- C31 pad 1: /S3_EN -> +3V3_RP
- C32 pad 1: +3V3 -> +3V3_RP
- C33 pad 1: +5V -> /rp-core/XIN
- C34 pad 1: VBUS -> +5V
- C35 pad 1: VBUS -> +5V
- C36 pad 1: +3V3 -> +3V3_RP
- C37 pad 1: +3V3 -> +3V3_RP
- C38 pad 1: CONS_5V -> +3V3_RP
- C39 pad 1: CONS_5V -> +5V
- C4 pad 1: +3V3_RP -> VBUS
- C44 pad 1: /power/BUCK_SW -> +5V
- C44 pad 2: /power/BUCK_BST -> GND
- C45 pad 1: +3V3 -> +5V
- C46 pad 1: +3V3 -> +5V
- C47 pad 1: +5V -> CONS_5V
- C48 pad 1: +3V3_RP -> CONS_5V
- C5 pad 1: +3V3_RP -> VBUS
- C6 pad 1: +3V3_RP -> +5V
- C7 pad 1: +3V3_RP -> /S3_EN
- C8 pad 1: +3V3_RP -> /rp-core/VREG_AVDD
- D1 pad 1: /rp2354b/RUN -> +5V
- D1 pad 2: /S3_EN -> VBUS
- D2 pad 1: GND -> VBUS
- D2 pad 2: /rp2354b/RP_LED_A -> GND
- D3 pad 1: unconnected-(D3-DOUT-Pad1) -> /usb/UBRG_DP
- D4 pad 1: /usb-uart/UBRG_DP -> /usb/UBRG_DM
- D5 pad 1: /usb-uart/UBRG_DM -> /rp-core/RUN
- D5 pad 2: GND -> /S3_EN
- D6 pad 1: VBUS -> unconnected-(D6-DOUT-Pad1)
- D7 pad 1: +5V -> GND
- D7 pad 2: VBUS -> /cart-bus/RP_LED_A
- J1 pad 10: /A11 -> /cart-bus/A11
- J1 pad 12: /A10 -> /cart-bus/A10
- J1 pad 13: /CE_N -> /cart-bus/CE_N
- J1 pad 14: /D7 -> /cart-bus/D7
- J1 pad 15: /D6 -> /cart-bus/D6
- J1 pad 16: /D5 -> /cart-bus/D5
- J1 pad 17: /D4 -> /cart-bus/D4
- J1 pad 18: /D3 -> /cart-bus/D3
- J1 pad 2: /WR_N -> /cart-bus/WR_N
- J1 pad 22: /D2 -> /cart-bus/D2
- J1 pad 23: /D1 -> /cart-bus/D1
- J1 pad 24: /D0 -> /cart-bus/D0
- J1 pad 25: /A0 -> /cart-bus/A0
- J1 pad 26: /A1 -> /cart-bus/A1
- J1 pad 27: /A2 -> /cart-bus/A2
- J1 pad 28: /A3 -> /cart-bus/A3
- J1 pad 29: /A4 -> /cart-bus/A4
- J1 pad 3: /MREQ_N -> /cart-bus/MREQ_N
- J1 pad 30: /A5 -> /cart-bus/A5
- J1 pad 31: /A6 -> /cart-bus/A6
- J1 pad 32: /A7 -> /cart-bus/A7
- J1 pad 33: /A12 -> /cart-bus/A12
- J1 pad 34: /edge/CONT_N -> /cart-bus/CONT_N
- J1 pad 36: /A15 -> /cart-bus/A15
- J1 pad 37: /M1_N -> /cart-bus/M1_N
- J1 pad 38: /IORQ_N -> /cart-bus/IORQ_N
- J1 pad 4: /RD_N -> /cart-bus/RD_N
- J1 pad 44: /edge/BUSREQ_N -> /cart-bus/BUSREQ_N
- J1 pad 46: /RESET_N -> /cart-bus/RESET_N
- J1 pad 47: /CLK -> /cart-bus/CLK
- J1 pad 6: /A14 -> /cart-bus/A14
- J1 pad 7: /A13 -> /cart-bus/A13
- J1 pad 8: /A8 -> /cart-bus/A8
- J1 pad 9: /A9 -> /cart-bus/A9
- J3 pad 1: /esp32s3-sd/SD_DAT2 -> /fujinet/SD_DAT2
- J3 pad 2: /esp32s3-sd/SD_CS -> /fujinet/SD_CS
- J3 pad 3: /esp32s3-sd/SD_MOSI -> /fujinet/SD_MOSI
- J3 pad 5: /esp32s3-sd/SD_SCK -> /fujinet/SD_SCK
- J3 pad 7: /esp32s3-sd/SD_MISO -> /fujinet/SD_MISO
- J3 pad 8: /esp32s3-sd/SD_DAT1 -> /fujinet/SD_DAT1
- J3 pad 9: /esp32s3-sd/SD_CD -> /fujinet/SD_CD
- L1 pad 2: /rp2354b/RP_LX -> /rp-core/RP_LX
- Q1 pad 1: /rp2354b/WAIT_GATE -> /cart-bus/WAIT_GATE
- R1 pad 1: +3V3_RP -> /usb/CC1
- R1 pad 2: /rp2354b/VREG_AVDD -> GND
- R10 pad 1: /rp2354b/RP_LED -> /USB_DM
- R10 pad 2: /rp2354b/RP_LED_A -> /rp-core/RP_USB_DM
- R11 pad 1: +3V3_RP -> /rp-core/XOUT
- R11 pad 2: /rp2354b/WAIT_GATE -> /rp-core/XOUT_Y
- R12 pad 1: CONS_5V -> VBUS
- R12 pad 2: /glue/VSENSE -> /usb/VBUS_SNS
- R13 pad 1: /glue/VSENSE -> /usb/VBUS_SNS
- R14 pad 1: +3V3 -> /rp-core/QSPI_SS
- R14 pad 2: /S3_EN -> /rp-core/BOOTSEL_BTN
- R15 pad 1: +3V3 -> /BOOTSEL_CTL
- R15 pad 2: /esp32s3-sd/SD_CD -> /rp-core/QSPI_SS
- R16 pad 1: /esp32s3-sd/LED_STRIP -> +3V3_RP
- R16 pad 2: /esp32s3-sd/WS_DIN -> /rp-core/QSPI_SS
- R17 pad 1: /usb-uart/CC1 -> /USB_DP
- R17 pad 2: GND -> /rp-core/RP_USB_DP
- R18 pad 1: /usb-uart/CC2 -> /cart-bus/SA19
- R19 pad 1: VBUS -> /cart-bus/MBOX
- R19 pad 2: /usb-uart/VBUS_SNS -> GND
- R2 pad 1: /rp2354b/XOUT -> /usb/CC2
- R2 pad 2: /rp2354b/XOUT_Y -> GND
- R20 pad 1: /usb-uart/VBUS_SNS -> /cart-bus/GAME
- R21 pad 1: +3V3 -> /cart-bus/RAM_WE
- R21 pad 2: /usb-uart/CP_RST -> GND
- R22 pad 1: VBUS -> /cart-bus/LOAD
- R3 pad 1: +3V3_RP -> VBUS
- R3 pad 2: /rp2354b/RUN -> GND
- R4 pad 1: +3V3_RP -> +3V3
- R4 pad 2: /rp2354b/QSPI_SS -> /fujinet/SD_CD
- R5 pad 1: /rp2354b/QSPI_SS -> +3V3
- R5 pad 2: /rp2354b/BOOTSEL_BTN -> /S3_EN
- R6 pad 1: /RUN_CTL -> +3V3_RP
- R6 pad 2: /rp2354b/RUN -> /rp-core/VREG_AVDD
- R7 pad 1: /BOOTSEL_CTL -> +3V3_RP
- R7 pad 2: /rp2354b/QSPI_SS -> /rp-core/RUN
- R8 pad 1: /USB_DP -> /RUN_CTL
- R8 pad 2: /rp2354b/RP_USB_DP -> /rp-core/RUN
- R9 pad 1: /USB_DM -> +3V3
- R9 pad 2: /rp2354b/RP_USB_DM -> /usb/CP_RST
- RN1 pad 1: /rp2354b/RP_D0 -> /fujinet/SD_CS
- RN1 pad 2: /rp2354b/RP_D1 -> /fujinet/SD_MISO
- RN1 pad 3: /rp2354b/RP_D2 -> /fujinet/SD_DAT1
- RN1 pad 4: /rp2354b/RP_D3 -> /fujinet/SD_DAT2
- RN1 pad 5: /D3 -> +3V3
- RN1 pad 6: /D2 -> +3V3
- RN1 pad 7: /D1 -> +3V3
- RN1 pad 8: /D0 -> +3V3
- RN2 pad 1: /rp2354b/RP_D4 -> /cart-bus/RP_D0
- RN2 pad 2: /rp2354b/RP_D5 -> /cart-bus/RP_D1
- RN2 pad 3: /rp2354b/RP_D6 -> /cart-bus/RP_D2
- RN2 pad 4: /rp2354b/RP_D7 -> /cart-bus/RP_D3
- RN2 pad 5: /D7 -> /cart-bus/D3
- RN2 pad 6: /D6 -> /cart-bus/D2
- RN2 pad 7: /D5 -> /cart-bus/D1
- RN2 pad 8: /D4 -> /cart-bus/D0
- RN3 pad 1: /esp32s3-sd/SD_CS -> /cart-bus/RP_D4
- RN3 pad 2: /esp32s3-sd/SD_MISO -> /cart-bus/RP_D5
- RN3 pad 3: /esp32s3-sd/SD_DAT1 -> /cart-bus/RP_D6
- RN3 pad 4: /esp32s3-sd/SD_DAT2 -> /cart-bus/RP_D7
- RN3 pad 5: +3V3 -> /cart-bus/D7
- RN3 pad 6: +3V3 -> /cart-bus/D6
- RN3 pad 7: +3V3 -> /cart-bus/D5
- RN3 pad 8: +3V3 -> /cart-bus/D4
- SW1 pad 1: /rp2354b/RST_BTN -> /S3_EN
- SW2 pad 1: /rp2354b/BOOTSEL_BTN -> /rp-core/RST_BTN
- SW3 pad 1: /S3_EN -> /S3_IO0
- SW4 pad 1: /S3_IO0 -> /rp-core/BOOTSEL_BTN
- TP1 pad 1: /edge/CONT_N -> DVDD
- TP2 pad 1: /edge/BUSREQ_N -> +3V3
- TP3 pad 1: /rp2354b/SWCLK -> /rp-core/SWCLK
- TP4 pad 1: /rp2354b/SWDIO -> /rp-core/SWDIO
- TP6 pad 1: /rp2354b/RUN -> /rp-core/RUN
- U1 pad 1: /A4 -> GND
- U1 pad 10: DVDD -> unconnected-(U1-IO17-Pad10)
- U1 pad 11: /A12 -> unconnected-(U1-IO18-Pad11)
- U1 pad 12: /A13 -> unconnected-(U1-IO8-Pad12)
- U1 pad 13: /A14 -> /USB_DM
- U1 pad 14: /A15 -> /USB_DP
- U1 pad 15: +3V3_RP -> unconnected-(U1-IO3-Pad15)
- U1 pad 16: /rp2354b/RP_D0 -> unconnected-(U1-IO46-Pad16)
- U1 pad 17: /rp2354b/RP_D1 -> unconnected-(U1-IO9-Pad17)
- U1 pad 18: /rp2354b/RP_D2 -> unconnected-(U1-IO10-Pad18)
- U1 pad 19: /rp2354b/RP_D3 -> unconnected-(U1-IO11-Pad19)
- U1 pad 2: /A5 -> +3V3
- U1 pad 20: /rp2354b/RP_D4 -> unconnected-(U1-IO12-Pad20)
- U1 pad 21: /rp2354b/RP_D5 -> unconnected-(U1-IO13-Pad21)
- U1 pad 22: /rp2354b/RP_D6 -> unconnected-(U1-IO14-Pad22)
- U1 pad 23: /rp2354b/RP_D7 -> unconnected-(U1-IO21-Pad23)
- U1 pad 24: +3V3_RP -> unconnected-(U1-IO47-Pad24)
- U1 pad 25: /RD_N -> /fujinet/LED_STRIP
- U1 pad 26: /WR_N -> unconnected-(U1-IO45-Pad26)
- U1 pad 27: /MREQ_N -> /S3_IO0
- U1 pad 28: /CE_N -> unconnected-(U1-IO35-Pad28)
- U1 pad 29: +3V3_RP -> unconnected-(U1-IO36-Pad29)
- U1 pad 3: /A6 -> /S3_EN
- U1 pad 30: /rp2354b/XIN -> unconnected-(U1-IO37-Pad30)
- U1 pad 31: /rp2354b/XOUT -> /fujinet/SD_MOSI
- U1 pad 32: DVDD -> /fujinet/SD_SCK
- U1 pad 33: /rp2354b/SWCLK -> /fujinet/SD_MISO
- U1 pad 34: /rp2354b/SWDIO -> /fujinet/SD_CS
- U1 pad 35: /rp2354b/RUN -> /fujinet/SD_CD
- U1 pad 36: /IORQ_N -> /S3_RXD
- U1 pad 37: /RESET_N -> /S3_TXD
- U1 pad 38: /M1_N -> unconnected-(U1-IO2-Pad38)
- U1 pad 39: /CLK -> unconnected-(U1-IO1-Pad39)
- U1 pad 4: /A7 -> /RUN_CTL
- U1 pad 40: /PWR_OK -> GND
- U1 pad 41: +3V3_RP -> GND
- U1 pad 5: +3V3_RP -> /BOOTSEL_CTL
- U1 pad 6: /A8 -> unconnected-(U1-IO6-Pad6)
- U1 pad 7: /A9 -> unconnected-(U1-IO7-Pad7)
- U1 pad 8: /A10 -> unconnected-(U1-IO15-Pad8)
- U1 pad 9: /A11 -> unconnected-(U1-IO16-Pad9)
- U10 pad 1: unconnected-(U10-~{DCD}-Pad1) -> /cart-bus/A11
- U10 pad 10: unconnected-(U10-NC-Pad10) -> /cart-bus/SA16
- U10 pad 11: unconnected-(U10-~{SUSPEND}-Pad11) -> /cart-bus/SA14
- U10 pad 12: unconnected-(U10-SUSPEND-Pad12) -> /cart-bus/A12
- U10 pad 13: unconnected-(U10-CHREN-Pad13) -> /cart-bus/A7
- U10 pad 14: unconnected-(U10-CHR1-Pad14) -> /cart-bus/A6
- U10 pad 15: unconnected-(U10-CHR0-Pad15) -> /cart-bus/A5
- U10 pad 16: unconnected-(U10-~{WAKEUP}/GPIO.3-Pad16) -> /cart-bus/A4
- U10 pad 17: unconnected-(U10-RS485/GPIO.2-Pad17) -> /cart-bus/A3
- U10 pad 18: unconnected-(U10-~{RXT}/GPIO.1-Pad18) -> /cart-bus/A2
- U10 pad 19: unconnected-(U10-~{TXT}/GPIO.0-Pad19) -> /cart-bus/A1
- U10 pad 2: unconnected-(U10-~{RI}/CLK-Pad2) -> /cart-bus/A9
- U10 pad 20: unconnected-(U10-GPIO.6-Pad20) -> /cart-bus/A0
- U10 pad 21: unconnected-(U10-GPIO.5-Pad21) -> /cart-bus/D0
- U10 pad 22: unconnected-(U10-GPIO.4-Pad22) -> /cart-bus/D1
- U10 pad 23: GND -> /cart-bus/D2
- U10 pad 24: /usb-uart/UART_RTS -> GND
- U10 pad 25: /S3_TXD -> /cart-bus/D3
- U10 pad 26: /S3_RXD -> /cart-bus/D4
- U10 pad 27: unconnected-(U10-~{DSR}-Pad27) -> /cart-bus/D5
- U10 pad 28: /usb-uart/UART_DTR -> /cart-bus/D6
- U10 pad 29: GND -> /cart-bus/D7
- U10 pad 3: GND -> /cart-bus/A8
- U10 pad 4: /usb-uart/UBRG_DP -> /cart-bus/SA13
- U10 pad 5: /usb-uart/UBRG_DM -> /cart-bus/SRAM_WE_N
- U10 pad 6: +3V3 -> /cart-bus/SA17
- U10 pad 7: +3V3 -> /cart-bus/SA15
- U10 pad 8: /usb-uart/VBUS_SNS -> +5V
- U10 pad 9: /usb-uart/CP_RST -> /cart-bus/SA18
- U11 pad 1: /usb-uart/UART_RTS -> /cart-bus/PWR_OK
- U11 pad 2: /usb-uart/UART_DTR -> /cart-bus/CE
- U11 pad 3: /S3_IO0 -> /cart-bus/CEP_N
- U11 pad 4: /usb-uart/UART_DTR -> /cart-bus/WIN8
- U11 pad 5: /usb-uart/UART_RTS -> /cart-bus/LOAD
- U11 pad 6: /S3_EN -> /cart-bus/LOADWIN_N
- U12 pad 1: +3V3 -> /cart-bus/VSENSE
- U12 pad 2: +5V -> /cart-bus/PWR_OK_N
- U12 pad 3: +5V -> /cart-bus/PWR_OK_N
- U12 pad 4: GND -> /cart-bus/PWR_OK
- U12 pad 5: /power/BUCK_SW -> /cart-bus/SA19
- U12 pad 6: /power/BUCK_BST -> /cart-bus/SA19_N
- U13 pad 1: +5V -> /cart-bus/CEP_N
- U13 pad 2: GND -> /cart-bus/RD_N
- U13 pad 3: +5V -> /cart-bus/A14
- U13 pad 4: unconnected-(U13-NC-Pad4) -> /cart-bus/A15_N
- U13 pad 5: +3V3_RP -> /cart-bus/A13
- U2 pad 1: /A11 -> unconnected-(U2-~{DCD}-Pad1)
- U2 pad 10: /SA16 -> unconnected-(U2-NC-Pad10)
- U2 pad 11: /SA14 -> unconnected-(U2-~{SUSPEND}-Pad11)
- U2 pad 12: /A12 -> unconnected-(U2-SUSPEND-Pad12)
- U2 pad 13: /A7 -> unconnected-(U2-CHREN-Pad13)
- U2 pad 14: /A6 -> unconnected-(U2-CHR1-Pad14)
- U2 pad 15: /A5 -> unconnected-(U2-CHR0-Pad15)
- U2 pad 16: /A4 -> unconnected-(U2-~{WAKEUP}/GPIO.3-Pad16)
- U2 pad 17: /A3 -> unconnected-(U2-RS485/GPIO.2-Pad17)
- U2 pad 18: /A2 -> unconnected-(U2-~{RXT}/GPIO.1-Pad18)
- U2 pad 19: /A1 -> unconnected-(U2-~{TXT}/GPIO.0-Pad19)
- U2 pad 2: /A9 -> unconnected-(U2-~{RI}/CLK-Pad2)
- U2 pad 20: /A0 -> unconnected-(U2-GPIO.6-Pad20)
- U2 pad 21: /D0 -> unconnected-(U2-GPIO.5-Pad21)
- U2 pad 22: /D1 -> unconnected-(U2-GPIO.4-Pad22)
- U2 pad 23: /D2 -> GND
- U2 pad 24: GND -> /usb/UART_RTS
- U2 pad 25: /D3 -> /S3_TXD
- U2 pad 26: /D4 -> /S3_RXD
- U2 pad 27: /D5 -> unconnected-(U2-~{DSR}-Pad27)
- U2 pad 28: /D6 -> /usb/UART_DTR
- U2 pad 29: /D7 -> GND
- U2 pad 3: /A8 -> GND
- U2 pad 4: /SA13 -> /usb/UBRG_DP
- U2 pad 5: /SRAM_WE_N -> /usb/UBRG_DM
- U2 pad 6: /SA17 -> +3V3
- U2 pad 7: /SA15 -> +3V3
- U2 pad 8: +5V -> /usb/VBUS_SNS
- U2 pad 9: /SA18 -> /usb/CP_RST
- U3 pad 1: /A11 -> /usb/UART_RTS
- U3 pad 2: /A9 -> /usb/UART_DTR
- U3 pad 3: /A8 -> /S3_IO0
- U3 pad 4: /SA13 -> /usb/UART_DTR
- U3 pad 5: /SRAM_WE_N -> /usb/UART_RTS
- U3 pad 6: /SA17 -> /S3_EN
- U4 pad 1: /glue/VSENSE -> /cart-bus/A4
- U4 pad 10: /glue/A15_N -> DVDD
- U4 pad 11: /A15 -> /cart-bus/A12
- U4 pad 12: /glue/MBA -> /cart-bus/A13
- U4 pad 13: /glue/MBA_N -> /cart-bus/A14
- U4 pad 14: +5V -> /cart-bus/A15
- U4 pad 2: /glue/PWR_OK_N -> /cart-bus/A5
- U4 pad 3: /glue/PWR_OK_N -> /cart-bus/A6
- U4 pad 4: /PWR_OK -> /cart-bus/A7
- U4 pad 5: /SA19 -> +3V3_RP
- U4 pad 6: /SA19_N -> /cart-bus/A8
- U4 pad 7: GND -> /cart-bus/A9
- U4 pad 8: /glue/CE -> /cart-bus/A10
- U4 pad 9: /CE_N -> /cart-bus/A11
- U5 pad 1: /glue/CEP_N -> +3V3
- U5 pad 2: /glue/LOADWIN_N -> +5V
- U5 pad 3: /glue/CEP_N -> +5V
- U5 pad 4: /glue/RAMWIN_N -> GND
- U5 pad 5: /WR_N -> /power/BUCK_SW
- U5 pad 6: /glue/WE_RAM -> /power/BUCK_BST
- U6 pad 1: /glue/CEP_N -> +5V
- U6 pad 2: /RD_N -> GND
- U6 pad 3: /A14 -> +5V
- U6 pad 4: /glue/A15_N -> unconnected-(U6-NC-Pad4)
- U6 pad 5: /A13 -> +3V3_RP
- U7 pad 1: /MBOX -> /cart-bus/A11
- U7 pad 10: /GAME -> /cart-bus/SA16
- U7 pad 11: /glue/RD_CEP -> /cart-bus/SA14
- U7 pad 12: /glue/MBA_N -> /cart-bus/A12
- U7 pad 13: /A12 -> /cart-bus/A7
- U7 pad 14: +5V -> /cart-bus/A6
- U7 pad 2: /A13 -> /cart-bus/A9
- U7 pad 3: /RAM_WE -> /cart-bus/A8
- U7 pad 4: /glue/SLOT2_NM -> /cart-bus/SA13
- U7 pad 5: +5V -> /cart-bus/SRAM_WE_N
- U7 pad 6: /glue/RAMWIN_N -> /cart-bus/SA17
- U7 pad 7: GND -> /cart-bus/SA15
- U7 pad 8: /SRAM_OE_N -> +5V
- U7 pad 9: /glue/OE_ADDR -> /cart-bus/SA18
- U8 pad 1: /PWR_OK -> /cart-bus/MBOX
- U8 pad 10: /glue/SLOT2_NM -> /cart-bus/GAME
- U8 pad 11: /glue/OE_ADDR -> /cart-bus/RD_CEP
- U8 pad 12: /glue/SLOT2_NM_N -> /cart-bus/MBA_N
- U8 pad 13: /A15 -> /cart-bus/A12
- U8 pad 2: /glue/CE -> /cart-bus/A13
- U8 pad 3: /glue/CEP_N -> /cart-bus/RAM_WE
- U8 pad 4: /glue/WIN8 -> /cart-bus/SLOT2_NM
- U8 pad 5: /LOAD -> +5V
- U8 pad 6: /glue/LOADWIN_N -> /cart-bus/RAMWIN_N
- U8 pad 8: /glue/SLOT2_NM_N -> /cart-bus/SRAM_OE_N
- U8 pad 9: /glue/SLOT2_NM -> /cart-bus/OE_ADDR
- U9 pad 1: GND -> /cart-bus/CEP_N
- U9 pad 10: unconnected-(U9-IO17-Pad10) -> GND
- U9 pad 11: unconnected-(U9-IO18-Pad11) -> /cart-bus/WE_RAM
- U9 pad 12: unconnected-(U9-IO8-Pad12) -> /cart-bus/WE_LOAD
- U9 pad 13: /USB_DM -> /cart-bus/RD_N
- U9 pad 14: /USB_DP -> +5V
- U9 pad 2: +3V3 -> /cart-bus/LOADWIN_N
- U9 pad 3: /S3_EN -> /cart-bus/CEP_N
- U9 pad 4: /RUN_CTL -> /cart-bus/RAMWIN_N
- U9 pad 5: /BOOTSEL_CTL -> /cart-bus/WR_N
- U9 pad 6: unconnected-(U9-IO6-Pad6) -> /cart-bus/WE_RAM
- U9 pad 7: unconnected-(U9-IO7-Pad7) -> GND
- U9 pad 8: unconnected-(U9-IO15-Pad8) -> /cart-bus/SRAM_WE_N
- U9 pad 9: unconnected-(U9-IO16-Pad9) -> /cart-bus/WE_LOAD
- Y1 pad 1: /rp2354b/XIN -> /rp-core/XIN
- Y1 pad 3: /rp2354b/XOUT_Y -> /rp-core/XOUT_Y
Routing:
- net /S3_EN: track 152.3 -> 0.00 mm, vias 5 -> 0
- net VBUS: track 121.5 -> 0.00 mm, vias 3 -> 0
- net /A15: track 116.8 -> 0.00 mm, vias 3 -> 0
- net /A12: track 103.9 -> 0.00 mm, vias 5 -> 0
- net CONS_5V: track 108.1 -> 13.4 mm, vias 5 -> 0
- net /RD_N: track 94.4 -> 0.00 mm, vias 5 -> 0
- net /S3_IO0: track 94.1 -> 0.00 mm, vias 2 -> 0
- net /A7: track 93.4 -> 0.00 mm, vias 3 -> 0
- net /A11: track 93.2 -> 0.00 mm, vias 5 -> 0
- net /A2: track 92.6 -> 0.00 mm, vias 4 -> 0
- net /SA19: track 92.2 -> 0.00 mm, vias 3 -> 0
- net /A5: track 88.6 -> 0.00 mm, vias 3 -> 0
- net /A8: track 88.1 -> 0.00 mm, vias 6 -> 0
- net /A13: track 87.5 -> 0.00 mm, vias 3 -> 0
- net /A1: track 86.0 -> 0.00 mm, vias 4 -> 0
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- removed copper zone on B.Cu, net GND
- removed copper zone on F.Cu, net GND

Commit message: SMS Rev0 v2: route the co-designed board, fab packages for JLCPCB and PCBWay
The board is the best of six routing variants (12/16/20 passes; hybrid,
global and greedy strategies; two pre-route sets).  All six plateaued
at 46-50 Freerouting "unrouted" by pass 8, most of them plane
connections that KiCad's zones make.  12 passes greedy left KiCad 2
links (A12, QSPI_SS), and the finisher closed them.

The routed board has 1951 segments, 6055 mm of track and 743 vias, 271
of them GND stitching.  KiCad DRC with schematic parity at every
severity is 0 / 0 / 0 against the redrawn schematic, and check_vias is
clean.  Every footprint sits exactly where placement.py puts it, so the
mirror check holds on the routed board, and the references are still
geographic.

Changes:
- The board title moves to a clear spot above the edge; the old spot
  overlapped R14, R15 and C18 in the new floorplan.  Both spots were
  found by rasterising the routed board and live in placement.py.
- fix_silk.py adds a bold pin-1 dot on each AS6C4008 (U7, U10), the
  parts JLC places without an EasyEDA footprint.
- export.py:
  - the JLC zip's F.Silkscreen carries JLCJLCJLCJLC at
    placement.JLC_ORDER; the PCBWay zip does not;
  - consigned.csv lists the lines JLC does not stock;
  - ORDER-JLCPCB.md and ORDER-PCBWay.md give the order step by step,
    with references taken from design.py.
- New tools/audit/check_fab.py checks:
  - designator sets: BOM = CPL = centroid = the board;
  - LCSC codes, MPNs and manufacturers;
  - CPL positions and rotations, recomputed from the measured offsets;
  - the centroid, unmodified;
  - the drill count, including the USB-C G85 slots;
  - that the order-number spot is clear and its text is present only in
    the JLC zip;
  - check_gerbers.
- New tools/audit/sourcing.py writes docs/sourcing.md from jlcsearch and
  LCSC: 42 of 45 lines are stocked for 5 boards, about USD 29 of parts
  per board.  The SRAMs and the Nexperia '27 / '10 are to be consigned,
  bought thro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
Routing:
- net /S3_EN: track 0.00 -> 135.4 mm, vias 0 -> 2
- net /cart-bus/A15: track 6.70 -> 114.5 mm, vias 0 -> 6
- net VBUS: track 0.00 -> 101.7 mm, vias 0 -> 2
- net /S3_IO0: track 0.00 -> 98.7 mm, vias 0 -> 2
- net /rp-core/RUN: track 0.00 -> 95.6 mm, vias 0 -> 5
- net /cart-bus/D6: track 17.9 -> 102.1 mm, vias 1 -> 3
- net /cart-bus/SA19: track 4.80 -> 87.7 mm, vias 1 -> 4
- net CONS_5V: track 13.4 -> 96.0 mm, vias 0 -> 2
- net /cart-bus/RD_N: track 6.70 -> 89.0 mm, vias 0 -> 5
- net /cart-bus/D1: track 17.1 -> 95.0 mm, vias 1 -> 4
- net /cart-bus/SRAM_WE_N: track 0.00 -> 76.8 mm, vias 0 -> 4
- net /cart-bus/A1: track 16.7 -> 90.1 mm, vias 0 -> 3
- net /cart-bus/RESET_N: track 6.70 -> 80.0 mm, vias 0 -> 2
- net /cart-bus/A0: track 17.7 -> 90.8 mm, vias 1 -> 3
- net /cart-bus/A14: track 6.70 -> 78.5 mm, vias 0 -> 4
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- added copper zone on B.Cu, net GND
- added copper zone on F.Cu, net GND
