File: Fairchild-Channel-F/FujiNet-ChannelF-Rev0/cart-rp.kicad_sch (KiCad schematic)
At the start: 52 parts, among them J1 ChannelF_Cart_Edge_22, Q1 2N7002, SW1 BOOTSEL, SW2 RESET, U1 RP2040, U2 SN74LVC4245APWR, U3 SN74LVC4245APWR, U4 W25Q16JVSSIQ, Y1 12MHz

Commit message: channel f pcb (#56)
Parts:
- removed C1, C10, C11, C12, C2, C3, C4, C5, C6, C7, C8, C9: 100nF, FujiNet-ChannelF:C_0603_1608Metric, symbol Device:C
- removed C13, C15: 1uF, FujiNet-ChannelF:C_0603_1608Metric, symbol Device:C
- removed C14: 10uF, FujiNet-ChannelF:C_0603_1608Metric, symbol Device:C
- removed D1: green, FujiNet-ChannelF:LED_0603_1608Metric, symbol Device:LED
- removed R1: 4.7k, FujiNet-ChannelF:R_0603_1608Metric, symbol Device:R
- removed R2, R9: 10k, FujiNet-ChannelF:R_0603_1608Metric, symbol Device:R
- removed R3: 100k, FujiNet-ChannelF:R_0603_1608Metric, symbol Device:R
- removed R4: 330R, FujiNet-ChannelF:R_0603_1608Metric, symbol Device:R
- removed R5, R7, R8: 1k, FujiNet-ChannelF:R_0603_1608Metric, symbol Device:R
- removed SW2: RESET, FujiNet-ChannelF:SW_SPST_TL3342, symbol Switch:SW_Push
- removed TP1: DIR, FujiNet-ChannelF:TestPoint_Pad_D1.5mm, symbol Connector:TestPoint
- removed TP3: PHI, FujiNet-ChannelF:TestPoint_Pad_D1.5mm, symbol Connector:TestPoint
- removed TP8: RUN, FujiNet-ChannelF:TestPoint_Pad_D1.5mm, symbol Connector:TestPoint
- removed U1: RP2040, FujiNet-ChannelF:QFN-56-1EP_7x7mm_P0.4mm_EP3.2x3.2mm, symbol FujiNet-ChannelF:RP2040_Fn
- removed U2, U3: SN74LVC4245APWR, FujiNet-ChannelF:TSSOP-24_4.4x7.8mm_P0.65mm, symbol FujiNet-ChannelF:SN74LVC4245A
- removed U4: W25Q16JVSSIQ, FujiNet-ChannelF:SOIC-8_5.3x5.3mm_P1.27mm, symbol Memory_Flash:W25Q16JVSS
- added C21, C24, C25, C26, C27, C28, C31, C32, C34, C35, C37, C38: 100nF, FujiNet-ChannelF:C_0603_1608Metric, symbol Device:C
- added C22, C29: 15pF, FujiNet-ChannelF:C_0603_1608Metric, symbol Device:C
- added C23: 10uF, FujiNet-ChannelF:C_0603_1608Metric, symbol Device:C
- added D3: green, FujiNet-ChannelF:LED_0603_1608Metric, symbol Device:LED
- added R13, R15, R20: 10k, FujiNet-ChannelF:R_0603_1608Metric, symbol Device:R
- added R14, R16, R17: 1k, FujiNet-ChannelF:R_0603_1608Metric, symbol Device:R
- added R18: 4.7k, FujiNet-ChannelF:R_0603_1608Metric, symbol Device:R
- added R19: 100k, FujiNet-ChannelF:R_0603_1608Metric, symbol Device:R
- added SW4: BOOTSEL, FujiNet-ChannelF:SW_SPST_TL3342, symbol Switch:SW_Push
- added TP10: WRITE, FujiNet-ChannelF:TestPoint_Pad_D1.5mm, symbol Connector:TestPoint
- added TP11: PHI, FujiNet-ChannelF:TestPoint_Pad_D1.5mm, symbol Connector:TestPoint
- added TP12: DIR, FujiNet-ChannelF:TestPoint_Pad_D1.5mm, symbol Connector:TestPoint
- added U5: RP2040, FujiNet-ChannelF:QFN-56-1EP_7x7mm_P0.4mm_EP3.2x3.2mm, symbol FujiNet-ChannelF:RP2040_Fn
- added U6: W25Q16JVSSIQ, FujiNet-ChannelF:SOIC-8_5.3x5.3mm_P1.27mm, symbol Memory_Flash:W25Q16JVSS
- added U8, U9: SN74LVC4245APWR, FujiNet-ChannelF:TSSOP-24_4.4x7.8mm_P0.65mm, symbol FujiNet-ChannelF:SN74LVC4245A
- C16, C17: Manufacturer (none) -> YAGEO
- C18: value 100nF -> 1uF; LCSC C14663 -> C15849; MPN CC0603KRX7R9BB104 -> CL10A105KB8NNNC; Manufacturer (none) -> Samsung Electro-Mechanics
- C19: value 15pF -> 1uF; LCSC C1644 -> C15849; MPN CL10C150JB8NNNC -> CL10A105KB8NNNC; Manufacturer (none) -> Samsung Electro-Mechanics
- C20: value 15pF -> 100nF; LCSC C1644 -> C14663; MPN CL10C150JB8NNNC -> CC0603KRX7R9BB104; Manufacturer (none) -> YAGEO
- D2: Manufacturer (none) -> Nexperia
- J1: footprint (none) -> FujiNet-ChannelF:ChannelF_Videocart_Edge_22
- Q1: Manufacturer (none) -> Jiangsu Changjing (JSCJ)
- R10, R11, R12: Manufacturer (none) -> UNI-ROYAL
- R6: value 10k -> 330R; LCSC C25804 -> C23138; MPN 0603WAF1002T5E -> 0603WAF3300T5E; Manufacturer (none) -> UNI-ROYAL
- SW1: value BOOTSEL -> RESET; Manufacturer (none) -> E-Switch
- TP2: value WRITE -> GP17
- TP4: value GP17 -> RUN
- TP5: value SWCLK -> SWDIO
- TP6: value SWDIO -> SWCLK
- Y1: Manufacturer (none) -> Abracon
Connections:
- net +3V3_RP: now also C20.1, C21.1, C23.1, C24.1, C25.1, C26.1, C27.1, C28.1, C31.1, C32.1, C34.1, C35.1, R13.1, R15.1, R18.1, U5.1 (IOVDD), U5.10 (IOVDD), U5.22 (IOVDD), U5.33 (IOVDD), U5.42 (IOVDD), U5.43 (ADC_AVDD), U5.44 (VREG_VIN), U5.48 (USB_VDD), U5.49 (IOVDD), U6.8 (VCC), U8.23 (V_{CCB}), U8.24 (V_{CCB}), U9.23 (V_{CCB}), U9.24 (V_{CCB}); no longer R6.1
- net BOOTSEL_BTN: now also R16.2, SW4.1; no longer SW1.1
- net BOOTSEL_CTL: now also R17.1
- net CBUF_A8: now also R20.1, U9.10 (A8)
- net CONS_5V: now also C37.1, C38.1, U8.1 (V_{CCA}), U9.1 (V_{CCA}), U9.2 (DIR)
- net D0: now also U8.3 (A1)
- net D1: now also U8.4 (A2)
- net D2: now also U8.5 (A3)
- net D3: now also U8.6 (A4)
- net D4: now also U8.7 (A5)
- net D5: now also U8.8 (A6)
- net D6: now also U8.9 (A7)
- net D7: now also U8.10 (A8)
- net DVDD: now also C19.1, U5.23 (DVDD), U5.45 (VREG_VOUT), U5.50 (DVDD)
- net GND: now also C21.2, C22.2, C23.2, C24.2, C25.2, C26.2, C27.2, C28.2, C29.2, C31.2, C32.2, C34.2, C35.2, C37.2, C38.2, D3.1 (K), R19.2, R20.2, SW4.2, U5.19 (TESTEN), U5.57 (GND), U6.4 (GND), U8.11 (GND), U8.12 (GND), U8.13 (GND), U8.22 (~{OE}), U9.11 (GND), U9.12 (GND), U9.13 (GND), U9.22 (~{OE})
- net PHI: now also U9.9 (A7)
- net QSPI_SCLK: now also U5.52 (QSPI_SCLK), U6.6 (CLK)
- net QSPI_SD0: now also U5.53 (QSPI_SD0), U6.5 (DI/IO_{0})
- net QSPI_SD1: now also U5.55 (QSPI_SD1), U6.2 (DO/IO_{1})
- net QSPI_SD2: now also U5.54 (QSPI_SD2), U6.3 (~{WP}/IO_{2})
- net QSPI_SD3: now also U5.51 (QSPI_SD3), U6.7 (~{HOLD}/~{RESET}/IO_{3})
- net QSPI_SS: now also R15.2, R16.1, R17.2, U5.56 (~{QSPI_SS}), U6.1 (~{CS}); no longer R6.2
- net ROMC0: now also U9.3 (A1)
- net ROMC1: now also U9.4 (A2)
- net ROMC2: now also U9.5 (A3)
- net ROMC3: now also U9.6 (A4)
- net ROMC4: now also U9.7 (A5)
- net RP_D0: now also U5.2 (GPIO0), U8.21 (B1)
- net RP_D1: now also U5.3 (GPIO1), U8.20 (B2)
- net RP_D2: now also U5.4 (GPIO2), U8.19 (B3)
- net RP_D3: now also U5.5 (GPIO3), U8.18 (B4)
- net RP_D4: now also U5.6 (GPIO4), U8.17 (B5)
- net RP_D5: now also U5.7 (GPIO5), U8.16 (B6)
- net RP_D6: now also U5.8 (GPIO6), U8.15 (B7)
- net RP_D7: now also U5.9 (GPIO7), U8.14 (B8)
- net RP_DIR: now also R18.2, TP12.1, U5.18 (GPIO15), U8.2 (DIR)
- net RP_GP17: now also TP2.1, U5.28 (GPIO17); no longer TP4.1
- net RP_INTREQ: now also R19.1, U5.27 (GPIO16)
- net RP_LED: now also R6.1, U5.37 (GPIO25)
- net RP_LED_A: now also R6.2, D3.2 (A)
- net RP_PHI: now also TP11.1, U5.17 (GPIO14), U9.15 (B7)
- net RP_ROMC0: now also U5.11 (GPIO8), U9.21 (B1)
- net RP_ROMC1: now also U5.12 (GPIO9), U9.20 (B2)
- net RP_ROMC2: now also U5.13 (GPIO10), U9.19 (B3)
- net RP_ROMC3: now also U5.14 (GPIO11), U9.18 (B4)
- net RP_ROMC4: now also U5.15 (GPIO12), U9.17 (B5)
- net RP_USB_DM: now also U5.46 (USB_DM)
- net RP_USB_DP: now also U5.47 (USB_DP)
- net RP_WRITE: now also TP10.1, U5.16 (GPIO13), U9.16 (B6); no longer TP2.1
- net RST_BTN: now also SW1.1
- net RUN: now also TP4.1, R13.2, U5.26 (RUN)
- net SWCLK: now also TP6.1, U5.24 (SWCLK); no longer TP5.1
- net SWDIO: now also TP5.1, U5.25 (SWDIO); no longer TP6.1
- net WRITE: now also U9.8 (A6)
- net XIN: now also C29.1, U5.20 (XIN); no longer C19.1
- net XOUT: now also R14.1, U5.21 (XOUT)
- net XOUT_Y: now also C22.1, R14.2; no longer C20.1
Other:
- note added: "The Fairchild Channel F Videocart edge, 22 contacts (channelf.se veswiki Pinouts): the F8 bus has NO address bus -- D0-D7, five ROMC lines, WRITE (one machine cycle per pulse) and PHI -- and no reset line (a console reset arrives as ROMC 08). +12V (22) and NC (21) are left open. U8 / U9 SN74LVC4245A: A port on CONS_5V (TTL inputs, VIH 2.0 V; drives 5 V levels -- the F3850 data bus wants VIH 2.9 V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"
- note removed: "The Fairchild Channel F Videocart edge, 22 contacts (channelf.se veswiki Pinouts): the F8 bus has NO address bus -- D0-D7, five ROMC lines, WRITE (one machine cycle per pulse) and PHI -- and no reset line (a console reset arrives as ROMC 08). +12V (22) and NC (21) are left open. U2 / U3 SN74LVC4245A: A port on CONS_5V (TTL inputs, VIH 2.0 V; drives 5 V levels -- the F3850 data bus wants VIH 2.9 V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"
- moved on the sheet: C18, C19, C20, R6, SW1, TP2, TP4, TP5, TP6
