File: Fairchild-Channel-F/FujiNet-ChannelF-Rev0/fujinet.kicad_sch (KiCad schematic)
At the start: 14 parts, among them J2 microSD, SW3 S3_RST, SW4 S3_BOOT, U5 ESP32-S3-WROOM-1-N16R8

Commit message: channel f pcb (#56)
Parts:
- removed C21: 22uF, FujiNet-ChannelF:C_0805_2012Metric, symbol Device:C
- removed C22, C25: 100nF, FujiNet-ChannelF:C_0603_1608Metric, symbol Device:C
- removed C23: 1uF, FujiNet-ChannelF:C_0603_1608Metric, symbol Device:C
- removed C24: 10uF, FujiNet-ChannelF:C_0603_1608Metric, symbol Device:C
- removed D3: WS2812B-2020-V6, FujiNet-ChannelF:LED_WS2812B-2020_PLCC4_2.0x2.0mm, symbol LED:WS2812B-2020
- removed J2: microSD, FujiNet-ChannelF:TF-SMD_TF-015, symbol FujiNet-ChannelF:MicroSD_TF015
- removed R13, R14: 10k, FujiNet-ChannelF:R_0603_1608Metric, symbol Device:R
- removed R15: 330R, FujiNet-ChannelF:R_0603_1608Metric, symbol Device:R
- removed SW4: S3_BOOT, FujiNet-ChannelF:SW_SPST_TL3342, symbol Switch:SW_Push
- removed U5: ESP32-S3-WROOM-1-N16R8, FujiNet-ChannelF:ESP32-S3-WROOM-1, symbol FujiNet-ChannelF:ESP32-S3-WROOM-1_Fn
- added C1: 22uF, FujiNet-ChannelF:C_0805_2012Metric, symbol Device:C
- added C2, C3: 100nF, FujiNet-ChannelF:C_0603_1608Metric, symbol Device:C
- added C4: 10uF, FujiNet-ChannelF:C_0603_1608Metric, symbol Device:C
- added C7: 1uF, FujiNet-ChannelF:C_0603_1608Metric, symbol Device:C
- added D1: WS2812B-2020-V6, FujiNet-ChannelF:LED_WS2812B-2020_PLCC4_2.0x2.0mm, symbol LED:WS2812B-2020
- added J3: microSD, FujiNet-ChannelF:TF-SMD_TF-015, symbol FujiNet-ChannelF:MicroSD_TF015
- added R1, R2: 10k, FujiNet-ChannelF:R_0603_1608Metric, symbol Device:R
- added R5: 330R, FujiNet-ChannelF:R_0603_1608Metric, symbol Device:R
- added SW2: S3_RST, FujiNet-ChannelF:SW_SPST_TL3342, symbol Switch:SW_Push
- added U1: ESP32-S3-WROOM-1-N16R8, FujiNet-ChannelF:ESP32-S3-WROOM-1, symbol FujiNet-ChannelF:ESP32-S3-WROOM-1_Fn
- RN1: Manufacturer (none) -> UNI-ROYAL
- SW3: value S3_RST -> S3_BOOT; Manufacturer (none) -> E-Switch
Connections:
- net +3V3: now also C1.1, C2.1, C4.1, J3.4 (VDD), R1.1, R2.1, U1.2 (3V3)
- net +5V: now also C3.1, D1.4 (VDD)
- net BOOTSEL_CTL: now also U1.5 (IO5)
- net GND: now also C1.2, C2.2, C3.2, C4.2, C7.2, D1.2 (VSS), J3.10 (SH), J3.11 (SH), J3.12 (SH), J3.13 (SH), J3.6 (VSS), SW2.2, U1.1 (GND), U1.40 (GND), U1.41 (GND)
- net LED_STRIP: now also R5.1, U1.25 (IO48)
- net RUN_CTL: now also U1.4 (IO4)
- net S3_EN: now also C7.1, R1.2, SW2.1, U1.3 (EN); no longer SW3.1
- net S3_IO0: now also SW3.1, U1.27 (IO0)
- net S3_RXD: now also U1.36 (RXD0)
- net S3_TXD: now also U1.37 (TXD0)
- net SD_CD: now also J3.9 (CD), R2.2, U1.35 (IO42)
- net SD_CS: now also J3.2 (DAT3/CS), U1.34 (IO41)
- net SD_DAT1: now also J3.8 (DAT1)
- net SD_DAT2: now also J3.1 (DAT2)
- net SD_MISO: now also J3.7 (DAT0/DO), U1.33 (IO40)
- net SD_MOSI: now also J3.3 (CMD/DI), U1.31 (IO38)
- net SD_SCK: now also J3.5 (CLK), U1.32 (IO39)
- net USB_DM: now also U1.13 (USB_D-)
- net USB_DP: now also U1.14 (USB_D+)
- net WS_DIN: now also D1.3 (DIN), R5.2
Other:
- moved on the sheet: SW3
Changed lines of the file:
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@@
 		(on_board yes)
 		(dnp no)
-		(property "Reference" "U5"
+		(property "Reference" "U1"
 			(at 200.66 87.122 0)
 			(effects
@@
 		)
 		(property "MPN" "ESP32-S3-WROOM-1-N16R8"
+			(at 228.6 124.46 0)
+			(effects
+				(font
+					(size 1.27 1.27)
+				)
+				(hide yes)
+			)
+		)
+		(property "Manufacturer" "Espressif"
 			(at 228.6 124.46 0)
 			(effects
@@
 			(project "FujiNet-ChannelF-Rev0"
 				(path "/94e41297-bf02-5fe3-9e3f-23dd2de0dc13/cdbe3c56-ac67-5d32-b622-767fbe1f06b4"
-					(reference "U5")
+					(reference "U1")
 					(unit 1)
 				)
@@
 		(on_board yes)
 		(dnp no)
-		(property "Reference" "C22"
+		(property "Reference" "C2"
 			(at 244.602 73.66 0)
 			(effects
@@
 		)
 		(property "MPN" "CC0603KRX7R9BB104"
+			(at 241.3 74.93 0)
+			(effects
+				(font
+					(size 1.27 1.27)
+				)
+				(hide yes)
+			)
+		)
+		(property "Manufacturer" "YAGEO"
 			(at 241.3 74.93 0)
 			(effects
@@
 			(project "FujiNet-ChannelF-Rev0"
 				(path "/94e41297-bf02-5fe3-9e3f-23dd2de0dc13/cdbe3c56-ac67-5d32-b622-767fbe1f06b4"
-					(reference "C22")
+					(reference "C2")
 					(unit 1)
 				)
@@
 		(on_board yes)
 		(dnp no)
-		(property "Reference" "C21"
+		(property "Reference" "C1"
 			(at 257.302 73.66 0)
 			(effects
@@
 		)
 		(property "MPN" "CL21A226MAQNNNE"
+			(at 254 74.93 0)
+			(effects
+				(font
+					(size 1.27 1.27)
+				)
+				(hide yes)
+			)
+		)
+		(property "Manufacturer" "Samsung Electro-Mechanics"
 			(at 254 74.93 0)
 			(effects
@@
 			(project "FujiNet-ChannelF-Rev0"
 				(path "/94e41297-bf02-5fe3-9e3f-23dd2de0dc13/cdbe3c56-ac67-5d32-b622-767fbe1f06b4"
-					(reference "C21")
+					(reference "C1")
 					(unit 1)
 				)
@@
 		(on_board yes)
 		(dnp no)
-		(property "Reference" "R13"
+		(property "Reference" "R1"
 			(at 213.106 60.96 0)
 			(effects
@@
 		)
 		(property "MPN" "0603WAF1002T5E"
+			(at 210.82 62.23 0)
+			(effects
+				(font
+					(size 1.27 1.27)
+				)
+				(hide yes)
+			)
+		)
+		(property "Manufacturer" "UNI-ROYAL"
 			(at 210.82 62.23 0)
 			(effects
@@
 			(project "FujiNet-ChannelF-Rev0"
 				(path "/94e41297-bf02-5fe3-9e3f-23dd2de0dc13/cdbe3c56-ac67-5d32-b622-767fbe1f06b4"
-					(reference "R13")
+					(reference "R1")
 					(unit 1)
 				)
@@
 		(on_board yes)
 		(dnp no)
-		(property "Reference" "C23"
+		(property "Reference" "C7"
 			(at 206.502 73.66 0)
 			(effects
@@
 		)
 		(property "MPN" "CL10A105KB8NNNC"
+			(at 203.2 74.93 0)
+			(effects
+				(font
+					(size 1.27 1.27)
+				)
+				(hide yes)
+			)
+		)
+		(property "Manufacturer" "Samsung Electro-Mechanics"
 			(at 203.2 74.93 0)
 			(effects
@@
 			(project "FujiNet-ChannelF-Rev0"
 				(path "/94e41297-bf02-5fe3-9e3f-23dd2de0dc13/cdbe3c56-ac67-5d32-b622-767fbe1f06b4"
-					(reference "C23")
+					(reference "C7")
 					(unit 1)
 				)
@@
 		(on_board yes)
 		(dnp no)
-		(property "Reference" "SW3"
+		(property "Reference" "SW2"
 			(at 156.718 74.93 90)
 			(effects
@@
 		)
 		(property "MPN" "TL3342F160QG"
+			(at 152.4 76.2 90)
+			(effects
+				(font
+					(size 1.27 1.27)
+				)
+				(hide yes)
+			)
+		)
+		(property "Manufacturer" "E-Switch"
 			(at 152.4 76.2 90)
 			(effects
@@
 			(project "FujiNet-ChannelF-Rev0"
 				(path "/94e41297-bf02-5fe3-9e3f-23dd2de0dc13/cdbe3c56-ac67-5d32-b622-767fbe1f06b4"
-					(reference "SW3")
+					(reference "SW2")
 					(unit 1)
 				)
@@
 		(on_board yes)
 		(dnp no)
-		(property "Reference" "SW4"
+		(property "Reference" "SW3"
 			(at 144.018 113.03 90)
 			(effects
@@
 		)
 		(property "MPN" "TL3342F160QG"
+			(at 139.7 114.3 90)
+			(effects
+				(font
+					(size 1.27 1.27)
+				)
+				(hide yes)
+			)
+		)
+		(property "Manufacturer" "E-Switch"
 			(at 139.7 114.3 90)
 			(effects
@@
 			(project "FujiNet-ChannelF-Rev0"
 				(path "/94e41297-bf02-5fe3-9e3f-23dd2de0dc13/cdbe3c56-ac67-5d32-b622-767fbe1f06b4"
-					(reference "SW4")
+					(reference "SW3")
 					(unit 1)
 				)
@@
 		(on_board yes)
 		(dnp no)
-		(property "Reference" "J2"
+		(property "Reference" "J3"
 			(at 284.48 170.942 0)
 			(effects
@@
 		)
 		(property "MPN" "TF-015"
+			(at 294.64 193.04 0)
+			(effects
+				(font
+					(size 1.27 1.27)
+				)
+				(hide yes)
+			)
+		)
+		(property "Manufacturer" "SOFNG"
 			(at 294.64 193.04 0)
 			(effects
@@
 			(project "FujiNet-ChannelF-Rev0"
 				(path "/94e41297-bf02-5fe3-9e3f-23dd2de0dc13/cdbe3c56-ac67-5d32-b622-767fbe1f06b4"
-					(reference "J2")
+					(reference "J3")
 					(unit 1)
 				)
@@
 		(on_board yes)
 		(dnp no)
-		(property "Reference" "R14"
+		(property "Reference" "R2"
 			(at 219.456 198.12 0)
 			(effects
@@
 		)
 		(property "MPN" "0603WAF1002T5E"
+			(at 217.17 199.39 0)
+			(effects
+				(font
+					(size 1.27 1.27)
+				)
+				(hide yes)
+			)
+		)
+		(property "Manufacturer" "UNI-ROYAL"
 			(at 217.17 199.39 0)
 			(effects
@@
 			(project "FujiNet-ChannelF-Rev0"
 				(path "/94e41297-bf02-5fe3-9e3f-23dd2de0dc13/cdbe3c56-ac67-5d32-b622-767fbe1f06b4"
-					(reference "R14")
+					(reference "R2")
 					(unit 1)
 				)
@@
 			)
 		)
+		(property "Manufacturer" "UNI-ROYAL"
+			(at 229.87 194.31 0)
+			(effects
+				(font
+					(size 1.27 1.27)
+				)
+				(hide yes)
+			)
+		)
 		(property "LCSC" "C29718"
 			(at 229.87 194.31 0)
@@
 			)
 		)
+		(property "Manufacturer" "UNI-ROYAL"
+			(at 240.03 189.23 0)
+			(effects
+				(font
+					(size 1.27 1.27)
+				)
+				(hide yes)
+			)
+		)
 		(property "LCSC" "C29718"
 			(at 240.03 189.23 0)
@@
 			)
 		)
+		(property "Manufacturer" "UNI-ROYAL"
+			(at 269.24 168.91 0)
+			(effects
+				(font
+					(size 1.27 1.27)
+				)
+				(hide yes)
+			)
+		)
 		(property "LCSC" "C29718"
 			(at 269.24 168.91 0)
@@
 			)
 		)
+		(property "Manufacturer" "UNI-ROYAL"
+			(at 261.62 173.99 0)
+			(effects
+				(font
+					(size 1.27 1.27)
+				)
+				(hide yes)
+			)
+		)
 		(property "LCSC" "C29718"
 			(at 261.62 173.99 0)
@@
 		(on_board yes)
 		(dnp no)
-		(property "Reference" "C24"
+		(property "Reference" "C4"
 			(at 271.018 218.44 0)
 			(effects
@@
 		)
 		(property "MPN" "CL10A106KP8NNNC"
+			(at 274.32 219.71 0)
+			(effects
+				(font
+					(size 1.27 1.27)
+				)
+				(hide yes)
+			)
+		)
+		(property "Manufacturer" "Samsung Electro-Mechanics"
 			(at 274.32 219.71 0)
 			(effects
@@
 			(project "FujiNet-ChannelF-Rev0"
 				(path "/94e41297-bf02-5fe3-9e3f-23dd2de0dc13/cdbe3c56-ac67-5d32-b622-767fbe1f06b4"
-					(reference "C24")
+					(reference "C4")
 					(unit 1)
 				)
@@
 		(on_board yes)
 		(dnp no)
-		(property "Reference" "R15"
+		(property "Reference" "R5"
 			(at 189.23 211.836 90)
 			(effects
@@
 		)
 		(property "MPN" "0603WAF3300T5E"
+			(at 189.23 217.17 90)
+			(effects
+				(font
+					(size 1.27 1.27)
+				)
+				(hide yes)
+			)
+		)
+		(property "Manufacturer" "UNI-ROYAL"
 			(at 189.23 217.17 90)
 			(effects
@@
 			(project "FujiNet-ChannelF-Rev0"
 				(path "/94e41297-bf02-5fe3-9e3f-23dd2de0dc13/cdbe3c56-ac67-5d32-b622-767fbe1f06b4"
-					(reference "R15")
+					(reference "R5")
 					(unit 1)
 				)
@@
 		(on_board yes)
 		(dnp no)
-		(property "Reference" "D3"
+		(property "Reference" "D1"
 			(at 168.91 220.98 0)
 			(effects
@@
 		)
 		(property "MPN" "WS2812B-2020-V6"
+			(at 162.56 217.17 0)
+			(effects
+				(font
+					(size 1.27 1.27)
+				)
+				(hide yes)
+			)
+		)
+		(property "Manufacturer" "Worldsemi"
 			(at 162.56 217.17 0)
 			(effects
@@
 			(project "FujiNet-ChannelF-Rev0"
 				(path "/94e41297-bf02-5fe3-9e3f-23dd2de0dc13/cdbe3c56-ac67-5d32-b622-767fbe1f06b4"
-					(reference "D3")
+					(reference "D1")
 					(unit 1)
 				)
@@
 		(on_board yes)
 		(dnp no)
-		(property "Reference" "C25"
+		(property "Reference" "C3"
 			(at 146.558 209.55 0)
 			(effects
@@
 		)
 		(property "MPN" "CC0603KRX7R9BB104"
+			(at 149.86 210.82 0)
+			(effects
+				(font
+					(size 1.27 1.27)
+				)
+				(hide yes)
+			)
+		)
+		(property "Manufacturer" "YAGEO"
 			(at 149.86 210.82 0)
 			(effects
@@
 			(project "FujiNet-ChannelF-Rev0"
 				(path "/94e41297-bf02-5fe3-9e3f-23dd2de0dc13/cdbe3c56-ac67-5d32-b622-767fbe1f06b4"
-					(reference "C25")
+					(reference "C3")
 					(unit 1)
 				)
