File: Fairchild-Channel-F/FujiNet-ChannelF-Rev0/power.kicad_sch (KiCad schematic)
At the start: 18 parts, among them U8 AP63203WU, U9 AP2112K-3.3

Commit message: channel f pcb (#56)
Parts:
- removed C31, C32, C37: 22uF, FujiNet-ChannelF:C_0805_2012Metric, symbol Device:C
- removed C34, C35: 100nF, FujiNet-ChannelF:C_0603_1608Metric, symbol Device:C
- removed C38: 1uF, FujiNet-ChannelF:C_0603_1608Metric, symbol Device:C
- removed TP10: +5V, FujiNet-ChannelF:TestPoint_Pad_D1.5mm, symbol Connector:TestPoint
- removed TP11: +3V3, FujiNet-ChannelF:TestPoint_Pad_D1.5mm, symbol Connector:TestPoint
- removed TP12: +3V3_RP, FujiNet-ChannelF:TestPoint_Pad_D1.5mm, symbol Connector:TestPoint
- removed U8: AP63203WU, FujiNet-ChannelF:TSOT-23-6, symbol Regulator_Switching:AP63203WU
- removed U9: AP2112K-3.3, FujiNet-ChannelF:SOT-23-5, symbol Regulator_Linear:AP2112K-3.3
- added C10, C11, C12, C15: 22uF, FujiNet-ChannelF:C_0805_2012Metric, symbol Device:C
- added C13, C14: 100nF, FujiNet-ChannelF:C_0603_1608Metric, symbol Device:C
- added TP1: +3V3, FujiNet-ChannelF:TestPoint_Pad_D1.5mm, symbol Connector:TestPoint
- added TP3: +3V3_RP, FujiNet-ChannelF:TestPoint_Pad_D1.5mm, symbol Connector:TestPoint
- added TP8: +5V, FujiNet-ChannelF:TestPoint_Pad_D1.5mm, symbol Connector:TestPoint
- added U4: AP63203WU, FujiNet-ChannelF:TSOT-23-6, symbol Regulator_Switching:AP63203WU
- added U7: AP2112K-3.3, FujiNet-ChannelF:SOT-23-5, symbol Regulator_Linear:AP2112K-3.3
- C30: value 100nF -> 1uF; LCSC C14663 -> C15849; MPN CC0603KRX7R9BB104 -> CL10A105KB8NNNC; Manufacturer (none) -> Samsung Electro-Mechanics
- C33: value 22uF -> 1uF; footprint FujiNet-ChannelF:C_0805_2012Metric -> FujiNet-ChannelF:C_0603_1608Metric; LCSC C45783 -> C15849; MPN CL21A226MAQNNNE -> CL10A105KB8NNNC; Manufacturer (none) -> Samsung Electro-Mechanics
- C36: Manufacturer (none) -> Samsung Electro-Mechanics
- C39: value 1uF -> 100nF; LCSC C15849 -> C14663; MPN CL10A105KB8NNNC -> CC0603KRX7R9BB104; Manufacturer (none) -> YAGEO
- D7, D8: Manufacturer (none) -> MDD (Microdiode Semiconductor)
- L1: Manufacturer (none) -> Sunlord
Connections:
- net +3V3: now also C10.1, C11.1, TP1.1, U4.1 (FB); no longer C36.1
- net +3V3_RP: now also C30.1, TP3.1, U7.5 (VOUT); no longer C39.1
- net +5V: now also C36.1, C12.1, C13.1, C15.1, TP8.1, U4.2 (EN), U4.3 (IN), U7.1 (VIN), U7.3 (EN)
- net BUCK_BST: now also C14.2, U4.6 (BST)
- net BUCK_SW: now also C14.1, U4.5 (SW)
- net CONS_5V: now also C39.1, D8.2 (A); no longer C30.1, D7.2 (A)
- net GND: now also C10.2, C11.2, C12.2, C13.2, C15.2, U4.4 (GND), U7.2 (GND)
- net VBUS: now also D7.2 (A); no longer D8.2 (A)
Other:
- note added: "Power tree: +5V is the OR of two sources, so neither can back-feed the other. CONS_5V edge pins 19 / 20, the console's +5V, through D8 SS34. VBUS USB-C, through D7 SS34. SS34 VF ~0.35 V at the cart's ~0.4 A: +5V is 4.4-4.9 V. The only 5 V logic is the two SN74LVC4245A A ports (cart-rp sheet), and they take CONS_5V itself, ahead of the diode: off with the console, so the translators isolate the bu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"
- note removed: "Power tree: +5V is the OR of two sources, so neither can back-feed the other. CONS_5V edge pins 19 / 20, the console's +5V, through D7 SS34. VBUS USB-C, through D8 SS34. SS34 VF ~0.35 V at the cart's ~0.4 A: +5V is 4.4-4.9 V. The only 5 V logic is the two SN74LVC4245A A ports (cart-rp sheet), and they take CONS_5V itself, ahead of the diode: off with the console, so the translators isolate the bu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"
- moved on the sheet: C30, C33, C36, C39, D7, D8
