File: Fairchild-Channel-F/FujiNet-ChannelF-Rev0/usb.kicad_sch (KiCad schematic)
At the start: 15 parts, among them J3 USB-C, U6 CP2102N-A02-GQFN28, U7 UMH3N

Commit message: channel f pcb (#56)
Parts:
- removed C26: 1uF, FujiNet-ChannelF:C_0603_1608Metric, symbol Device:C
- removed C27, C28: 100nF, FujiNet-ChannelF:C_0603_1608Metric, symbol Device:C
- removed C29: 4.7uF, FujiNet-ChannelF:C_0603_1608Metric, symbol Device:C
- removed J3: USB-C, FujiNet-ChannelF:USB_C_Receptacle_HRO_TYPE-C-31-M-12, symbol FujiNet-ChannelF:USB_C_USB2.0_16P_Fn
- removed R16, R17: 5.1k, FujiNet-ChannelF:R_0603_1608Metric, symbol Device:R
- removed R18: 22k, FujiNet-ChannelF:R_0603_1608Metric, symbol Device:R
- removed R19: 47k, FujiNet-ChannelF:R_0603_1608Metric, symbol Device:R
- removed R20: 10k, FujiNet-ChannelF:R_0603_1608Metric, symbol Device:R
- removed U6: CP2102N-A02-GQFN28, FujiNet-ChannelF:QFN-28-1EP_5x5mm_P0.5mm_EP3.35x3.35mm, symbol Interface_USB:CP2102N-Axx-xQFN28
- removed U7: UMH3N, FujiNet-ChannelF:SOT-363_SC-70-6, symbol Transistor_BJT:UMH3N
- added C5: 1uF, FujiNet-ChannelF:C_0603_1608Metric, symbol Device:C
- added C6, C9: 100nF, FujiNet-ChannelF:C_0603_1608Metric, symbol Device:C
- added C8: 4.7uF, FujiNet-ChannelF:C_0603_1608Metric, symbol Device:C
- added J2: USB-C, FujiNet-ChannelF:USB_C_Receptacle_HRO_TYPE-C-31-M-12, symbol FujiNet-ChannelF:USB_C_USB2.0_16P_Fn
- added R3, R4: 5.1k, FujiNet-ChannelF:R_0603_1608Metric, symbol Device:R
- added R7: 10k, FujiNet-ChannelF:R_0603_1608Metric, symbol Device:R
- added R8: 22k, FujiNet-ChannelF:R_0603_1608Metric, symbol Device:R
- added R9: 47k, FujiNet-ChannelF:R_0603_1608Metric, symbol Device:R
- added U2: UMH3N, FujiNet-ChannelF:SOT-363_SC-70-6, symbol Transistor_BJT:UMH3N
- added U3: CP2102N-A02-GQFN28, FujiNet-ChannelF:QFN-28-1EP_5x5mm_P0.5mm_EP3.35x3.35mm, symbol Interface_USB:CP2102N-Axx-xQFN28
- D4, D5, D6: Manufacturer (none) -> onsemi
Connections:
- net +3V3: now also C8.1, C9.1, R7.1, U3.6 (VDD), U3.7 (VREGIN)
- net CC1: now also J2.A5 (CC1), R3.1
- net CC2: now also J2.B5 (CC2), R4.1
- net CP_RST: now also R7.2, U3.9 (~{RST})
- net GND: now also C5.2, C6.2, C8.2, C9.2, J2.A1 (GND), J2.A12 (GND), J2.B1 (GND), J2.B12 (GND), J2.SH (SHIELD), R3.2, R4.2, R9.2, U3.23 (~{CTS}), U3.29 (GND), U3.3 (GND)
- net S3_EN: now also U2.6 (C1)
- net S3_IO0: now also U2.3 (C2)
- net S3_RXD: now also U3.26 (TXD)
- net S3_TXD: now also U3.25 (RXD)
- net UART_DTR: now also U2.2 (B1), U2.4 (E2), U3.28 (~{DTR})
- net UART_RTS: now also U2.1 (E1), U2.5 (B2), U3.24 (~{RTS})
- net UBRG_DM: now also D6.1 (K), J2.A7 (D-), J2.B7 (D-), U3.5 (D-); no longer D5.1 (K)
- net UBRG_DP: now also J2.A6 (D+), J2.B6 (D+), U3.4 (D+)
- net VBUS: now also D5.1 (K), C5.1, C6.1, J2.A4 (VBUS), J2.A9 (VBUS), J2.B4 (VBUS), J2.B9 (VBUS), R8.1; no longer D6.1 (K)
- net VBUS_SNS: now also R8.2, R9.1, U3.8 (VBUS)
Other:
- moved on the sheet: D5, D6
Changed lines of the file:
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@@
 		(on_board yes)
 		(dnp no)
-		(property "Reference" "U6"
+		(property "Reference" "U3"
 			(at 187.96 107.442 0)
 			(effects
@@
 		)
 		(property "MPN" "CP2102N-A02-GQFN28R"
+			(at 198.12 139.7 0)
+			(effects
+				(font
+					(size 1.27 1.27)
+				)
+				(hide yes)
+			)
+		)
+		(property "Manufacturer" "Silicon Labs"
 			(at 198.12 139.7 0)
 			(effects
@@
 			(project "FujiNet-ChannelF-Rev0"
 				(path "/94e41297-bf02-5fe3-9e3f-23dd2de0dc13/ed7d2797-f6fd-5e59-a65f-20b06df2bfd6"
-					(reference "U6")
+					(reference "U3")
 					(unit 1)
 				)
@@
 		(on_board yes)
 		(dnp no)
-		(property "Reference" "C28"
+		(property "Reference" "C9"
 			(at 211.582 96.52 0)
 			(effects
@@
 		)
 		(property "MPN" "CC0603KRX7R9BB104"
+			(at 208.28 97.79 0)
+			(effects
+				(font
+					(size 1.27 1.27)
+				)
+				(hide yes)
+			)
+		)
+		(property "Manufacturer" "YAGEO"
 			(at 208.28 97.79 0)
 			(effects
@@
 			(project "FujiNet-ChannelF-Rev0"
 				(path "/94e41297-bf02-5fe3-9e3f-23dd2de0dc13/ed7d2797-f6fd-5e59-a65f-20b06df2bfd6"
-					(reference "C28")
+					(reference "C9")
 					(unit 1)
 				)
@@
 		(on_board yes)
 		(dnp no)
-		(property "Reference" "C29"
+		(property "Reference" "C8"
 			(at 187.198 96.52 0)
 			(effects
@@
 		)
 		(property "MPN" "CL10A475KO8NNNC"
+			(at 190.5 97.79 0)
+			(effects
+				(font
+					(size 1.27 1.27)
+				)
+				(hide yes)
+			)
+		)
+		(property "Manufacturer" "Samsung Electro-Mechanics"
 			(at 190.5 97.79 0)
 			(effects
@@
 			(project "FujiNet-ChannelF-Rev0"
 				(path "/94e41297-bf02-5fe3-9e3f-23dd2de0dc13/ed7d2797-f6fd-5e59-a65f-20b06df2bfd6"
-					(reference "C29")
+					(reference "C8")
 					(unit 1)
 				)
@@
 		(on_board yes)
 		(dnp no)
-		(property "Reference" "U7"
+		(property "Reference" "U2"
 			(at 151.13 135.89 0)
 			(effects
@@
 		)
 		(property "MPN" "UMH3N"
+			(at 143.51 132.08 0)
+			(effects
+				(font
+					(size 1.27 1.27)
+				)
+				(hide yes)
+			)
+		)
+		(property "Manufacturer" "Jiangsu Changjing (JSCJ)"
 			(at 143.51 132.08 0)
 			(effects
@@
 			(project "FujiNet-ChannelF-Rev0"
 				(path "/94e41297-bf02-5fe3-9e3f-23dd2de0dc13/ed7d2797-f6fd-5e59-a65f-20b06df2bfd6"
-					(reference "U7")
+					(reference "U2")
 					(unit 2)
 				)
@@
 		(on_board yes)
 		(dnp no)
-		(property "Reference" "U7"
+		(property "Reference" "U2"
 			(at 133.35 153.67 0)
 			(effects
@@
 		)
 		(property "MPN" "UMH3N"
+			(at 125.73 149.86 0)
+			(effects
+				(font
+					(size 1.27 1.27)
+				)
+				(hide yes)
+			)
+		)
+		(property "Manufacturer" "Jiangsu Changjing (JSCJ)"
 			(at 125.73 149.86 0)
 			(effects
@@
 			(project "FujiNet-ChannelF-Rev0"
 				(path "/94e41297-bf02-5fe3-9e3f-23dd2de0dc13/ed7d2797-f6fd-5e59-a65f-20b06df2bfd6"
-					(reference "U7")
+					(reference "U2")
 					(unit 1)
 				)
@@
 		(on_board yes)
 		(dnp no)
-		(property "Reference" "R20"
+		(property "Reference" "R7"
 			(at 225.806 104.14 0)
 			(effects
@@
 		)
 		(property "MPN" "0603WAF1002T5E"
+			(at 223.52 105.41 0)
+			(effects
+				(font
+					(size 1.27 1.27)
+				)
+				(hide yes)
+			)
+		)
+		(property "Manufacturer" "UNI-ROYAL"
 			(at 223.52 105.41 0)
 			(effects
@@
 			(project "FujiNet-ChannelF-Rev0"
 				(path "/94e41297-bf02-5fe3-9e3f-23dd2de0dc13/ed7d2797-f6fd-5e59-a65f-20b06df2bfd6"
-					(reference "R20")
+					(reference "R7")
 					(unit 1)
 				)
@@
 		(on_board yes)
 		(dnp no)
-		(property "Reference" "J3"
+		(property "Reference" "J2"
 			(at 299.72 104.902 0)
 			(effects
@@
 		)
 		(property "MPN" "TYPE-C-31-M-12"
+			(at 307.34 129.54 0)
+			(effects
+				(font
+					(size 1.27 1.27)
+				)
+				(hide yes)
+			)
+		)
+		(property "Manufacturer" "Korean Hroparts Elec"
 			(at 307.34 129.54 0)
 			(effects
@@
 			(project "FujiNet-ChannelF-Rev0"
 				(path "/94e41297-bf02-5fe3-9e3f-23dd2de0dc13/ed7d2797-f6fd-5e59-a65f-20b06df2bfd6"
-					(reference "J3")
+					(reference "J2")
 					(unit 1)
 				)
@@
 		(on_board yes)
 		(dnp no)
-		(property "Reference" "D6"
+		(property "Reference" "D5"
 			(at 274.32 99.06 90)
 			(effects
@@
 		)
 		(property "MPN" "ESD5Z5.0T1G"
+			(at 271.78 100.33 90)
+			(effects
+				(font
+					(size 1.27 1.27)
+				)
+				(hide yes)
+			)
+		)
+		(property "Manufacturer" "onsemi"
 			(at 271.78 100.33 90)
 			(effects
@@
 			(project "FujiNet-ChannelF-Rev0"
 				(path "/94e41297-bf02-5fe3-9e3f-23dd2de0dc13/ed7d2797-f6fd-5e59-a65f-20b06df2bfd6"
-					(reference "D6")
+					(reference "D5")
 					(unit 1)
 				)
@@
 		(on_board yes)
 		(dnp no)
-		(property "Reference" "C26"
+		(property "Reference" "C5"
 			(at 262.382 99.06 0)
 			(effects
@@
 		)
 		(property "MPN" "CL10A105KB8NNNC"
+			(at 259.08 100.33 0)
+			(effects
+				(font
+					(size 1.27 1.27)
+				)
+				(hide yes)
+			)
+		)
+		(property "Manufacturer" "Samsung Electro-Mechanics"
 			(at 259.08 100.33 0)
 			(effects
@@
 			(project "FujiNet-ChannelF-Rev0"
 				(path "/94e41297-bf02-5fe3-9e3f-23dd2de0dc13/ed7d2797-f6fd-5e59-a65f-20b06df2bfd6"
-					(reference "C26")
+					(reference "C5")
 					(unit 1)
 				)
@@
 		(on_board yes)
 		(dnp no)
-		(property "Reference" "C27"
+		(property "Reference" "C6"
 			(at 249.682 99.06 0)
 			(effects
@@
 		)
 		(property "MPN" "CC0603KRX7R9BB104"
+			(at 246.38 100.33 0)
+			(effects
+				(font
+					(size 1.27 1.27)
+				)
+				(hide yes)
+			)
+		)
+		(property "Manufacturer" "YAGEO"
 			(at 246.38 100.33 0)
 			(effects
@@
 			(project "FujiNet-ChannelF-Rev0"
 				(path "/94e41297-bf02-5fe3-9e3f-23dd2de0dc13/ed7d2797-f6fd-5e59-a65f-20b06df2bfd6"
-					(reference "C27")
+					(reference "C6")
 					(unit 1)
 				)
@@
 		(on_board yes)
 		(dnp no)
-		(property "Reference" "R18"
+		(property "Reference" "R8"
 			(at 233.934 99.06 0)
 			(effects
@@
 		)
 		(property "MPN" "0603WAF2202T5E"
+			(at 236.22 100.33 0)
+			(effects
+				(font
+					(size 1.27 1.27)
+				)
+				(hide yes)
+			)
+		)
+		(property "Manufacturer" "UNI-ROYAL"
 			(at 236.22 100.33 0)
 			(effects
@@
 			(project "FujiNet-ChannelF-Rev0"
 				(path "/94e41297-bf02-5fe3-9e3f-23dd2de0dc13/ed7d2797-f6fd-5e59-a65f-20b06df2bfd6"
-					(reference "R18")
+					(reference "R8")
 					(unit 1)
 				)
@@
 		(on_board yes)
 		(dnp no)
-		(property "Reference" "R19"
+		(property "Reference" "R9"
 			(at 245.11 119.126 90)
 			(effects
@@
 		)
 		(property "MPN" "0603WAF4702T5E"
+			(at 245.11 124.46 90)
+			(effects
+				(font
+					(size 1.27 1.27)
+				)
+				(hide yes)
+			)
+		)
+		(property "Manufacturer" "UNI-ROYAL"
 			(at 245.11 124.46 90)
 			(effects
@@
 			(project "FujiNet-ChannelF-Rev0"
 				(path "/94e41297-bf02-5fe3-9e3f-23dd2de0dc13/ed7d2797-f6fd-5e59-a65f-20b06df2bfd6"
-					(reference "R19")
+					(reference "R9")
 					(unit 1)
 				)
@@
 		(on_board yes)
 		(dnp no)
-		(property "Reference" "R16"
+		(property "Reference" "R3"
 			(at 285.75 103.886 90)
 			(effects
@@
 		)
 		(property "MPN" "0603WAF5101T5E"
+			(at 285.75 109.22 90)
+			(effects
+				(font
+					(size 1.27 1.27)
+				)
+				(hide yes)
+			)
+		)
+		(property "Manufacturer" "UNI-ROYAL"
 			(at 285.75 109.22 90)
 			(effects
@@
 			(project "FujiNet-ChannelF-Rev0"
 				(path "/94e41297-bf02-5fe3-9e3f-23dd2de0dc13/ed7d2797-f6fd-5e59-a65f-20b06df2bfd6"
-					(reference "R16")
+					(reference "R3")
 					(unit 1)
 				)
@@
 		(on_board yes)
 		(dnp no)
-		(property "Reference" "R17"
+		(property "Reference" "R4"
 			(at 285.75 111.506 90)
 			(effects
@@
 		)
 		(property "MPN" "0603WAF5101T5E"
+			(at 285.75 116.84 90)
+			(effects
+				(font
+					(size 1.27 1.27)
+				)
+				(hide yes)
+			)
+		)
+		(property "Manufacturer" "UNI-ROYAL"
 			(at 285.75 116.84 90)
 			(effects
@@
 			(project "FujiNet-ChannelF-Rev0"
 				(path "/94e41297-bf02-5fe3-9e3f-23dd2de0dc13/ed7d2797-f6fd-5e59-a65f-20b06df2bfd6"
-					(reference "R17")
+					(reference "R4")
 					(unit 1)
 				)
@@
 		(on_board yes)
 		(dnp no)
-		(property "Reference" "D5"
+		(property "Reference" "D6"
 			(at 270.51 116.332 0)
 			(effects
@@
 		)
 		(property "MPN" "ESD5Z5.0T1G"
+			(at 270.51 121.92 0)
+			(effects
+				(font
+					(size 1.27 1.27)
+				)
+				(hide yes)
+			)
+		)
+		(property "Manufacturer" "onsemi"
 			(at 270.51 121.92 0)
 			(effects
@@
 			(project "FujiNet-ChannelF-Rev0"
 				(path "/94e41297-bf02-5fe3-9e3f-23dd2de0dc13/ed7d2797-f6fd-5e59-a65f-20b06df2bfd6"
-					(reference "D5")
+					(reference "D6")
 					(unit 1)
 				)
@@
 			(at 284.48 140.97 90)
 			(effects
+				(font
+					(size 1.27 1.27)
+				)
+				(hide yes)
+			)
+		)
+		(property "Manufacturer" "onsemi"
+			(at 284.48 140.97 90)
+			(effects
