File: Fairchild-Channel-F/FujiNet-ChannelF-Rev0/FujiNet-ChannelF-Rev0.kicad_pcb (KiCad board)
At the start: 4 copper layers, 77 x 131.5 mm, 106 parts, among them J1 ChannelF_Cart_Edge_22, J2 USB-C, J3 microSD, Q1 2N7002, SW1 RESET, SW2 S3_RST, SW3 S3_BOOT, SW4 BOOTSEL, U1 ESP32-S3-WROOM-1-N16R8, U2 UMH3N, U3 CP2102N-A02-GQFN28, U4 AP63203WU, U5 RP2040, U6 W25Q16JVSSIQ, U7 AP2112K-3.3, U8 SN74LVC4245APWR, U9 SN74LVC4245APWR, Y1 12MHz

Commit message: Channel F Rev0: fix the microSD / USB-C alignment (J2 to the board edge, 3D models)
The same defect as NES Rev0: every cart copies the same HRO USB-C and SOFNG
TF-015 footprints and set_models.py rows.

- J2's shell face sat 1.35 mm inside the grip-end edge, where a plug's
  overmold meets the PCB before the plug mates. HRO's recommended layout
  puts the edge at footprint y +3.19 (face 0.46 mm past it): J2 moves
  (131, 23.5) -> (131, 21.7). tools/usbc_to_edge.py, no re-route: the
  VBUS tie and the CC1 via move with J2 (its B.Cu segment stretches),
  eight 1.8 mm F.Cu stubs join the new pad centres to the old ones, one
  GND stitching via under the new pad row goes. The CC2 exit west and
  the VBUS exit east ran between the shield slots: CC2 now drops at
  x 125.3 outside the slot column; VBUS drops at x 136.9, in place of an
  edge-guard GND via, so the rear slot keeps two F.Cu thermal spokes.
  Front silk past the edge dropped; a Dwgs.User line marks HRO's edge.
- J2's 3D model: offset (0, -1.045, 0), not (0, +1.42, 0).
- J3's 3D model: offset (-0.9, -5.5, 0), not (0, 0, 0). J3's copper and
  position unchanged.

KiCad DRC at every severity with schematic parity on the saved fills:
0 / 0 / 0. check_vias, check_plane_shorts, check_gerbers and check_fab
clean. Drill changes: J2's slots and pegs, the two removed vias, the moved
CC1 via; the CPL changes J2's Y only.

Co-Authored-By: Claude Opus 5.5 <noreply@anthropic.com>
Parts:
- moved J2 1.80 mm to (131.0, 21.7)
Routing:
- net VBUS: track 55.7 -> 61.6 mm
- net GND: track 113.3 -> 116.9 mm, vias 588 -> 586
- net /usb/UBRG_DP: track 24.4 -> 28.0 mm
- net /usb/UBRG_DM: track 25.0 -> 28.6 mm
- net /usb/CC2: track 22.9 -> 25.1 mm
- net /usb/CC1: track 22.0 -> 23.5 mm
Changed lines of the file:
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@@
 	(footprint "FujiNet-ChannelF:USB_C_Receptacle_HRO_TYPE-C-31-M-12"
 		(layer "F.Cu")
-		(at 131 23.5 180)
-		(descr "USB Type-C receptacle for USB 2.0 and PD, http://www.krhro.com/uploads/soft/180320/1-1P320120243.pdf")
+		(at 131 21.7 180)
+		(descr "USB Type-C receptacle for USB 2.0 and PD, http://www.krhro.com/uploads/soft/180320/1-1P320120243.pdf; PCB edge at y 3.19 (HRO recommended layout: 5.79 mm in front of the pegs), the shell face overhangs it by 0.46 mm")
 		(tags "usb usb-c 2.0 pd")
 		(property "Reference" "J2"
@@
 		(duplicate_pad_numbers_are_jumpers no)
 		(fp_line
-			(start 4.7 2)
-			(end 4.7 3.9)
-			(stroke
-				(width 0.12)
-				(type solid)
-			)
-			(layer "F.SilkS")
-		)
-		(fp_line
 			(start 4.7 -1.9)
 			(end 4.7 0.1)
@@
 		)
 		(fp_line
-			(start -4.7 3.9)
-			(end 4.7 3.9)
-			(stroke
-				(width 0.12)
-				(type solid)
-			)
-			(layer "F.SilkS")
-		)
-		(fp_line
-			(start -4.7 2)
-			(end -4.7 3.9)
+			(start -4.7 -1.9)
+			(end -4.7 0.1)
 			(stroke
 				(width 0.12)
@@
 		)
 		(fp_line
-			(start -4.7 -1.9)
-			(end -4.7 0.1)
+			(start -5.32 3.19)
+			(end 5.32 3.19)
 			(stroke
-				(width 0.12)
-				(type solid)
+				(width 0.1)
+				(type dash)
 			)
-			(layer "F.SilkS")
+			(layer "Dwgs.User")
 		)
 		(fp_line
@@
 		(model "${KIPRJMOD}/3d/USB-C_HRO_TYPE-C-31-M-12.step"
 			(offset
-				(xyz 0 1.42 0)
+				(xyz 0 -1.045 0)
 			)
 			(scale
@@
 		(model "${KIPRJMOD}/3d/TF-015.step"
 			(offset
-				(xyz 0 0 0)
+				(xyz -0.9 -5.5 0)
 			)
 			(scale
@@
 	)
 	(segment
-		(start 133.45 26.8998)
-		(end 133.45 27.545)
+		(start 133.45 25.0998)
+		(end 133.45 25.745)
 		(width 0.3)
 		(layer "F.Cu")
@@
 	)
 	(segment
-		(start 135.5844 25.2089)
-		(end 133.4722 25.2089)
+		(start 135.5844 23.4089)
+		(end 133.4722 23.4089)
 		(width 0.3)
 		(layer "F.Cu")
@@
 	)
 	(segment
-		(start 132.985 26.4348)
-		(end 133.45 26.8998)
+		(start 132.985 24.6348)
+		(end 133.45 25.0998)
+		(width 0.3)
+		(layer "F.Cu")
+		(net "VBUS")
+	)
+	(segment
+		(start 136.3 23.4089)
+		(end 135.5844 23.4089)
 		(width 0.3)
 		(layer "F.Cu")
@@
 	)
 	(segment
-		(start 133.4722 25.2089)
-		(end 132.985 25.6961)
+		(start 133.4722 23.4089)
+		(end 132.985 23.8961)
 		(width 0.3)
 		(layer "F.Cu")
@@
 	)
 	(segment
-		(start 134.925 41.7)
-		(end 135 41.775)
+		(start 133.45 25.745)
+		(end 133.45 27.545)
 		(width 0.3)
 		(layer "F.Cu")
@@
 	)
 	(segment
-		(start 137.4908 27.1153)
-		(end 135.5844 25.2089)
+		(start 136.9 24.0089)
+		(end 136.3 23.4089)
+		(width 0.3)
+		(layer "F.Cu")
+		(net "VBUS")
+	)
+	(segment
+		(start 136.9 26.5245)
+		(end 136.9 24.0089)
+		(width 0.3)
+		(layer "F.Cu")
+		(net "VBUS")
+	)
+	(segment
+		(start 134.925 41.7)
+		(end 135 41.775)
 		(width 0.3)
 		(layer "F.Cu")
@@
 	)
 	(segment
-		(start 132.985 25.6961)
-		(end 132.985 26.4348)
+		(start 132.985 23.8961)
+		(end 132.985 24.6348)
 		(width 0.3)
 		(layer "F.Cu")
@@
 	)
 	(segment
+		(start 137.4908 27.1153)
+		(end 136.9 26.5245)
+		(width 0.3)
+		(layer "F.Cu")
+		(net "VBUS")
+	)
+	(segment
 		(start 136.7 41.775)
 		(end 135 41.775)
@@
 	)
 	(segment
+		(start 128.55 25.745)
+		(end 128.55 27.545)
+		(width 0.3)
+		(layer "F.Cu")
+		(net "VBUS")
+	)
+	(segment
 		(start 136.7 41.775)
 		(end 137.4908 40.9842)
@@
 	)
 	(segment
+		(start 134.25 25.745)
+		(end 134.25 27.545)
+		(width 0.3)
+		(layer "F.Cu")
+		(net "GND")
+	)
+	(segment
 		(start 102.6 111.375)
 		(end 102.6 112.275)
@@
 		(net "GND")
 	)
+	(segment
+		(start 127.75 25.745)
+		(end 127.75 27.545)
+		(width 0.3)
+		(layer "F.Cu")
+		(net "GND")
+	)
 	(via
 		(at 122.53 47.57)
@@
 	)
 	(via
-		(at 131.56 26.08)
-		(size 0.6)
-		(drill 0.3)
-		(layers "F.Cu" "B.Cu")
-		(locked yes)
-		(net "GND")
-	)
-	(via
 		(at 118.7 53.7)
 		(size 0.6)
@@
 	)
 	(via
-		(at 137.3 25.94)
-		(size 0.6)
-		(drill 0.3)
-		(layers "F.Cu" "B.Cu")
-		(locked yes)
-		(net "GND")
-	)
-	(via
 		(at 80.24 132.04)
 		(size 0.6)
@@
 	)
 	(segment
-		(start 129.25 26.0427)
-		(end 128.4691 25.2618)
+		(start 129.25 24.2427)
+		(end 128.4691 23.4618)
 		(width 0.2)
 		(layer "F.Cu")
@@
 	)
 	(segment
-		(start 129.25 27.545)
-		(end 129.25 26.0427)
+		(start 129.25 25.745)
+		(end 129.25 24.2427)
 		(width 0.2)
 		(layer "F.Cu")
@@
 	)
 	(segment
-		(start 126.367 25.2618)
-		(end 125.2992 26.3296)
+		(start 126.367 23.4618)
+		(end 125.7004 23.4618)
 		(width 0.2)
 		(layer "F.Cu")
@@
 	)
 	(segment
+		(start 125.2992 23.8626)
+		(end 125.2992 26.3296)
+		(width 0.2)
+		(layer "F.Cu")
+		(net "/usb/CC2")
+	)
+	(segment
 		(start 122.4856 36.9105)
 		(end 122.4856 40.8894)
@@
 	)
 	(segment
-		(start 128.4691 25.2618)
-		(end 126.367 25.2618)
+		(start 125.7004 23.4618)
+		(end 125.2992 23.8626)
+		(width 0.2)
+		(layer "F.Cu")
+		(net "/usb/CC2")
+	)
+	(segment
+		(start 128.4691 23.4618)
+		(end 126.367 23.4618)
 		(width 0.2)
 		(layer "F.Cu")
@@
 	)
 	(segment
+		(start 131.25 25.745)
+		(end 131.25 27.545)
+		(width 0.15)
+		(layer "F.Cu")
+		(net "/usb/UBRG_DP")
+	)
+	(segment
 		(start 125.6875 43.7509)
 		(end 125.6875 42.4125)
@@
 	)
 	(segment
+		(start 130.25 25.745)
+		(end 130.25 27.545)
+		(width 0.15)
+		(layer "F.Cu")
+		(net "/usb/UBRG_DP")
+	)
+	(segment
 		(start 100.8125 39.4)
 		(end 100.8125 41.1875)
@@
 	)
 	(segment
+		(start 131.75 25.745)
+		(end 131.75 27.545)
+		(width 0.15)
+		(layer "F.Cu")
+		(net "/usb/UBRG_DM")
+	)
+	(segment
 		(start 128.6861 41.77)
 		(end 127.0564 43.3997)
@@
 	)
 	(segment
+		(start 130.75 25.745)
+		(end 130.75 27.545)
+		(width 0.15)
+		(layer "F.Cu")
+		(net "/usb/UBRG_DM")
+	)
+	(segment
 		(start 131.75 28.85)
 		(end 131.75 30.3406)
@@
 	)
 	(segment
-		(start 132.25 27.545)
-		(end 132.25 26.3661)
+		(start 132.25 25.745)
+		(end 132.25 24.5661)
 		(width 0.2)
 		(layer "F.Cu")
@@
 	)
 	(via
-		(at 132.25 26.3661)
+		(at 132.25 24.5661)
 		(size 0.6)
 		(drill 0.3)
@@
 	(segment
 		(start 129.7652 28.8509)
-		(end 132.25 26.3661)
+		(end 132.25 24.5661)
 		(width 0.2)
 		(layer "B.Cu")
