File: RCA-Studio-II/FujiNet-StudioII-Rev0/cart-bus.kicad_sch (KiCad schematic)
At the start: 38 parts, among them J1 StudioII_Cart_Edge_22, J2 DBG UART, U1 RP2354B, U2 74HCT541, U3 74HCT1G02, U4 74HCT32, U5 74HCT14

Commit message: Studio II Rev0: ESP32-S3 on the cart, 4-layer board, JLCPCB package
The schematic is redone with the FujiNet's ESP32-S3 on the cartridge (it was
on a separate board), and the board is laid out, routed and audited for
JLCPCB assembly.

Schematic (5 sheets: cart-bus, rp-core, fujinet, usb, power):
- ESP32-S3-WROOM-1-N16R8 as the FujiNet and the RP2354B's USB host, with
  microSD, WS2812, EN RC and buttons (ported from FujiNet-ChannelF Rev0)
- USB-C -> USBLC6-2SC6 -> CP2102N with the UMH3N auto-program pair
- a TPS2116 power mux (USB first, the console's 5 V second) replaces the
  P-FET / SS34 OR, so the 74HCT glue stays at >= 4.72 V on either source
- AP63203 buck for the S3 side; RESET reaches both MCUs; the S3 drives the
  RP's RUN / BOOTSEL through 1k
- ERC 0, netlist parity 97 / 97, check_nets 364 / 0 failed / 1 warning
  (fujiversal-studio2.h lacks PIN_RP2040_RUN / _BOOTSEL), margins positive

Board: FliP's multicart outline from the insertion edge, 28 mm taller
(90.9 x 111.5 mm, printed shell), 22 hard-gold fingers on B.Cu, 4 layers,
every part on F.Cu; the S3 flush at the top edge with its antenna keep-out.
- KiCad DRC with schematic parity, all severities: 0 / 0 / 0, on the
  saved zone fills; layout_checks 65 / 65; check_fab 10 / 10
- LAYOUT=1 regenerates and re-routes it from scratch with every gate green

Fixes found by the audit, each now in the generator and gated:
- the gerbers plotted stale zone fills: 427 GND vias sat inside the In2
  power pours. tools/fill_zones.py refills after the last via, DRC runs
  on the saved fills, export uses --check-zones, and check_gerbers.py
  check 9 tests every plated hole against the plotted inner layers
- a 20 mm D+ loop at the flow-through USBLC6: twin pins now joined under
  the body, its 100 nF moved to the VBUS pin as ST draws it
- the USB-C 1.35 mm inside the edge: moved to HRO's layout (face 0.46 mm
  past the edge), USB-C and microSD 3D models fixed (FujiNet-NES 63ccf57)
- the antenna keep-out added as board ru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
Connections:
- net D0: now also U2.11 (Y7); no longer U2.18 (Y0)
- net D1: now also U2.12 (Y6); no longer U2.17 (Y1)
- net D2: now also U2.13 (Y5); no longer U2.16 (Y2)
- net D3: now also U2.14 (Y4); no longer U2.15 (Y3)
- net D4: now also U2.15 (Y3); no longer U2.14 (Y4)
- net D5: now also U2.16 (Y2); no longer U2.13 (Y5)
- net D6: now also U2.17 (Y1); no longer U2.12 (Y6)
- net D7: now also U2.18 (Y0); no longer U2.11 (Y7)
- net RP_D0: now also U2.9 (A7); no longer U2.2 (A0)
- net RP_D1: now also U2.8 (A6); no longer U2.3 (A1)
- net RP_D2: now also U2.7 (A5); no longer U2.4 (A2)
- net RP_D3: now also U2.6 (A4); no longer U2.5 (A3)
- net RP_D4: now also U2.5 (A3); no longer U2.6 (A4)
- net RP_D5: now also U2.4 (A2); no longer U2.7 (A5)
- net RP_D6: now also U2.3 (A1); no longer U2.8 (A6)
- net RP_D7: now also U2.2 (A0); no longer U2.9 (A7)
Changed lines of the file:
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@@
 	(title_block
 		(title "FujiNet Studio II Rev0 - Cart bus: edge, glue, RP GPIO")
-		(date "2026-10-10")
+		(date "2026-10-11")
 		(rev "0")
 		(company "FujiNet")
 		(comment 1 "Generated from tools/design.py + tools/sch_layout.py - edit those, not this file")
-		(comment 2 "CERN-OHL-W-2.0 (core and generators from FujiNet-5200-Rev0)")
-		(comment 3 "Rev0 2026-10-10: schematic only; firmware pico/studio2 s2_cart.h")
+		(comment 2 "CERN-OHL-W-2.0 (RP core from FujiNet-5200-Rev0, S3 half from FujiNet-ChannelF-Rev0)")
+		(comment 3 "Rev0 2026-10-11: RP2354B + ESP32-S3; firmware pico/studio2 s2_cart.h, fujiversal-studio2.h")
 	)
 	(symbol
@@
 			)
 		)
-		(property "Description" "RCA Studio II 22-pin cartridge edge, 3.96 mm (0.156\") pitch, contacts on one face (PROVISIONAL geometry)"
+		(property "Description" "RCA Studio II 22-pin cartridge edge, 0.156\" (3.9624 mm) pitch, contacts on one face (B.Cu), FliP multicart geometry"
 			(at 48.26 129.54 0)
 			(effects
@@
 	(wire
 		(pts
-			(xy 58.42 55.88)
-			(xy 109.22 55.88)
+			(xy 58.42 73.66)
+			(xy 109.22 73.66)
 		)
 		(stroke
@@
 	(wire
 		(pts
-			(xy 134.62 55.88)
-			(xy 241.3 55.88)
+			(xy 134.62 73.66)
+			(xy 241.3 73.66)
 		)
 		(stroke
@@
 	(wire
 		(pts
-			(xy 58.42 58.42)
-			(xy 109.22 58.42)
+			(xy 58.42 71.12)
+			(xy 109.22 71.12)
 		)
 		(stroke
@@
 	(wire
 		(pts
-			(xy 134.62 58.42)
-			(xy 241.3 58.42)
+			(xy 134.62 71.12)
+			(xy 241.3 71.12)
 		)
 		(stroke
@@
 	(wire
 		(pts
-			(xy 58.42 60.96)
-			(xy 109.22 60.96)
+			(xy 58.42 68.58)
+			(xy 109.22 68.58)
 		)
 		(stroke
@@
 	(wire
 		(pts
-			(xy 134.62 60.96)
-			(xy 241.3 60.96)
+			(xy 134.62 68.58)
+			(xy 241.3 68.58)
 		)
 		(stroke
@@
 	(wire
 		(pts
-			(xy 58.42 63.5)
-			(xy 109.22 63.5)
+			(xy 58.42 66.04)
+			(xy 109.22 66.04)
 		)
 		(stroke
@@
 	(wire
 		(pts
-			(xy 134.62 63.5)
-			(xy 241.3 63.5)
+			(xy 134.62 66.04)
+			(xy 241.3 66.04)
 		)
 		(stroke
@@
 	(wire
 		(pts
-			(xy 58.42 66.04)
-			(xy 109.22 66.04)
+			(xy 58.42 63.5)
+			(xy 109.22 63.5)
 		)
 		(stroke
@@
 	(wire
 		(pts
-			(xy 134.62 66.04)
-			(xy 241.3 66.04)
+			(xy 134.62 63.5)
+			(xy 241.3 63.5)
 		)
 		(stroke
@@
 	(wire
 		(pts
-			(xy 58.42 68.58)
-			(xy 109.22 68.58)
+			(xy 58.42 60.96)
+			(xy 109.22 60.96)
 		)
 		(stroke
@@
 	(wire
 		(pts
-			(xy 134.62 68.58)
-			(xy 241.3 68.58)
+			(xy 134.62 60.96)
+			(xy 241.3 60.96)
 		)
 		(stroke
@@
 	(wire
 		(pts
-			(xy 58.42 71.12)
-			(xy 109.22 71.12)
+			(xy 58.42 58.42)
+			(xy 109.22 58.42)
 		)
 		(stroke
@@
 	(wire
 		(pts
-			(xy 134.62 71.12)
-			(xy 241.3 71.12)
+			(xy 134.62 58.42)
+			(xy 241.3 58.42)
 		)
 		(stroke
@@
 	(wire
 		(pts
-			(xy 58.42 73.66)
-			(xy 109.22 73.66)
+			(xy 58.42 55.88)
+			(xy 109.22 55.88)
 		)
 		(stroke
@@
 	(wire
 		(pts
-			(xy 134.62 73.66)
-			(xy 241.3 73.66)
+			(xy 134.62 55.88)
+			(xy 241.3 55.88)
 		)
 		(stroke
@@
 	)
 	(label "D0"
-		(at 59.69 55.88 0)
+		(at 59.69 73.66 0)
 		(effects
 			(font
@@
 	)
 	(label "RP_D0"
-		(at 135.89 55.88 0)
+		(at 135.89 73.66 0)
 		(effects
 			(font
@@
 	)
 	(label "D1"
-		(at 59.69 58.42 0)
+		(at 59.69 71.12 0)
 		(effects
 			(font
@@
 	)
 	(label "RP_D1"
-		(at 135.89 58.42 0)
+		(at 135.89 71.12 0)
 		(effects
 			(font
@@
 	)
 	(label "D2"
-		(at 59.69 60.96 0)
+		(at 59.69 68.58 0)
 		(effects
 			(font
@@
 	)
 	(label "RP_D2"
-		(at 135.89 60.96 0)
+		(at 135.89 68.58 0)
 		(effects
 			(font
@@
 	)
 	(label "D3"
-		(at 59.69 63.5 0)
+		(at 59.69 66.04 0)
 		(effects
 			(font
@@
 	)
 	(label "RP_D3"
-		(at 135.89 63.5 0)
+		(at 135.89 66.04 0)
 		(effects
 			(font
@@
 	)
 	(label "D4"
-		(at 59.69 66.04 0)
+		(at 59.69 63.5 0)
 		(effects
 			(font
@@
 	)
 	(label "RP_D4"
-		(at 135.89 66.04 0)
+		(at 135.89 63.5 0)
 		(effects
 			(font
@@
 	)
 	(label "D5"
-		(at 59.69 68.58 0)
+		(at 59.69 60.96 0)
 		(effects
 			(font
@@
 	)
 	(label "RP_D5"
-		(at 135.89 68.58 0)
+		(at 135.89 60.96 0)
 		(effects
 			(font
@@
 	)
 	(label "D6"
-		(at 59.69 71.12 0)
+		(at 59.69 58.42 0)
 		(effects
 			(font
@@
 	)
 	(label "RP_D6"
-		(at 135.89 71.12 0)
+		(at 135.89 58.42 0)
 		(effects
 			(font
@@
 	)
 	(label "D7"
-		(at 59.69 73.66 0)
+		(at 59.69 55.88 0)
 		(effects
 			(font
@@
 	)
 	(label "RP_D7"
-		(at 135.89 73.66 0)
+		(at 135.89 55.88 0)
 		(effects
 			(font
@@
 		)
 	)
-	(text "The glue (s2_cart.h): the '541 (U2) drives D0-D7 while /OE1 = /MRD and\n/OE2 = /DRIVE | /PWROK are both low (s2_glue_drive); CART CS = NOR(/MRD,\n/CLAIM | /PWROK) (U4, U3; s2_glue_cartcs) turns the console RAM off for a\nread the RP claims.  /MRD alone ends both.  With the console off (PWR_OK_N\nhigh) nothing is driven into it, whatever the RP, on USB, left on /DRIVE\nand /CLAIM.  5 V CMOS levels: the 1802 VIH is 3.5 V at 5 V.\nR11 / R12 10k to +5V hold /DRIVE and /CLAIM high, the cart silent, while\nthe RP is unpowered or booting (they beat its reset pull-down; RP2350-E9).\nPWR_OK: edge 15 (the console's 5 V, before the P-FET) through R13 / R14 into\ntwo '14 Schmitt stages; the first, PWR_OK_N, gates the two ORs.  Every\nconsole line reaches the RP through 330R; GPIO0-31 are 5 V tolerant\nwhenever IOVDD is up.  ADC0 (GPIO40) reads edge 15 through R15 / R16.\nEdge pin 6 (ROM DISABLE) is grounded, as on a stock cartridge."
+	(text "The glue (s2_cart.h): the '541 (U2) drives D0-D7 while /OE1 = /MRD and\n/OE2 = /DRIVE | /PWROK are both low (s2_glue_drive); CART CS = NOR(/MRD,\n/CLAIM | /PWROK) (U4, U3; s2_glue_cartcs) turns the console RAM off for a\nread the RP claims.  /MRD alone ends both.  With the console off (PWR_OK_N\nhigh) nothing is driven into it, whatever the RP, on USB, left on /DRIVE\nand /CLAIM.  5 V CMOS levels: the 1802 VIH is 3.5 V at 5 V.\nR11 / R12 10k to +5V hold /DRIVE and /CLAIM high, the cart silent, while\nthe RP is unpowered or booting (they beat its reset pull-down; RP2350-E9).\nPWR_OK: edge 15 (the console's 5 V, before the mux) through R13 / R14 into\ntwo '14 Schmitt stages; the first, PWR_OK_N, gates the two ORs.  Every\nconsole line reaches the RP through 330R; GPIO0-31 are 5 V tolerant\nwhenever IOVDD is up.  ADC0 (GPIO40) reads edge 15 through R15 / R16.\nEdge pin 6 (ROM DISABLE) is grounded, as on a stock cartridge."
 		(exclude_from_sim no)
 		(at 304.8 198.12 0)
