File: RCA-Studio-II/FujiNet-StudioII-Rev0/rp-core.kicad_sch (KiCad schematic)
At the start: 37 parts, among them SW1 RESET, SW2 BOOTSEL, U1 RP2354B, Y1 12MHz

Commit message: Studio II Rev0: ESP32-S3 on the cart, 4-layer board, JLCPCB package
The schematic is redone with the FujiNet's ESP32-S3 on the cartridge (it was
on a separate board), and the board is laid out, routed and audited for
JLCPCB assembly.

Schematic (5 sheets: cart-bus, rp-core, fujinet, usb, power):
- ESP32-S3-WROOM-1-N16R8 as the FujiNet and the RP2354B's USB host, with
  microSD, WS2812, EN RC and buttons (ported from FujiNet-ChannelF Rev0)
- USB-C -> USBLC6-2SC6 -> CP2102N with the UMH3N auto-program pair
- a TPS2116 power mux (USB first, the console's 5 V second) replaces the
  P-FET / SS34 OR, so the 74HCT glue stays at >= 4.72 V on either source
- AP63203 buck for the S3 side; RESET reaches both MCUs; the S3 drives the
  RP's RUN / BOOTSEL through 1k
- ERC 0, netlist parity 97 / 97, check_nets 364 / 0 failed / 1 warning
  (fujiversal-studio2.h lacks PIN_RP2040_RUN / _BOOTSEL), margins positive

Board: FliP's multicart outline from the insertion edge, 28 mm taller
(90.9 x 111.5 mm, printed shell), 22 hard-gold fingers on B.Cu, 4 layers,
every part on F.Cu; the S3 flush at the top edge with its antenna keep-out.
- KiCad DRC with schematic parity, all severities: 0 / 0 / 0, on the
  saved zone fills; layout_checks 65 / 65; check_fab 10 / 10
- LAYOUT=1 regenerates and re-routes it from scratch with every gate green

Fixes found by the audit, each now in the generator and gated:
- the gerbers plotted stale zone fills: 427 GND vias sat inside the In2
  power pours. tools/fill_zones.py refills after the last via, DRC runs
  on the saved fills, export uses --check-zones, and check_gerbers.py
  check 9 tests every plated hole against the plotted inner layers
- a 20 mm D+ loop at the flow-through USBLC6: twin pins now joined under
  the body, its 100 nF moved to the VBUS pin as ST draws it
- the USB-C 1.35 mm inside the edge: moved to HRO's layout (face 0.46 mm
  past the edge), USB-C and microSD 3D models fixed (FujiNet-NES 63ccf57)
- the antenna keep-out added as board ru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
Parts:
- added D2: BAT54C, FujiNet-StudioII:SOT-23, symbol Diode:BAT54C
- added R25, R26: 27R, FujiNet-StudioII:RPI_R0402, symbol Device:R
- C12, C16, C22: footprint FujiNet-StudioII:C_0603_1608Metric -> FujiNet-StudioII:RPI_C0402; LCSC C14663 -> C1525; MPN CC0603KRX7R9BB104 -> CL05B104KO5NNNC; Manufacturer YAGEO -> Samsung Electro-Mechanics
- C19, C23: footprint FujiNet-StudioII:C_0603_1608Metric -> FujiNet-StudioII:RPI_C0402_wide; LCSC C19666 -> C23733; MPN CL10A475KO8NNNC -> CL05A475MP5NRNC
- C24: footprint FujiNet-StudioII:C_0603_1608Metric -> FujiNet-StudioII:RPI_C0402; LCSC C19666 -> C23733; MPN CL10A475KO8NNNC -> CL05A475MP5NRNC
- R18: footprint FujiNet-StudioII:R_0603_1608Metric -> FujiNet-StudioII:RPI_R0402; LCSC C23140 -> C25105; MPN 0603WAF330JT5E -> 0402WGF330JTCE
- R21: value 10k -> 1k; LCSC C25804 -> C21190; MPN 0603WAF1002T5E -> 0603WAF1001T5E
- R22: value 1k -> 10k; LCSC C21190 -> C25804; MPN 0603WAF1001T5E -> 0603WAF1002T5E
- R23, R24: value 27R -> 1k; LCSC C25190 -> C21190; MPN 0603WAF270JT5E -> 0603WAF1001T5E
- SW1: value RESET -> BOOTSEL
- SW2: value BOOTSEL -> RESET
Connections:
- net +3V3: now also R22.1; no longer R21.1
- net BOOTSEL_BTN: now also R23.2, SW1.1; no longer R22.2, SW2.1
- net QSPI_SS: now also R22.2, R23.1, R24.2; no longer R21.2, R22.1
- net RP_USB_DM: now also R26.2; no longer R24.2
- net RP_USB_DP: now also R25.2; no longer R23.2
- net RUN: now also R21.2, D2.1; no longer SW1.1
- net USB_DM: now also R26.1; no longer R24.1
- net USB_DP: now also R25.1; no longer R23.1
- new net BOOTSEL_CTL: R24.1
- new net RST_BTN: D2.3, SW2.1
- new net RUN_CTL: R21.1
- new net S3_EN: D2.2
Other:
- note added: "Supplies (RP2350 datasheet 6.3.7): IOVDD, QSPI_IOVDD, USB_OTP_VDD, ADC_AVDD and VREG_VIN on +3V3, the AP2112K LDO that rises with +5V; the core regulator switches VREG_LX through 3.3 uH onto DVDD (VREG_FB senses it), its analog supply VREG_AVDD through 33R / 4.7 uF. One 100 nF at every supply pin, drawn at the pin it serves. RESET resets the RP2354B and the ESP32-S3 together (D2 steers RST_BTN on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"
- note removed: "Supplies (RP2350 datasheet 6.3.7): IOVDD, QSPI_IOVDD, USB_OTP_VDD, ADC_AVDD and VREG_VIN on +3V3, the AP2112K LDO that rises with +5V; the core regulator switches VREG_LX through 3.3 uH onto DVDD (VREG_FB senses it), its analog supply VREG_AVDD through 33R / 4.7 uF. One 100 nF at every supply pin, drawn at the pin it serves. RESET pulls RUN low. Hold BOOTSEL while pressing RESET for the RP's USB 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"
- moved on the sheet: C10, C11, C12, C13, C14, C15, C16, C17, C18, C19, C20, C21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
