File: ATARI-2600/Fujiversal-Atari2600-Rev1/Fujiversal-Atari2600-Rev1.kicad_pcb (KiCad board)
At the start: 4 copper layers, 54.4 x 88 mm, 95 parts, among them J1 Atari2600_Cart_Edge_24, J2 microSD, J3 USB-C, Q1 AO3401A, SW1 RESET, SW2 BOOTSEL, SW3 S3_RST, SW4 S3_BOOT, U1 RP2354A, U2 ESP32-S3-WROOM-1-N16R8, U3 CP2102N-A02-GQFN28, U4 UMH3N, U5 AP63203WU, U6 AP2112K-3.3, Y1 12MHz

Commit message: Fujiversal-Atari2600 Rev1: fix the microSD / USB-C alignment (J3 to the board edge, 3D models)
The same defect as NES Rev0: every cart copies the same HRO USB-C and SOFNG
TF-015 footprints and set_models.py rows.

- J3's shell face sat 0.55 mm inside the top edge, where a plug's
  overmold meets the PCB before the plug fully mates. HRO's recommended
  layout puts the edge at footprint y +3.19 (face 0.46 mm past it): J3
  moves (121, 34.2) -> (121, 33.2). tools/usbc_to_edge.py, no re-route:
  the D- tie and the VBUS / CC2 / CC1 vias move with J3 (their B.Cu
  segments stretch), six 1.0 mm F.Cu stubs join the new pad centres to
  the old ones, three GND stitching vias under the new pads / slots / D-
  tie go. The B.Cu CC1 run under the connector moves 1.0 mm north clear
  of the moved peg, slot and vias; the D- exit west is back at 45 degrees.
  Front silk past the edge dropped; a Dwgs.User line marks HRO's edge.
- J3's 3D model: offset (0, -1.045, 0), not (0, +1.42, 0).
- J2's 3D model: offset (-0.9, -5.5, 0), not (0, 0, 0); make_tf015_fp.py
  too. J2's copper and position unchanged.

KiCad DRC at every severity with schematic parity on the saved fills:
0 errors, 0 unconnected, 0 parity, the same 4 silk warnings. No via in a
foreign pad (339), check_plane_shorts clean. Drill changes: J3's slots
and pegs, three removed and three moved vias; the CPL changes J3's Y only.

Co-Authored-By: Claude Opus 5.5 <noreply@anthropic.com>
Parts:
- moved J3 1.00 mm to (121.0, 33.2)
Routing:
- net UBRG_DP: track 20.8 -> 22.8 mm
- net GND: track 84.7 -> 86.7 mm, vias 199 -> 196
- net VBUS: track 83.1 -> 85.1 mm
- net UBRG_DM: track 26.4 -> 27.9 mm
- net CC2: track 13.0 -> 13.9 mm
Changed lines of the file:
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@@
 		(model "${KIPRJMOD}/3d/TF-015.step"
 			(offset
-				(xyz 0 0 0)
+				(xyz -0.9 -5.5 0)
 			)
 			(scale
@@
 	(footprint "Fujiversal-Atari2600:USB_C_Receptacle_HRO_TYPE-C-31-M-12"
 		(layer "F.Cu")
-		(at 121 34.2 180)
-		(descr "USB Type-C receptacle for USB 2.0 and PD, http://www.krhro.com/uploads/soft/180320/1-1P320120243.pdf")
+		(at 121 33.2 180)
+		(descr "USB Type-C receptacle for USB 2.0 and PD, http://www.krhro.com/uploads/soft/180320/1-1P320120243.pdf; PCB edge at y 3.19 (HRO recommended layout: 5.79 mm in front of the pegs), the shell face overhangs it by 0.46 mm")
 		(tags "usb usb-c 2.0 pd")
 		(property "Reference" "J3"
@@
 		(duplicate_pad_numbers_are_jumpers no)
 		(fp_line
-			(start 4.7 2)
-			(end 4.7 3.9)
-			(stroke
-				(width 0.12)
-				(type solid)
-			)
-			(layer "F.SilkS")
-		)
-		(fp_line
 			(start 4.7 -1.9)
 			(end 4.7 0.1)
@@
 		)
 		(fp_line
-			(start -4.7 3.9)
-			(end 4.7 3.9)
-			(stroke
-				(width 0.12)
-				(type solid)
-			)
-			(layer "F.SilkS")
-		)
-		(fp_line
-			(start -4.7 2)
-			(end -4.7 3.9)
+			(start -4.7 -1.9)
+			(end -4.7 0.1)
 			(stroke
 				(width 0.12)
@@
 		)
 		(fp_line
-			(start -4.7 -1.9)
-			(end -4.7 0.1)
+			(start -5.32 3.19)
+			(end 5.32 3.19)
 			(stroke
-				(width 0.12)
-				(type solid)
+				(width 0.1)
+				(type dash)
 			)
-			(layer "F.SilkS")
+			(layer "Dwgs.User")
 		)
 		(fp_line
@@
 		(model "${KIPRJMOD}/3d/USB-C_HRO_TYPE-C-31-M-12.step"
 			(offset
-				(xyz 0 1.42 0)
+				(xyz 0 -1.045 0)
 			)
 			(scale
@@
 	)
 	(segment
+		(start 117.75 37.245)
+		(end 117.75 38.245)
+		(width 0.3)
+		(layer "F.Cu")
+		(net "GND")
+	)
+	(segment
 		(start 113.97 108.4)
 		(end 115.24 108.4)
@@
 	)
 	(segment
+		(start 124.25 37.245)
+		(end 124.25 38.245)
+		(width 0.3)
+		(layer "F.Cu")
+		(net "GND")
+	)
+	(segment
 		(start 122.5 60.33)
 		(end 122.219 61.7)
@@
 	)
 	(via
-		(at 126 35.42)
-		(size 0.6)
-		(drill 0.3)
-		(layers "F.Cu" "B.Cu")
-		(locked yes)
-		(net "GND")
-	)
-	(via
 		(at 113.6 31.2)
 		(size 0.6)
@@
 	)
 	(via
-		(at 116.32 31.2)
-		(size 0.6)
-		(drill 0.3)
-		(layers "F.Cu" "B.Cu")
-		(locked yes)
-		(net "GND")
-	)
-	(via
 		(at 110.677 55.403)
 		(size 0.6)
@@
 	)
 	(via
-		(at 118 33.2)
-		(size 0.6)
-		(drill 0.3)
-		(layers "F.Cu" "B.Cu")
-		(locked yes)
-		(net "GND")
-	)
-	(via
 		(at 126 51.66)
 		(size 0.6)
@@
 	)
 	(segment
+		(start 123.45 37.245)
+		(end 123.45 38.245)
+		(width 0.3)
+		(layer "F.Cu")
+		(net "VBUS")
+	)
+	(segment
 		(start 114.2 41.8748)
 		(end 122.1156 41.8748)
@@
 	)
 	(segment
-		(start 119.05 36.895)
-		(end 118.75 37.445)
+		(start 119.05 35.895)
+		(end 118.75 36.445)
 		(width 0.3)
 		(layer "F.Cu")
@@
 	)
 	(segment
-		(start 118.75 37.445)
-		(end 118.55 38.245)
+		(start 118.75 36.445)
+		(end 118.55 37.245)
 		(width 0.3)
 		(layer "F.Cu")
@@
 	)
 	(via
-		(at 119.05 36.895)
+		(at 119.05 35.895)
 		(size 0.6)
 		(drill 0.3)
@@
 	(segment
 		(start 119.15 36.995)
-		(end 119.05 36.895)
+		(end 119.05 35.895)
 		(width 0.3)
 		(layer "B.Cu")
@@
 	)
 	(segment
-		(start 121.75 37.4726)
-		(end 121.75 38.245)
+		(start 121.75 36.4726)
+		(end 121.75 37.245)
 		(width 0.25)
 		(layer "F.Cu")
@@
 	)
 	(segment
-		(start 120.75 37.5022)
-		(end 121.0133 37.2389)
+		(start 115.9561 32.9318)
+		(end 114.9561 33.9318)
+		(width 0.25)
+		(layer "F.Cu")
+		(net "UBRG_DM")
+	)
+	(segment
+		(start 120.75 36.5022)
+		(end 121.0133 36.2389)
 		(width 0.25)
 		(layer "F.Cu")
@@
 	)
 	(segment
-		(start 116.6399 34.6156)
-		(end 115.9561 33.9318)
+		(start 121.75 37.245)
+		(end 121.75 38.245)
 		(width 0.25)
 		(layer "F.Cu")
@@
 	)
 	(segment
-		(start 115.9561 33.9318)
-		(end 113.9439 33.9318)
+		(start 116.6399 33.6156)
+		(end 115.9561 32.9318)
+		(width 0.25)
+		(layer "F.Cu")
+		(net "UBRG_DM")
+	)
+	(segment
+		(start 121.0133 36.2389)
+		(end 121.5163 36.2389)
 		(width 0.25)
 		(layer "F.Cu")
@@
 	)
 	(segment
-		(start 121.0133 37.2389)
-		(end 121.5163 37.2389)
+		(start 114.9561 33.9318)
+		(end 113.9439 33.9318)
 		(width 0.25)
 		(layer "F.Cu")
@@
 	)
 	(segment
-		(start 121.0133 37.2389)
-		(end 121.0133 36.9871)
+		(start 121.0133 36.2389)
+		(end 121.0133 35.9871)
 		(width 0.25)
 		(layer "F.Cu")
@@
 	)
 	(segment
-		(start 120.75 38.245)
-		(end 120.75 37.5022)
+		(start 120.75 37.245)
+		(end 120.75 36.5022)
 		(width 0.25)
 		(layer "F.Cu")
@@
 	)
 	(segment
-		(start 118.6418 34.6156)
-		(end 116.6399 34.6156)
+		(start 118.6418 33.6156)
+		(end 116.6399 33.6156)
 		(width 0.25)
 		(layer "F.Cu")
@@
 	)
 	(segment
-		(start 121.0133 36.9871)
-		(end 118.6418 34.6156)
+		(start 121.0133 35.9871)
+		(end 118.6418 33.6156)
 		(width 0.25)
 		(layer "F.Cu")
@@
 	)
 	(segment
-		(start 121.5163 37.2389)
-		(end 121.75 37.4726)
+		(start 121.5163 36.2389)
+		(end 121.75 36.4726)
 		(width 0.25)
 		(layer "F.Cu")
@@
 	)
 	(segment
+		(start 120.25 37.245)
+		(end 120.25 38.245)
+		(width 0.25)
+		(layer "F.Cu")
+		(net "UBRG_DP")
+	)
+	(segment
 		(start 116.7 41.2)
 		(end 118.5738 39.3262)
@@
 	)
 	(segment
+		(start 121.25 37.245)
+		(end 121.25 38.245)
+		(width 0.25)
+		(layer "F.Cu")
+		(net "UBRG_DP")
+	)
+	(segment
 		(start 114.4403 38.1369)
 		(end 115.0039 38.7005)
@@
 	)
 	(segment
-		(start 122.25 38.245)
-		(end 122.25 36.7092)
+		(start 122.25 37.245)
+		(end 122.25 35.7092)
 		(width 0.2)
 		(layer "F.Cu")
@@
 	)
 	(via
-		(at 122.25 36.7092)
+		(at 122.25 35.7092)
 		(size 0.6)
 		(drill 0.3)
@@
 	)
 	(segment
-		(start 121.4854 35.9446)
-		(end 113.8809 35.9446)
+		(start 115 34.9446)
+		(end 114 35.9446)
 		(width 0.2)
 		(layer "B.Cu")
@@
 	)
 	(segment
-		(start 122.25 36.7092)
-		(end 121.4854 35.9446)
+		(start 113.8809 35.9446)
+		(end 113.5279 36.2976)
 		(width 0.2)
 		(layer "B.Cu")
@@
 	)
 	(segment
-		(start 113.8809 35.9446)
-		(end 113.5279 36.2976)
+		(start 121.4854 34.9446)
+		(end 115 34.9446)
+		(width 0.2)
+		(layer "B.Cu")
+		(net "CC1")
+	)
+	(segment
+		(start 122.25 35.7092)
+		(end 121.4854 34.9446)
+		(width 0.2)
+		(layer "B.Cu")
+		(net "CC1")
+	)
+	(segment
+		(start 114 35.9446)
+		(end 113.8809 35.9446)
 		(width 0.2)
 		(layer "B.Cu")
@@
 	)
 	(segment
-		(start 119.25 37.5442)
-		(end 119.9654 36.8288)
+		(start 119.25 36.5442)
+		(end 119.9654 35.8288)
 		(width 0.2)
 		(layer "F.Cu")
@@
 	)
 	(segment
-		(start 119.25 38.245)
-		(end 119.25 37.5442)
+		(start 119.25 37.245)
+		(end 119.25 36.5442)
 		(width 0.2)
 		(layer "F.Cu")
@@
 	)
 	(via
-		(at 119.9654 36.8288)
+		(at 119.9654 35.8288)
 		(size 0.6)
 		(drill 0.3)
@@
 	(segment
 		(start 120.3975 37.2609)
-		(end 119.9654 36.8288)
+		(end 119.9654 35.8288)
 		(width 0.2)
 		(layer "B.Cu")
