File: INTV/FujiNet-INTV-Rev0/FujiNet-INTV-Rev0.kicad_pcb (KiCad board)
At the start: 4 copper layers, 58.2 x 78 mm, 84 parts, among them J1 INTV_Cart_Edge_44, J2 microSD, J3 USB-C, Q1 BC847, Q2 BC847, Q3 BC847, SW1 RUN, SW2 BOOTSEL, SW3 RESET, SW4 BOOT, U1 RP2354A, U2 ESP32-S3-WROOM-1-N16R8, U3 CP2102N-A02-GQFN28, U4 UMH3N, U5 AP63203WU, Y1 12MHz

Commit message: INTV Rev0: USB-C (J3) to HRO's board-edge position
The same placement defect as the other carts: J3's shell face sat 1.35 mm
inside the top edge, where a plug's overmold meets the PCB before the plug
mates. HRO's recommended layout puts the edge at footprint y +3.19 (face
0.46 mm past it): J3 moves (60, 77) -> (60, 75.2). The board is not routed
yet, so only the footprint moves. The library footprint gets the fixed
graphics (front silk past the edge dropped, a Dwgs.User line at HRO's
edge) and keeps KiCad's stock model, whose offset 0 is right for KiCad's
stock footprint.

KiCad DRC with schematic parity: no new finding (one silk-over-copper
fewer); the unconnected count is the unrouted board's, unchanged.

Co-Authored-By: Claude Opus 5.5 <noreply@anthropic.com>
Parts:
- moved J3 1.80 mm to (60.0, 75.2)
